Commit message: Update collision box of cam3d_tower and asus
In cam3d_tower
- added a collision offset of 3cm

In robot.urdf
- Switched asus xacro from youbot_description to mcr_description
- Switched camera tower from youbot_description to  mir_description
- Rearranged imports of BRSU includes to match urdf tree order

File: mir_common/mir_description/urdf/misc/cam3d_tower.urdf.xacro (robot description, xacro)
@@ -7,4 +7,5 @@
   <property name="cam3d_tower_width" value="0.03" />
   <property name="cam3d_tower_depth" value="0.03" />
+  <property name="cam3d_tower_collision_offset" value="0.03" />
   <xacro:macro name="cam3d_tower" params="name parent *origin">
   	<link name="${name}_link">
@@ -24,5 +25,5 @@
         <origin xyz="0 0 ${cam3d_tower_height - (cam3d_tower_height/2)}" rpy="0 0 0" />
         <geometry>
-           <box size="${cam3d_tower_depth} ${cam3d_tower_width} ${cam3d_tower_height}"/>
+           <box size="${cam3d_tower_depth + cam3d_tower_collision_offset} ${cam3d_tower_width + cam3d_tower_collision_offset} ${cam3d_tower_height}"/>
         </geometry>
       </collision >

File: mir_robots/mir_hardware_config/youbot-brsu-2/urdf/robot.urdf.xacro (robot description, xacro)
@@ -30,8 +30,8 @@
   </xacro:youbot_arm>
   <!-- BRSU SPECIFIC STUFF -->
-  <xacro:include filename="$(find youbot_description)/urdf/sensors/asus_xtion_camera.urdf.xacro"/>
-  <xacro:include filename="$(find youbot_description)/urdf/misc/camera_tower.urdf.xacro"/>
+  <xacro:include filename="$(find mcr_description)/urdf/materials.urdf.xacro" />
+  <xacro:include filename="$(find mir_description)/urdf/misc/cam3d_tower.urdf.xacro"/>
+  <xacro:include filename="$(find mcr_description)/urdf/sensors/asus_xtion_camera.urdf.xacro"/>
   <xacro:include filename="$(find mcr_description)/urdf/mounts/microsoft_lifecam_1080_mount.urdf.xacro"/>
-  <xacro:include filename="$(find mcr_description)/urdf/materials.urdf.xacro" />
   <xacro:include filename="$(find mir_description)/urdf/grippers/festo_gripper.urdf.xacro" />
   <!-- base laser front -->
@@ -44,7 +44,7 @@
   </xacro:hokuyo_urg04_laser>
   <!-- camera tower -->
-  <xacro:camera_tower name="camera_tower" parent="plate_link">
+  <xacro:cam3d_tower name="camera_tower" parent="plate_link">
     <origin xyz="-0.075 0.0 0.023" rpy="0 0 0" />
-  </xacro:camera_tower>
+  </xacro:cam3d_tower>
   <!-- 3D camera on tower -->
   <xacro:asus_xtion_camera name="tower_cam3d" parent="camera_tower_link" tilt="0.5">
