Commit message: updated for new arm adapter plate
updated origin of adapter plate to centre of arm mounting location
added new adapter plate mesh

File: mir_common/mir_description/urdf/misc/adapter_plate.urdf.xacro (robot description, xacro)
@@ -13,19 +13,19 @@
 		<link name="${name}_link">
 			<inertial>
-				<origin xyz="0 0 0" rpy="0 0 0"/>
+				<origin xyz="-0.09947 -0.09947 0" rpy="${M_PI / 2} 0 0"/>
 				<mass value="1"/>
 				<inertia ixx="0.01" ixy="0" ixz="0" iyy="0.01" iyz="0" izz="0.01" />
 			</inertial>
 			<visual>
-				<origin xyz="0 0 0" rpy="0 0 0" />
+				<origin xyz="-0.09947 0.09947 0" rpy="${M_PI / 2} 0 0" />
 				<geometry>
-					<mesh filename="package://mir_description/meshes/misc/plate.dae"/>
+					<mesh filename="package://mir_description/meshes/misc/adapter_plate.dae"/>
 				</geometry>
 				<material name="DarkGrey"/>
 			</visual>
 			<collision>
-				<origin xyz="0 0 0" rpy="0 0 0" />
+				<origin xyz="-0.09947 0.09947 0" rpy="${M_PI / 2} 0 0" />
 				<geometry>
-					<mesh filename="package://mir_description/meshes/misc/plate.dae" />
+					<mesh filename="package://mir_description/meshes/misc/adapter_plate.dae" />
 				</geometry>
 			</collision>

Commit message: Added adapter_plate_arm_root joint and link
Adapter plate now takes arm_angle as param, and sets up dummy link
Arm is mounted to adapter_plate_arm_root_link at arm_angle.

File: mir_common/mir_description/urdf/misc/adapter_plate.urdf.xacro (robot description, xacro)
@@ -4,5 +4,5 @@
        xmlns:interface="http://playerstage.sourceforge.net/gazebo/xmlschema/#interface"
        xmlns:xacro="http://ros.org/wiki/xacro">
-	<xacro:macro name="adapter_plate" params="parent name *origin">
+	<xacro:macro name="adapter_plate" params="parent name arm_angle *origin">
 		<!-- joint between arm_7_link and sdh_palm_link -->
 		<joint name="${name}_joint" type="fixed" >
@@ -31,4 +31,10 @@
 			</collision>
 		</link>
+		<joint name="${name}_arm_root" type="fixed" >
+			<origin xyz="0 0 0" rpy="0 0 ${arm_angle}" />
+			<parent link="${name}_link" />
+			<child link="${name}_arm_root_link" />
+		</joint>
+		<link name="${name}_arm_root_link" />
 		<!-- extensions -->
 	</xacro:macro>

Commit message: [description] update masses

File: mir_common/mir_description/urdf/misc/adapter_plate.urdf.xacro (robot description, xacro)
@@ -14,5 +14,5 @@
 			<inertial>
 				<origin xyz="-0.09947 -0.09947 0" rpy="${M_PI / 2} 0 0"/>
-				<mass value="1"/>
+				<mass value="0.764"/>
 				<inertia ixx="0.01" ixy="0" ixz="0" iyy="0.01" iyz="0" izz="0.01" />
 			</inertial>

File: mir_common/mir_description/urdf/misc/rear_platform_v2.urdf.xacro (robot description, xacro)
@@ -14,5 +14,5 @@
 			<inertial>
 				<origin xyz="0 0 0" rpy="0 0 0"/>
-				<mass value="1"/>
+				<mass value="2.062"/>
 				<inertia ixx="0.01" ixy="0" ixz="0" iyy="0.01" iyz="0" izz="0.01" />
 			</inertial>
@@ -38,5 +38,5 @@
 			<inertial>
 				<origin xyz="0 0 0" rpy="0 0 0"/>
-				<mass value="1"/>
+				<mass value="${4 * 0.204}"/>
 				<inertia ixx="0.01" ixy="0" ixz="0" iyy="0.01" iyz="0" izz="0.01" />
 			</inertial>
