Commit message: [urdf] Fixed realsense camera macro and missing material

File: mir_common/mir_description/urdf/misc/full_platform.urdf.xacro (robot description, xacro)
@@ -5,4 +5,7 @@
        xmlns:xacro="http://ros.org/wiki/xacro">
 	<xacro:macro name="full_platform" params="parent name arm_angle *origin">
+        <material name="Silver">
+            <color rgba="0.9 0.9 0.9 1.0" />
+        </material>
 		<!-- joint between arm_7_link and sdh_palm_link -->
 		<joint name="${name}_joint" type="fixed" >
@@ -23,5 +26,5 @@
 					<!--mesh filename="package://mir_description/meshes/misc/full_platform.dae"/-->
 				</geometry>
-				<material name="DarkGrey"/>
+				<material name="Silver"/>
 			</visual>
 			<collision>

File: mir_robots/mir_hardware_config/youbot-brsu-2/urdf/robot.urdf.xacro (robot description, xacro)
@@ -25,5 +25,5 @@
   <xacro:include filename="$(find mcr_description)/urdf/sensors/intel_realsense_f200_camera.urdf.xacro"/>
   <xacro:include filename="$(find mir_description)/urdf/sensors/asus_xtion_camera.urdf.xacro"/>
-  <xacro:include filename="$(find mir_description)/urdf/sensors/d435.urdf.xacro"/>
+  <xacro:include filename="$(find mcr_description)/urdf/sensors/realsense_d435.urdf.xacro"/>
   <xacro:include filename="$(find mir_description)/urdf/sensor_mounts/asus_xtion_camera_mount.urdf.xacro"/>
   <!-- Now we can start using the macros included above to define the actual youbot -->
@@ -56,9 +56,6 @@
     <origin xyz="-0.05 -0.01 0.03" rpy="0.0 -${M_PI/2 - 0.03} 0.0" />
   </xacro:intel_realsense_f200_camera -->
-   <xacro:sensor_d435 name="arm_cam3d" parent="camera_mount_link">
-       <!--origin xyz="-0.01 -0.012 0.05" rpy="0 ${M_PI/2 - 0.25} 0.00" /-->
-       <!--origin xyz="0.016 0 0.01" rpy="0 ${M_PI/2 - 0} -0.09" />  -->
-   <origin xyz="0.010 -0.022 0.017" rpy="0 ${M_PI/2 - 0.18} -${M_PI/2}" />
-       <!--origin xyz="0.023 -0.015 0.03" rpy="0 0 0" /-->
-   </xacro:sensor_d435>
+   <xacro:realsense_d435 name="arm_cam3d" parent="camera_mount_link">
+       <origin xyz="0.010 -0.022 0.017" rpy="0 ${M_PI/2 - 0.18} -${M_PI/2}" />
+   </xacro:realsense_d435>
 </robot>
