Commit message: Integrates feedback and fixes issues to get dynamixel gripper working
Simplifies things by adding static fingers in the open position for collision checking.

Limits have been checked on hardware.

The "real" links for the fingers have no Visual of Collison tags, to disable them from any collision checking.

File: mir_common/mir_description/urdf/grippers/dynamixel_gripper.urdf.xacro (robot description, xacro)
@@ -4,7 +4,7 @@
        xmlns:interface="http://playerstage.sourceforge.net/gazebo/xmlschema/#interface"
        xmlns:xacro="http://ros.org/wiki/xacro">
-  <xacro:include filename="$(find youbot_description)/urdf/youbot_gripper/gripper.gazebo.xacro" />
-  <xacro:include filename="$(find youbot_description)/urdf/youbot_gripper/gripper.transmission.xacro" />
-  <xacro:include filename="$(find youbot_description)/urdf/youbot_gripper/limits.urdf.xacro" />
+  <xacro:include filename="$(find mir_description)/urdf/grippers/dynamixel_gripper.gazebo.xacro" />
+  <xacro:include filename="$(find mir_description)/urdf/grippers/dynamixel_gripper.transmission.xacro" />
+  <xacro:include filename="$(find mir_description)/urdf/grippers/dynamixel_limits.urdf.xacro" />
   <xacro:macro name="dynamixel_gripper" params="parent name *origin">
     <!-- joint between arm_5_link and dynamixel_palm_link -->
@@ -51,17 +51,8 @@
         <inertia ixx="0.01" ixy="0" ixz="0" iyy="0.01" iyz="0" izz="0.01" />
       </inertial>
-      <visual>
-        <origin xyz="-0.0125 0 0" rpy="0 0 ${-M_PI/2}" />
-        <geometry>
-          <mesh filename="package://mir_description/meshes/grippers/dynamixel_small_finger_assembly_l.dae" scale="0.01 0.01 0.01" />
-        </geometry>
-        <material name="White" />
-      </visual>
-      <collision>
-        <origin xyz="-0.0125 0 0" rpy="0 0 ${-M_PI/2}" />
-        <geometry>
-          <mesh filename="package://mir_description/meshes/grippers/dynamixel_small_finger_assembly_l_convexhull.dae" scale="0.01 0.01 0.01" />
-        </geometry>
-      </collision>
+      <!--
+        No Visual or Collision tags to avoid collision checking
+        Done below with gripper in static open position
+      -->
     </link>
     <joint name="${name}_finger_joint_r" type="prismatic">
@@ -80,17 +71,8 @@
         <inertia ixx="0.01" ixy="0" ixz="0" iyy="0.01" iyz="0" izz="0.01" />
       </inertial>
-      <visual>
-        <origin xyz="0.0125 0 0" rpy="0 0 ${M_PI/2}" />
-        <geometry>
-          <mesh filename="package://mir_description/meshes/grippers/dynamixel_small_finger_assembly_r.dae" scale="0.01 0.01 0.01" />
-        </geometry>
-        <material name="White" />
-      </visual>
-      <collision>
-        <origin xyz="0.0125 0 0" rpy="0 0 ${M_PI/2}" />
-        <geometry>
-          <mesh filename="package://mir_description/meshes/grippers/dynamixel_small_finger_assembly_r_convexhull.dae" scale="0.01 0.01 0.01" />
-        </geometry>
-      </collision>
+      <!--
+        No Visual or Collision tags to avoid collision checking
+        Done below with gripper in static open position
+      -->
     </link>
     <!-- tip joint -->
@@ -121,7 +103,67 @@
       </inertial>
     </link>
+    <joint name="${name}_static_finger_joint_l" type="fixed">
+      <!--<origin xyz="0.004 0.008 0.046" rpy="0 0 ${M_PI}" />
+      -->
+      <origin xyz="0.0 0.04 0.05" rpy="0 0 ${M_PI}" />
+      <parent link="${name}_palm_link"/>
+      <child link="${name}_static_finger_link_l"/>
+      <axis xyz="0 -1 0" />
+      <dynamics damping="1.0" friction="1.0" />
+      <limit effort="1" velocity="0.1" lower="0" upper="${finger_joint}"/>
+      <safety_controller k_position="20" k_velocity="25" soft_lower_limit="${threshold}" soft_upper_limit="${finger_joint_soft}" />
+    </joint>
+    <link name="${name}_static_finger_link_l">
+      <inertial>
+        <origin xyz="0 -0.001 0" rpy="0 0 0" />
+        <mass value="0.01"/>
+        <inertia ixx="0.01" ixy="0" ixz="0" iyy="0.01" iyz="0" izz="0.01" />
+      </inertial>
+      <visual>
+        <origin xyz="-0.0125 0 0" rpy="0 0 ${-M_PI/2}" />
+        <geometry>
+          <mesh filename="package://mir_description/meshes/grippers/dynamixel_small_finger_assembly_l.dae" scale="0.01 0.01 0.01" />
+        </geometry>
+        <material name="White" />
+      </visual>
+      <collision>
+        <origin xyz="-0.0125 0 0" rpy="0 0 ${-M_PI/2}" />
+        <geometry>
+          <mesh filename="package://mir_description/meshes/grippers/dynamixel_small_finger_assembly_l_convexhull.dae" scale="0.01 0.01 0.01" />
+        </geometry>
+      </collision>
+    </link>
+    <joint name="${name}_static_finger_joint_r" type="fixed">
+      <origin xyz="0.0 -0.04 0.05" rpy="0 0 0" />
+      <parent link="${name}_palm_link"/>
+      <child link="${name}_static_finger_link_r"/>
+      <axis xyz="0 -1 0" />
+      <dynamics damping="1.0" friction="1.0" />
+      <limit effort="1" velocity="0.1" lower="0" upper="${finger_joint}"/>
+      <safety_controller k_position="20" k_velocity="25" soft_lower_limit="${threshold}" soft_upper_limit="${finger_joint_soft}" />
+    </joint>
+    <link name="${name}_static_finger_link_r">
+      <inertial>
+        <origin xyz="0.000 -0.001 0" rpy="0 0 0" />
+        <mass value="0.01"/>
+        <inertia ixx="0.01" ixy="0" ixz="0" iyy="0.01" iyz="0" izz="0.01" />
+      </inertial>
+      <visual>
+        <origin xyz="0.0125 0 0" rpy="0 0 ${M_PI/2}" />
+        <geometry>
+          <mesh filename="package://mir_description/meshes/grippers/dynamixel_small_finger_assembly_r.dae" scale="0.01 0.01 0.01" />
+        </geometry>
+        <material name="White" />
+      </visual>
+      <collision>
+        <origin xyz="0.0125 0 0" rpy="0 0 ${M_PI/2}" />
+        <geometry>
+          <mesh filename="package://mir_description/meshes/grippers/dynamixel_small_finger_assembly_r_convexhull.dae" scale="0.01 0.01 0.01" />
+        </geometry>
+      </collision>
+    </link>
     <!-- extensions -->
-    <xacro:youbot_gripper_gazebo name="${name}" />
-    <xacro:youbot_gripper_transmission name="${name}" />
+    <xacro:dynamixel_gripper_gazebo name="${name}" />
+    <xacro:dynamixel_gripper_transmission name="${name}" />
   </xacro:macro>
 </robot>

Commit message: Rename and set Dynamixel joint limits
Renames from threshold to dynamixel min
Removes soft limit (dynamixel motors have this in firmware)
Renames hard limit

File: mir_common/mir_description/urdf/grippers/dynamixel_gripper.urdf.xacro (robot description, xacro)
@@ -42,6 +42,6 @@
       <axis xyz="0 -1 0" />
       <dynamics damping="1.0" friction="1.0" />
-      <limit effort="1" velocity="0.1" lower="0" upper="${finger_joint}"/>
-      <safety_controller k_position="20" k_velocity="25" soft_lower_limit="${threshold}" soft_upper_limit="${finger_joint_soft}" />
+      <limit effort="1" velocity="0.1" lower="0" upper="${dynamixel_joint_max}"/>
+      <safety_controller k_position="20" k_velocity="25" soft_lower_limit="${dynamixel_joint_min}" soft_upper_limit="${dynamixel_joint_max}" />
     </joint>
     <link name="${name}_finger_link_l">
@@ -62,6 +62,6 @@
       <axis xyz="0 -1 0" />
       <dynamics damping="1.0" friction="1.0" />
-      <limit effort="1" velocity="0.1" lower="0" upper="${finger_joint}"/>
-      <safety_controller k_position="20" k_velocity="25" soft_lower_limit="${threshold}" soft_upper_limit="${finger_joint_soft}" />
+      <limit effort="1" velocity="0.1" lower="0" upper="${dynamixel_joint_max}"/>
+      <safety_controller k_position="20" k_velocity="25" soft_lower_limit="${dynamixel_joint_min}" soft_upper_limit="${dynamixel_joint_max}" />
     </joint>
     <link name="${name}_finger_link_r">
@@ -104,13 +104,7 @@
     </link>
     <joint name="${name}_static_finger_joint_l" type="fixed">
-      <!--<origin xyz="0.004 0.008 0.046" rpy="0 0 ${M_PI}" />
-      -->
       <origin xyz="0.0 0.04 0.05" rpy="0 0 ${M_PI}" />
       <parent link="${name}_palm_link"/>
       <child link="${name}_static_finger_link_l"/>
-      <axis xyz="0 -1 0" />
-      <dynamics damping="1.0" friction="1.0" />
-      <limit effort="1" velocity="0.1" lower="0" upper="${finger_joint}"/>
-      <safety_controller k_position="20" k_velocity="25" soft_lower_limit="${threshold}" soft_upper_limit="${finger_joint_soft}" />
     </joint>
     <link name="${name}_static_finger_link_l">
@@ -138,8 +132,4 @@
       <parent link="${name}_palm_link"/>
       <child link="${name}_static_finger_link_r"/>
-      <axis xyz="0 -1 0" />
-      <dynamics damping="1.0" friction="1.0" />
-      <limit effort="1" velocity="0.1" lower="0" upper="${finger_joint}"/>
-      <safety_controller k_position="20" k_velocity="25" soft_lower_limit="${threshold}" soft_upper_limit="${finger_joint_soft}" />
     </joint>
     <link name="${name}_static_finger_link_r">

File: mir_common/mir_description/urdf/grippers/dynamixel_limits.urdf.xacro (robot description, xacro)
@@ -3,7 +3,6 @@
   <!-- common properties -->
   <property name="M_PI" value="3.1415926535897931" />
-  <property name="threshold" value="0.001" />
   <!-- fingers limits, values are in meters -->
-  <property name="finger_joint" value="2.17" />
-  <property name="finger_joint_soft" value="2.16" />
+  <property name="dynamixel_joint_min" value="0.0" />
+  <property name="dynamixel_joint_max" value="2.17" />
 </robot>
