Commit message: [description] fix masses temporally
to get the arm properly working in simulation

File: mir_common/mir_description/urdf/grippers/dynamixel/v2/festo_finger_mount.urdf.xacro (robot description, xacro)
@@ -13,5 +13,5 @@
       <inertial>
         <origin xyz="0 0 0" rpy="0 0 0"/>
-        <mass value="0.1"/>
+        <mass value="0.001"/>
         <inertia ixx="0.01" ixy="0" ixz="0" iyy="0.01" iyz="0" izz="0.01" />
       </inertial>

File: mir_common/mir_description/urdf/misc/plugbar.xacro (robot description, xacro)
@@ -13,5 +13,5 @@
 			<inertial>
 				<origin xyz="0 0 0" rpy="0 0 0"/>
-				<mass value="1"/>
+				<mass value="0.1"/>
 				<inertia ixx="0.01" ixy="0" ixz="0" iyy="0.01" iyz="0" izz="0.01" />
 			</inertial>

File: mir_common/mir_description/urdf/sensor_mounts/intel_f200_camera_mount.urdf.xacro (robot description, xacro)
@@ -13,5 +13,5 @@
 			<inertial>
 				<origin xyz="0 0 0" rpy="0 0 0"/>
-				<mass value="1"/>
+				<mass value="0.01"/>
 				<inertia ixx="0.01" ixy="0" ixz="0" iyy="0.01" iyz="0" izz="0.01" />
 			</inertial>
