Commit message: [description] add URDF and meshes for dynamixel gripper

File: mir_common/mir_description/urdf/grippers/dynamixel/v2/dynamixel_gripper.urdf.xacro (robot description, xacro)
@@ -4,15 +4,19 @@
        xmlns:interface="http://playerstage.sourceforge.net/gazebo/xmlschema/#interface"
        xmlns:xacro="http://ros.org/wiki/xacro">
-  <xacro:include filename="$(find mir_description)/urdf/grippers/dynamixel/v2/dynamixel_gripper.gazebo.xacro" />
-  <xacro:include filename="$(find mir_description)/urdf/grippers/dynamixel/v2/dynamixel_gripper.transmission.xacro" />
-  <xacro:include filename="$(find mir_description)/urdf/grippers/dynamixel/v2/dynamixel_gripper_limits.urdf.xacro" />
+  <!--xacro:include filename="$(find mir_description)/urdf/grippers/dynamixel/v2/dynamixel_gripper.gazebo.xacro" /-->
+  <!--xacro:include filename="$(find mir_description)/urdf/grippers/dynamixel/v2/dynamixel_gripper.transmission.xacro" /-->
+  <!--xacro:include filename="$(find mir_description)/urdf/grippers/dynamixel/v2/dynamixel_gripper_limits.urdf.xacro" /-->
+  <xacro:include filename="$(find mcr_description)/urdf/motors/dynamixel_motor_ax-12a.urdf.xacro" />
+  <xacro:include filename="$(find mcr_description)/urdf/motors/dynamixel_bracket_fp04-f2.urdf.xacro" />
+  <xacro:include filename="$(find mir_description)/urdf/grippers/dynamixel/v2/festo_finger_mount.urdf.xacro" />
+  <xacro:include filename="$(find mcr_description)/urdf/fingers/festo_finger_dhas-gf-shm.urdf.xacro" />
   <xacro:macro name="dynamixel_gripper_v2" params="parent name *origin">
-    <!-- joint between arm_5_link and dynamixel_palm_link -->
-    <joint name="${name}_palm_joint" type="fixed" >
+    <joint name="${name}_motor_mount_joint" type="fixed" >
       <insert_block name="origin" />
       <parent link="${parent}" />
-      <child link="${name}_palm_link" />
+      <child link="${name}_motor_mount_link" />
     </joint>
-    <link name="${name}_palm_link">
+    <!-- motor mount -->
+    <link name="${name}_motor_mount_link">
       <inertial>
         <origin xyz="0 0 0" rpy="0 0 0"/>
@@ -23,15 +27,42 @@
         <origin xyz="0 0 -0.0275" rpy="0 ${M_PI/2} 0" />
         <geometry>
-          <mesh filename="package://mir_description/meshes/grippers/dynamixel/v2/motor_mount.dae" scale="0.001 0.001 0.001" />
+          <mesh filename="package://mir_description/meshes/grippers/dynamixel/v2/dynamixel_motor_mount.dae" scale="0.001 0.001 0.001" />
         </geometry>
-        <material name="black" />
       </visual>
       <collision>
         <origin xyz="0 0 -0.0275" rpy="0 ${M_PI/2} 0" />
         <geometry>
-          <mesh filename="package://mir_description/meshes/grippers/dynamixel/v2/motor_mount.dae" scale="0.001 0.001 0.001" />
+          <mesh filename="package://mir_description/meshes/grippers/dynamixel/v2/dynamixel_motor_mount_convex_hull.dae" scale="0.001 0.001 0.001" />
         </geometry>
       </collision>
     </link>
+    <!-- motors -->
+    <xacro:dynamixel_motor_AX-12A name="${name}_motor_left" parent="${name}_motor_mount_link">
+      <origin xyz="0.0 0.034 0.021" rpy="0 0 0" />
+    </xacro:dynamixel_motor_AX-12A>
+    <xacro:dynamixel_motor_AX-12A name="${name}_motor_right" parent="${name}_motor_mount_link">
+      <origin xyz="0.0 -0.034 0.021" rpy="0 0 0" />
+    </xacro:dynamixel_motor_AX-12A>
+    <!-- brackets -->
+    <xacro:dynamixel_bracket_FP04-F2 name="${name}_bracket_left" parent="${name}_motor_left_link">
+      <origin xyz="0 0 0" rpy="0 0 0" />
+    </xacro:dynamixel_bracket_FP04-F2>
+    <xacro:dynamixel_bracket_FP04-F2 name="${name}_bracket_right" parent="${name}_motor_right_link">
+      <origin xyz="0 0 0" rpy="0 0 0" />
+    </xacro:dynamixel_bracket_FP04-F2>
+    <!-- finger mounts -->
+    <xacro:festo_finger_mount name="${name}_finger_mount_left" parent="${name}_bracket_left_link">
+      <origin xyz="-0.014 -0.0125 0.026" rpy="0 0 0" />
+    </xacro:festo_finger_mount>
+    <xacro:festo_finger_mount name="${name}_finger_mount_right" parent="${name}_bracket_right_link">
+      <origin xyz="0.014 0.0125 0.026" rpy="0 0 ${M_PI}" />
+    </xacro:festo_finger_mount>
+    <!-- fingers -->
+    <xacro:festo_finger_DHAS-GF-shm name="${name}_finger_left" parent="${name}_finger_mount_left_link">
+      <origin xyz="0.004 0 0.0045" rpy="0 0 0" />
+    </xacro:festo_finger_DHAS-GF-shm>
+    <xacro:festo_finger_DHAS-GF-shm name="${name}_finger_right" parent="${name}_finger_mount_right_link">
+      <origin xyz="0.004 0 0.0045" rpy="0 0 0" />
+    </xacro:festo_finger_DHAS-GF-shm>
   </xacro:macro>
 </robot>

File: mir_common/mir_description/urdf/misc/adapter_plate.urdf.xacro (robot description, xacro)
@@ -27,5 +27,5 @@
 				<origin xyz="-0.09947 0.09947 0" rpy="${M_PI / 2} 0 0" />
 				<geometry>
-					<mesh filename="package://mir_description/meshes/misc/adapter_plate.dae" />
+					<mesh filename="package://mir_description/meshes/misc/adapter_plate_convex_hull.dae" />
 				</geometry>
 			</collision>

File: mir_common/mir_description/urdf/misc/plugbar.xacro (robot description, xacro)
@@ -4,5 +4,5 @@
        xmlns:interface="http://playerstage.sourceforge.net/gazebo/xmlschema/#interface"
        xmlns:xacro="http://ros.org/wiki/xacro">
-	<xacro:macro name="rear_platform_v2" params="parent name *origin">
+	<xacro:macro name="plugbar" params="parent name *origin">
 		<joint name="${name}_joint" type="fixed" >
 			<insert_block name="origin" />
@@ -19,11 +19,12 @@
 				<origin xyz="0 0 0" rpy="0 0 0" />
 				<geometry>
-					<mesh filename="package://mir_description/meshes/misc/rear_platform_v2.dae" scale="0.001 0.001 0.001" />
+					<mesh filename="package://mir_description/meshes/misc/plugbar.dae" scale="0.001 0.001 0.001" />
 				</geometry>
+				<material name="DarkGrey"/>
 			</visual>
 			<collision>
 				<origin xyz="0 0 0" rpy="0 0 0" />
 				<geometry>
-					<mesh filename="package://mir_description/meshes/misc/rear_platform_v2_convex_hull.dae" scale="0.001 0.001 0.001" />
+					<mesh filename="package://mir_description/meshes/misc/plugbar_convex_hull.dae" scale="0.001 0.001 0.001" />
 				</geometry>
 			</collision>

Commit message: [description] correct motor position

File: mir_common/mir_description/urdf/grippers/dynamixel/v2/dynamixel_gripper.urdf.xacro (robot description, xacro)
@@ -39,8 +39,8 @@
     <!-- motors -->
     <xacro:dynamixel_motor_AX-12A name="${name}_motor_left" parent="${name}_motor_mount_link">
-      <origin xyz="0.0 0.034 0.021" rpy="0 0 0" />
+      <origin xyz="0.0 0.034 -0.009" rpy="0 0 0" />
     </xacro:dynamixel_motor_AX-12A>
     <xacro:dynamixel_motor_AX-12A name="${name}_motor_right" parent="${name}_motor_mount_link">
-      <origin xyz="0.0 -0.034 0.021" rpy="0 0 0" />
+      <origin xyz="0.0 -0.034 -0.009" rpy="0 0 0" />
     </xacro:dynamixel_motor_AX-12A>
     <!-- brackets -->

Commit message: [description] use new interface of dynamixel motor URDF

File: mir_common/mir_description/urdf/grippers/dynamixel/v2/dynamixel_gripper.urdf.xacro (robot description, xacro)
@@ -38,8 +38,8 @@
     </link>
     <!-- motors -->
-    <xacro:dynamixel_motor_AX-12A name="${name}_motor_left" parent="${name}_motor_mount_link">
+    <xacro:dynamixel_motor_AX-12A name="${name}_motor_left" parent="${name}_motor_mount_link" motor_direction="1">
       <origin xyz="0.0 0.034 -0.009" rpy="0 0 0" />
     </xacro:dynamixel_motor_AX-12A>
-    <xacro:dynamixel_motor_AX-12A name="${name}_motor_right" parent="${name}_motor_mount_link">
+    <xacro:dynamixel_motor_AX-12A name="${name}_motor_right" parent="${name}_motor_mount_link" motor_direction="-1">
       <origin xyz="0.0 -0.034 -0.009" rpy="0 0 0" />
     </xacro:dynamixel_motor_AX-12A>
@@ -53,8 +53,8 @@
     <!-- finger mounts -->
     <xacro:festo_finger_mount name="${name}_finger_mount_left" parent="${name}_bracket_left_link">
-      <origin xyz="-0.014 -0.0125 0.026" rpy="0 0 0" />
+      <origin xyz="0.014 +0.0125 0.026" rpy="0 0 ${M_PI}" />
     </xacro:festo_finger_mount>
     <xacro:festo_finger_mount name="${name}_finger_mount_right" parent="${name}_bracket_right_link">
-      <origin xyz="0.014 0.0125 0.026" rpy="0 0 ${M_PI}" />
+      <origin xyz="-0.014 -0.0125 0.026" rpy="0 0 0" />
     </xacro:festo_finger_mount>
     <!-- fingers -->

Commit message: [description] update masses of gripper motor mount, intel cam mount and festo finger mount

File: mir_common/mir_description/urdf/grippers/dynamixel/v2/dynamixel_gripper.urdf.xacro (robot description, xacro)
@@ -21,5 +21,5 @@
       <inertial>
         <origin xyz="0 0 0" rpy="0 0 0"/>
-        <mass value="0.1"/>
+        <mass value="0.038"/>
         <inertia ixx="0.01" ixy="0" ixz="0" iyy="0.01" iyz="0" izz="0.01" />
       </inertial>

File: mir_common/mir_description/urdf/grippers/dynamixel/v2/festo_finger_mount.urdf.xacro (robot description, xacro)
@@ -13,5 +13,5 @@
       <inertial>
         <origin xyz="0 0 0" rpy="0 0 0"/>
-        <mass value="0.001"/>
+        <mass value="0.009"/>
         <inertia ixx="0.01" ixy="0" ixz="0" iyy="0.01" iyz="0" izz="0.01" />
       </inertial>

File: mir_common/mir_description/urdf/sensor_mounts/intel_f200_camera_mount.urdf.xacro (robot description, xacro)
@@ -13,5 +13,5 @@
 			<inertial>
 				<origin xyz="0 0 0" rpy="0 0 0"/>
-				<mass value="0.01"/>
+				<mass value="0.028"/>
 				<inertia ixx="0.01" ixy="0" ixz="0" iyy="0.01" iyz="0" izz="0.01" />
 			</inertial>

Commit message: [urdf/moveit] update urdf and moveit config for static tower camera

File: mir_common/mir_description/urdf/grippers/dynamixel/v2/dynamixel_gripper.urdf.xacro (robot description, xacro)
@@ -11,4 +11,5 @@
   <xacro:include filename="$(find mir_description)/urdf/grippers/dynamixel/v2/festo_finger_mount.urdf.xacro" />
   <xacro:include filename="$(find mcr_description)/urdf/fingers/festo_finger_dhas-gf-shm.urdf.xacro" />
+  <xacro:arg name="grasp_link_offset" default="0.11"/>
   <xacro:macro name="dynamixel_gripper_v2" params="parent name *origin">
     <joint name="${name}_motor_mount_joint" type="fixed" >
@@ -17,4 +18,11 @@
       <child link="${name}_motor_mount_link" />
     </joint>
+    <joint name="${name}_static_grasp_link_joint" type="fixed" >
+      <origin xyz="0 0 $(arg grasp_link_offset)" rpy="0 0 0"/>
+      <parent link="${parent}" />
+      <child link="${name}_static_grasp_link" />
+    </joint>
+    <link name="${name}_static_grasp_link">
+    </link>
     <!-- motor mount -->
     <link name="${name}_motor_mount_link">
@@ -45,8 +53,8 @@
     </xacro:dynamixel_motor_AX-12A>
     <!-- brackets -->
-    <xacro:dynamixel_bracket_FP04-F2 name="${name}_bracket_left" parent="${name}_motor_left_link">
+    <xacro:dynamixel_bracket_FP04-F2 name="${name}_bracket_left" parent="${name}_motor_left_base_link">
       <origin xyz="0 0 0" rpy="0 0 0" />
     </xacro:dynamixel_bracket_FP04-F2>
-    <xacro:dynamixel_bracket_FP04-F2 name="${name}_bracket_right" parent="${name}_motor_right_link">
+    <xacro:dynamixel_bracket_FP04-F2 name="${name}_bracket_right" parent="${name}_motor_right_base_link">
       <origin xyz="0 0 0" rpy="0 0 0" />
     </xacro:dynamixel_bracket_FP04-F2>

File: mir_robots/mir_hardware_config/youbot-brsu-2/urdf/robot.urdf.xacro (robot description, xacro)
@@ -16,4 +16,5 @@
   <xacro:include filename="$(find mir_description)/urdf/misc/full_platform.urdf.xacro" />
   <xacro:include filename="$(find mir_description)/urdf/grippers/dynamixel/v2/dynamixel_gripper.urdf.xacro" />
+  <!--xacro:include filename="$(find mir_description)/urdf/grippers/dynamixel/d435_center/dynamixel_gripper.urdf.xacro" /-->
   <!-- controller manager -->
   <xacro:include filename="$(find youbot_description)/controller/ros_controller.urdf.xacro" />
@@ -49,13 +50,35 @@
   </xacro:dynamixel_gripper_v2>
   <!-- camera mount for Intel RealSense F200 -->
-  <xacro:asus_xtion_camera_mount  name="camera_mount" parent="gripper_motor_mount_link">
+  <!--xacro:asus_xtion_camera_mount  name="camera_mount" parent="gripper_motor_mount_link">
       <origin xyz="0.035 -0.00 0.0" rpy="0 0.025 ${M_PI/2} " />
-  </xacro:asus_xtion_camera_mount>
+  </xacro:asus_xtion_camera_mount-->
   <!-- 3D camera on arm -->
   <!-- xacro:intel_realsense_f200_camera name="arm_cam3d" parent="camera_mount_link">
     <origin xyz="-0.05 -0.01 0.03" rpy="0.0 -${M_PI/2 - 0.03} 0.0" />
   </xacro:intel_realsense_f200_camera -->
-   <xacro:realsense_d435 name="arm_cam3d" parent="camera_mount_link">
-       <origin xyz="0.010 -0.022 0.017" rpy="0 ${M_PI/2 - 0.18} -${M_PI/2}" />
+   <xacro:realsense_d435 name="arm_cam3d" parent="base_link">
+       <!--origin xyz="0.25 0.0 0.83" rpy="-0.05 0.917 -0.1" /-->
+       <origin xyz="0.29 -0.03 0.80" rpy="-0.05 1.137 -0.1" />
    </xacro:realsense_d435>
+   <joint name="fixed_camera_joint" type="fixed">
+       <origin xyz="0.0149 0.0325 0.0125" rpy="${-M_PI/2} 0 ${-M_PI/2}" />
+       <parent link="arm_cam3d_camera_link"/>
+       <child link="fixed_camera_link"/>
+   </joint>
+   <!-- we create a fixed link from arm_cam3d_camera_link to
+        arm_cam3d_camera_color_optical_frame. See commit: https://github.com/b-it-bots/mas_industrial_robotics/commit/f6e3bfa997b430278adbf4b552a285ce43e47936 -->
+        <!-- this also means you have to edit the source frame of the input
+             pointcloud before transforming it. see commit: https://github.com/b-it-bots/mas_industrial_robotics/commit/f4dd2f3124779fbedd28beb636e9ca7019baa9cf -->
+   <link name="fixed_camera_link">
+       <visual>
+           <geometry>
+               <box size="0.0000001 0.000001 0.000001"/>
+           </geometry>
+       </visual>
+       <collision>
+           <geometry>
+               <box size="0.0000001 0.000001 0.000001"/>
+           </geometry>
+       </collision>
+   </link>
 </robot>

Commit message: [urdf][gripper] Added a static grasp link

File: mir_common/mir_description/urdf/grippers/dynamixel/v2/dynamixel_gripper.urdf.xacro (robot description, xacro)
@@ -11,4 +11,5 @@
   <xacro:include filename="$(find mir_description)/urdf/grippers/dynamixel/v2/festo_finger_mount.urdf.xacro" />
   <xacro:include filename="$(find mcr_description)/urdf/fingers/festo_finger_dhas-gf-shm.urdf.xacro" />
+  <xacro:arg name="grasp_link_offset" default="0.11"/>
   <xacro:macro name="dynamixel_gripper_v2" params="parent name *origin">
     <joint name="${name}_motor_mount_joint" type="fixed" >
@@ -17,4 +18,11 @@
       <child link="${name}_motor_mount_link" />
     </joint>
+    <joint name="${name}_static_grasp_link_joint" type="fixed" >
+        <origin xyz="0 0 $(arg grasp_link_offset)" rpy="0 0 0"/>
+      <parent link="${parent}" />
+      <child link="${name}_static_grasp_link" />
+    </joint>
+    <link name="${name}_static_grasp_link">
+    </link>
     <!-- motor mount -->
     <link name="${name}_motor_mount_link">

Commit message: gripper controller changes

File: mir_common/mir_description/urdf/grippers/dynamixel/v2/dynamixel_gripper.urdf.xacro (robot description, xacro)
@@ -25,12 +25,5 @@
     <link name="${name}_static_grasp_link">
     </link>
-    <joint name="${name}_static_grasp_link_joint" type="fixed" >
-        <origin xyz="0 0 $(arg grasp_link_offset)" rpy="0 0 0"/>
-      <parent link="${parent}" />
-      <child link="${name}_static_grasp_link" />
-    </joint>
-    <link name="${name}_static_grasp_link">
-    </link>
-    <!-- motor mount -->
+        <!-- motor mount -->
     <link name="${name}_motor_mount_link">
       <inertial>

File: mir_robots/mir_hardware_config/youbot-brsu-2/urdf/robot.urdf.xacro (robot description, xacro)
@@ -40,9 +40,9 @@
   <!-- base laser front -->
   <xacro:hokuyo_urg04_laser name="base_laser_front" parent="base" ros_topic="scan_front" update_rate="10" min_angle="-1.57" max_angle="1.57">
-    <origin xyz="0.3 0 -0.035" rpy="0 0 0"/>
+    <origin xyz="0.3 0 -0.035" rpy="${M_PI} 0 0"/>
   </xacro:hokuyo_urg04_laser>
   <!-- base laser rear -->
   <xacro:hokuyo_urg04_laser name="base_laser_rear" parent="base" ros_topic="scan_rear" update_rate="10" min_angle="-1.57" max_angle="1.57" >
-     <origin xyz="-0.3 0.0 -0.035" rpy="0 0 ${M_PI}" />
+     <origin xyz="-0.3 0.0 -0.035" rpy="${M_PI} 0 ${M_PI}" />
   </xacro:hokuyo_urg04_laser>
   <xacro:dynamixel_gripper_v2 name="gripper" parent="arm_link_5">

Commit message: [urdf] updated gripper urdf to correct the mount position

File: mir_common/mir_description/urdf/grippers/dynamixel/v2/dynamixel_gripper.urdf.xacro (robot description, xacro)
@@ -28,16 +28,19 @@
     <link name="${name}_motor_mount_link">
       <inertial>
-        <origin xyz="0 0 0" rpy="0 0 0"/>
+        <origin xyz="-0.023 -0.046 0.024" rpy="0 0 0"/>
         <mass value="0.038"/>
         <inertia ixx="0.01" ixy="0" ixz="0" iyy="0.01" iyz="0" izz="0.01" />
       </inertial>
       <visual>
-        <origin xyz="0 0 0.0" rpy="0 ${M_PI/2} 0" />
+        <origin xyz="-0.023 -0.046 0.024" rpy="0 ${M_PI/2} 0" />
         <geometry>
           <mesh filename="package://mir_description/meshes/grippers/dynamixel/v3/dynamixel_intel_camera_combined.stl" scale="0.001 0.001 0.001" />
         </geometry>
+        <material name="">
+          <color rgba="0.85098 0.85098 0.85098 1"/>
+        </material>
       </visual>
       <collision>
-        <origin xyz="0 0 -0.0" rpy="0 ${M_PI/2} 0" />
+        <origin xyz="-0.023 -0.046 0.024" rpy="0 ${M_PI/2} 0" />
         <geometry>
           <mesh filename="package://mir_description/meshes/grippers/dynamixel/v2/dynamixel_motor_mount_convex_hull.dae" scale="0.001 0.001 0.001" />
