Commit message: [yb5] flip laser scanner upside-down

File: mir_robots/mir_hardware_config/youbot-brsu-5/urdf/robot.urdf.xacro (robot description, xacro)
@@ -39,9 +39,9 @@
   <!-- base laser front -->
   <xacro:hokuyo_urg04_laser name="base_laser_front" parent="base" ros_topic="scan_front" update_rate="10" min_angle="-1.57" max_angle="1.57">
-    <origin xyz="0.3 0 -0.03" rpy="0 0 0"/>
+    <origin xyz="0.3 0 -0.035" rpy="${M_PI} 0 0"/>
   </xacro:hokuyo_urg04_laser>
   <!-- base laser rear -->
   <xacro:hokuyo_urg04_laser name="base_laser_rear" parent="base" ros_topic="scan_rear" update_rate="10" min_angle="-1.57" max_angle="1.57" >
-     <origin xyz="-0.3 0.0 -0.03" rpy="0 0 ${M_PI}" />
+     <origin xyz="-0.3 0.0 -0.035" rpy="${M_PI} 0 ${M_PI}" />
   </xacro:hokuyo_urg04_laser>
   <!-- 3D camera on arm --> <!-- NOTE: still called arm_cam3d due to legacy code -->

Commit message: [description] correct arm height

File: mir_robots/mir_hardware_config/youbot-brsu-5/urdf/robot.urdf.xacro (robot description, xacro)
@@ -32,5 +32,5 @@
   <!-- Arm Plate moving arm 8cm foward and 45 degree rotation -->
   <xacro:adapter_plate name="adapter_plate" parent="base_link" arm_angle="${-M_PI / 4}">
-    <origin xyz="${0.159+0.08} 0 0.051" rpy="0 0 0" />
+    <origin xyz="${0.159+0.08} 0 ${0.021 + 0.025 + 0.025}" rpy="0 0 0" />    <!-- ${alignment with base top + spacer height + spacer height } -->
   </xacro:adapter_plate>
   <xacro:youbot_arm name="arm" parent="adapter_plate_arm_root_link">

Commit message: [description] add new rear platform

File: mir_robots/mir_hardware_config/youbot-brsu-5/urdf/robot.urdf.xacro (robot description, xacro)
@@ -11,5 +11,5 @@
   <!-- youbot base and rear platform -->
   <xacro:include filename="$(find youbot_description)/urdf/youbot_base/base.urdf.xacro" />
-  <xacro:include filename="$(find mir_description)/urdf/misc/rear_platform.urdf.xacro" />
+  <xacro:include filename="$(find mir_description)/urdf/misc/rear_platform_v2.urdf.xacro" />
   <!-- youbot arm and gripper-->
   <xacro:include filename="$(find youbot_description)/urdf/youbot_arm/arm.urdf.xacro"/>
@@ -27,7 +27,7 @@
   <xacro:youbot_base name="base"/>
   <!-- Rear Platform -->
-  <xacro:rear_platform name="rear_platform" parent="base_link">
-    <origin xyz="-0.005 -0.175 0.051" rpy="0 0 0" />
-  </xacro:rear_platform>
+  <xacro:rear_platform_v2 name="rear_platform" parent="base_link">
+    <origin xyz="0.12 -0.175 ${0.021 + 0.0062 + 0.025 + 0.012}" rpy="0 0 0" />  <!-- ${alignment with base top + nut height + spacer height + slide height } -->
+  </xacro:rear_platform_v2>
   <!-- Arm Plate moving arm 8cm foward and 45 degree rotation -->
   <xacro:adapter_plate name="adapter_plate" parent="base_link" arm_angle="${-M_PI / 4}">

Commit message: [description] start adding the v2 gripper parts

File: mir_robots/mir_hardware_config/youbot-brsu-5/urdf/robot.urdf.xacro (robot description, xacro)
@@ -15,5 +15,5 @@
   <xacro:include filename="$(find youbot_description)/urdf/youbot_arm/arm.urdf.xacro"/>
   <xacro:include filename="$(find mir_description)/urdf/misc/adapter_plate.urdf.xacro" />
-  <xacro:include filename="$(find mir_description)/urdf/grippers/dynamixel_gripper.urdf.xacro" />
+  <xacro:include filename="$(find mir_description)/urdf/grippers/dynamixel/v2/dynamixel_gripper.urdf.xacro" />
   <!-- controller manager -->
   <xacro:include filename="$(find youbot_description)/controller/ros_controller.urdf.xacro" />
@@ -49,6 +49,6 @@
     <origin xyz="-0.055 0.03 0.02" rpy="-0.09 ${-M_PI / 2 + 0.15} -0.05" />
   </xacro:realsense_camera>
-  <xacro:dynamixel_gripper name="gripper" parent="arm_link_5">
-    <origin xyz="0 0 -0.02" rpy="0 0 0" />
-  </xacro:dynamixel_gripper>
+  <xacro:dynamixel_gripper_v2 name="gripper" parent="arm_link_5">
+    <origin xyz="0.003 0 0.0052" rpy="0 0 0" />
+  </xacro:dynamixel_gripper_v2>
 </robot>

Commit message: [description] add intel camera + sensor mount to yb5

File: mir_robots/mir_hardware_config/youbot-brsu-5/urdf/robot.urdf.xacro (robot description, xacro)
@@ -22,5 +22,6 @@
   <!-- sensors -->
   <xacro:include filename="$(find youbot_description)/urdf/sensors/hokuyo_urg04_laser.urdf.xacro"/>
-  <xacro:include filename="$(find mcr_description)/urdf/sensors/realsense_camera.urdf.xacro"/>
+  <xacro:include filename="$(find mir_description)/urdf/sensor_mounts/intel_f200_camera_mount.urdf.xacro"/>
+  <xacro:include filename="$(find mcr_description)/urdf/sensors/intel_realsense_f200_camera.urdf.xacro"/>
   <!-- Now we can start using the macros included above to define the actual youbot -->
   <!-- standard youBot configuration -->
@@ -45,10 +46,14 @@
      <origin xyz="-0.3 0.0 -0.035" rpy="${M_PI} 0 ${M_PI}" />
   </xacro:hokuyo_urg04_laser>
-  <!-- 3D camera on arm --> <!-- NOTE: still called arm_cam3d due to legacy code -->
-  <xacro:realsense_camera name="arm_cam3d" parent="arm_link_5">
-    <origin xyz="-0.055 0.03 0.02" rpy="-0.09 ${-M_PI / 2 + 0.15} -0.05" />
-  </xacro:realsense_camera>
   <xacro:dynamixel_gripper_v2 name="gripper" parent="arm_link_5">
     <origin xyz="0.003 0 0.0052" rpy="0 0 0" />
   </xacro:dynamixel_gripper_v2>
+  <!-- camera mount for Intel RealSense F200 -->
+  <xacro:intel_f200_camera_mount name="camera_mount" parent="gripper_motor_mount_link">
+    <origin xyz="-0.00375 -0.0007 0.0002" rpy="0 0 0" />
+  </xacro:intel_f200_camera_mount>
+  <!-- 3D camera on arm -->
+  <xacro:intel_realsense_f200_camera name="tower_cam3d" parent="camera_mount_link">
+    <origin xyz="-0.0405 -0.074 0.029" rpy="0 -${M_PI/2} 0" />
+  </xacro:intel_realsense_f200_camera>
 </robot>

Commit message: [description] fix intel calibration

File: mir_robots/mir_hardware_config/youbot-brsu-5/urdf/robot.urdf.xacro (robot description, xacro)
@@ -55,5 +55,5 @@
   <!-- 3D camera on arm -->
   <xacro:intel_realsense_f200_camera name="arm_cam3d" parent="camera_mount_link">
-    <origin xyz="-0.0405 -0.074 0.029" rpy="0 -${M_PI/2} 0" />
+    <origin xyz="-0.0405 0.0 0.029" rpy="0 -${M_PI/2} 0" />
   </xacro:intel_realsense_f200_camera>
 </robot>
