Commit message: [description] fix path to mesh files

File: mir_common/mir_description/urdf/grippers/dynamixel/v1/dynamixel_gripper.urdf.xacro (robot description, xacro)
@@ -23,5 +23,5 @@
         <origin xyz="0 0 0" rpy="${M_PI/2} 0 ${M_PI}" />
         <geometry>
-          <mesh filename="package://mir_description/meshes/grippers/dynamixel_gripper_core_assembly.dae" scale="0.01 0.01 0.01" />
+          <mesh filename="package://mir_description/meshes/grippers/dynamixel/v1/dynamixel_gripper_core_assembly.dae" scale="0.01 0.01 0.01" />
         </geometry>
         <material name="White" />
@@ -30,5 +30,5 @@
         <origin xyz="0 0 0" rpy="${M_PI/2} 0 ${M_PI}" />
         <geometry>
-          <mesh filename="package://mir_description/meshes/grippers/dynamixel_gripper_core_assembly_convexhull.dae" scale="0.01 0.01 0.01" />
+          <mesh filename="package://mir_description/meshes/grippers/dynamixel/v1/dynamixel_gripper_core_assembly_convexhull.dae" scale="0.01 0.01 0.01" />
         </geometry>
       </collision>
@@ -117,5 +117,5 @@
         <origin xyz="-0.0125 0 0" rpy="0 0 ${-M_PI/2}" />
         <geometry>
-          <mesh filename="package://mir_description/meshes/grippers/dynamixel_small_finger_assembly_l.dae" scale="0.01 0.01 0.01" />
+          <mesh filename="package://mir_description/meshes/grippers/dynamixel/v1/dynamixel_small_finger_assembly_l.dae" scale="0.01 0.01 0.01" />
         </geometry>
         <material name="White" />
@@ -124,5 +124,5 @@
         <origin xyz="-0.0125 0 0" rpy="0 0 ${-M_PI/2}" />
         <geometry>
-          <mesh filename="package://mir_description/meshes/grippers/dynamixel_small_finger_assembly_l_convexhull.dae" scale="0.01 0.01 0.01" />
+          <mesh filename="package://mir_description/meshes/grippers/dynamixel/v1/dynamixel_small_finger_assembly_l_convexhull.dae" scale="0.01 0.01 0.01" />
         </geometry>
       </collision>
@@ -142,5 +142,5 @@
         <origin xyz="0.0125 0 0" rpy="0 0 ${M_PI/2}" />
         <geometry>
-          <mesh filename="package://mir_description/meshes/grippers/dynamixel_small_finger_assembly_r.dae" scale="0.01 0.01 0.01" />
+          <mesh filename="package://mir_description/meshes/grippers/dynamixel/v1/dynamixel_small_finger_assembly_r.dae" scale="0.01 0.01 0.01" />
         </geometry>
         <material name="White" />
@@ -149,5 +149,5 @@
         <origin xyz="0.0125 0 0" rpy="0 0 ${M_PI/2}" />
         <geometry>
-          <mesh filename="package://mir_description/meshes/grippers/dynamixel_small_finger_assembly_r_convexhull.dae" scale="0.01 0.01 0.01" />
+          <mesh filename="package://mir_description/meshes/grippers/dynamixel/v1/dynamixel_small_finger_assembly_r_convexhull.dae" scale="0.01 0.01 0.01" />
         </geometry>
       </collision>
