Commit message: fixed xacro syntax and added joint_state_publisher node in launch file in order to get tf

File: mir_calibration/mir_calibration_data/youbot-brsu-1/calibration.urdf.xacro (robot description, xacro)
@@ -2,16 +2,16 @@
 <robot>
   <!-- Pose of PMD (arm_cam3d) relative to ? -->
-  <property name="cal_arm_cam3d_x" value="0.0"/>
-  <property name="cal_arm_cam3d_y" value="-0.025"/>
-  <property name="cal_arm_cam3d_z" value="-0.015"/>
-  <property name="cal_arm_cam3d_roll" value="0.0"/>
-  <property name="cal_arm_cam3d_pitch" value="${-M_PI}"/>
-  <property name="cal_arm_cam3d_yaw" value="0.0"/>
+  <xacro:property name="cal_arm_cam3d_x" value="0.0"/>
+  <xacro:property name="cal_arm_cam3d_y" value="-0.025"/>
+  <xacro:property name="cal_arm_cam3d_z" value="-0.015"/>
+  <xacro:property name="cal_arm_cam3d_roll" value="0.0"/>
+  <xacro:property name="cal_arm_cam3d_pitch" value="${-M_PI}"/>
+  <xacro:property name="cal_arm_cam3d_yaw" value="0.0"/>
    <!-- Pose of Kinect (arm_cam3d) relative to tower_link -->
-  <property name="cal_arm_cam3d_x" value="0.097"/>
-  <property name="cal_arm_cam3d_y" value="-0.001"/>
-  <property name="cal_arm_cam3d_z" value="0.469"/>
-  <property name="cal_arm_cam3d_roll" value="0.037"/>
-  <property name="cal_arm_cam3d_pitch" value="0.329"/>
-  <property name="cal_arm_cam3d_yaw" value="-0.028"/>
+  <xacro:property name="cal_arm_cam3d_x" value="0.097"/>
+  <xacro:property name="cal_arm_cam3d_y" value="-0.001"/>
+  <xacro:property name="cal_arm_cam3d_z" value="0.469"/>
+  <xacro:property name="cal_arm_cam3d_roll" value="0.037"/>
+  <xacro:property name="cal_arm_cam3d_pitch" value="0.329"/>
+  <xacro:property name="cal_arm_cam3d_yaw" value="-0.028"/>
 </robot>

File: mir_common/mir_description/urdf/grippers/dynamixel/v1/dynamixel_gripper.gazebo.xacro (robot description, xacro)
@@ -3,5 +3,5 @@
        xmlns:controller="http://playerstage.sourceforge.net/gazebo/xmlschema/#controller"
        xmlns:interface="http://playerstage.sourceforge.net/gazebo/xmlschema/#interface"
-       xmlns:xacro="http://ros.org/wiki/xacro">
+       xmlns:xacro="http://www.ros.org/wiki/xacro">
 	<xacro:macro name="dynamixel_gripper_gazebo" params="name">
 		<gazebo reference="${name}_palm_link">

File: mir_common/mir_description/urdf/grippers/dynamixel/v1/dynamixel_gripper.transmission.xacro (robot description, xacro)
@@ -3,5 +3,5 @@
        xmlns:controller="http://playerstage.sourceforge.net/gazebo/xmlschema/#controller"
        xmlns:interface="http://playerstage.sourceforge.net/gazebo/xmlschema/#interface"
-       xmlns:xacro="http://ros.org/wiki/xacro">
+       xmlns:xacro="http://www.ros.org/wiki/xacro">
   <xacro:macro name="dynamixel_gripper_transmission" params="name">
   <transmission name="${name}_finger_l_trans">

File: mir_common/mir_description/urdf/grippers/dynamixel/v1/dynamixel_gripper.urdf.xacro (robot description, xacro)
@@ -3,5 +3,5 @@
        xmlns:controller="http://playerstage.sourceforge.net/gazebo/xmlschema/#controller"
        xmlns:interface="http://playerstage.sourceforge.net/gazebo/xmlschema/#interface"
-       xmlns:xacro="http://ros.org/wiki/xacro">
+       xmlns:xacro="http://www.ros.org/wiki/xacro">
   <xacro:include filename="$(find mir_description)/urdf/grippers/dynamixel/v1/dynamixel_gripper.gazebo.xacro" />
   <xacro:include filename="$(find mir_description)/urdf/grippers/dynamixel/v1/dynamixel_gripper.transmission.xacro" />
@@ -10,5 +10,5 @@
     <!-- joint between arm_5_link and dynamixel_palm_link -->
     <joint name="${name}_palm_joint" type="fixed" >
-      <insert_block name="origin" />
+      <xacro:insert_block name="origin" />
       <parent link="${parent}" />
       <child link="${name}_palm_link" />

File: mir_common/mir_description/urdf/grippers/dynamixel/v1/dynamixel_limits.urdf.xacro (robot description, xacro)
@@ -2,7 +2,7 @@
 <robot>
   <!-- common properties -->
-  <property name="M_PI" value="3.1415926535897931" />
+  <xacro:property name="M_PI" value="3.1415926535897931" />
   <!-- fingers limits, values are in meters -->
-  <property name="dynamixel_joint_min" value="0.0" />
-  <property name="dynamixel_joint_max" value="2.17" />
+  <xacro:property name="dynamixel_joint_min" value="0.0" />
+  <xacro:property name="dynamixel_joint_max" value="2.17" />
 </robot>

File: mir_common/mir_description/urdf/grippers/dynamixel/v2/dynamixel_gripper.urdf.xacro (robot description, xacro)
@@ -3,5 +3,5 @@
        xmlns:controller="http://playerstage.sourceforge.net/gazebo/xmlschema/#controller"
        xmlns:interface="http://playerstage.sourceforge.net/gazebo/xmlschema/#interface"
-       xmlns:xacro="http://ros.org/wiki/xacro">
+       xmlns:xacro="http://www.ros.org/wiki/xacro">
   <!--xacro:include filename="$(find mir_description)/urdf/grippers/dynamixel/v2/dynamixel_gripper.gazebo.xacro" /-->
   <!--xacro:include filename="$(find mir_description)/urdf/grippers/dynamixel/v2/dynamixel_gripper.transmission.xacro" /-->
@@ -13,5 +13,5 @@
   <xacro:macro name="dynamixel_gripper_v2" params="parent name *origin">
     <joint name="${name}_motor_mount_joint" type="fixed" >
-      <insert_block name="origin" />
+      <xacro:insert_block name="origin" />
       <parent link="${parent}" />
       <child link="${name}_motor_mount_link" />

File: mir_common/mir_description/urdf/grippers/dynamixel/v2/festo_finger_mount.urdf.xacro (robot description, xacro)
@@ -3,8 +3,8 @@
        xmlns:controller="http://playerstage.sourceforge.net/gazebo/xmlschema/#controller"
        xmlns:interface="http://playerstage.sourceforge.net/gazebo/xmlschema/#interface"
-       xmlns:xacro="http://ros.org/wiki/xacro">
+       xmlns:xacro="http://www.ros.org/wiki/xacro">
   <xacro:macro name="festo_finger_mount" params="parent name *origin">
     <joint name="${name}_joint" type="fixed" >
-      <insert_block name="origin" />
+      <xacro:insert_block name="origin" />
       <parent link="${parent}" />
       <child link="${name}_link" />

File: mir_common/mir_description/urdf/grippers/festo_gripper.urdf.xacro (robot description, xacro)
@@ -3,10 +3,10 @@
        xmlns:controller="http://playerstage.sourceforge.net/gazebo/xmlschema/#controller"
        xmlns:interface="http://playerstage.sourceforge.net/gazebo/xmlschema/#interface"
-       xmlns:xacro="http://ros.org/wiki/xacro">
+       xmlns:xacro="http://www.ros.org/wiki/xacro">
     <xacro:include filename="$(find youbot_description)/urdf/youbot_gripper/gripper.transmission.xacro" />
     <xacro:include filename="$(find youbot_description)/urdf/youbot_gripper/limits.urdf.xacro" />
     <xacro:macro name="festo_gripper" params="parent name *origin">
         <joint name="${name}_palm_joint" type="fixed" >
-            <insert_block name="origin" />
+            <xacro:insert_block name="origin" />
             <parent link="${parent}" />
             <child link="${name}_palm_link" />

File: mir_common/mir_description/urdf/misc/adapter_plate.urdf.xacro (robot description, xacro)
@@ -3,9 +3,9 @@
        xmlns:controller="http://playerstage.sourceforge.net/gazebo/xmlschema/#controller"
        xmlns:interface="http://playerstage.sourceforge.net/gazebo/xmlschema/#interface"
-       xmlns:xacro="http://ros.org/wiki/xacro">
+       xmlns:xacro="http://www.ros.org/wiki/xacro">
 	<xacro:macro name="adapter_plate" params="parent name arm_angle *origin">
 		<!-- joint between arm_7_link and sdh_palm_link -->
 		<joint name="${name}_joint" type="fixed" >
-			<insert_block name="origin" />
+			<xacro:insert_block name="origin" />
 			<parent link="${parent}" />
 			<child link="${name}_link" />

File: mir_common/mir_description/urdf/misc/cam3d_tower.urdf.xacro (robot description, xacro)
@@ -3,9 +3,9 @@
        xmlns:controller="http://playerstage.sourceforge.net/gazebo/xmlschema/#controller"
        xmlns:interface="http://playerstage.sourceforge.net/gazebo/xmlschema/#interface"
-       xmlns:xacro="http://ros.org/wiki/xacro">
-  <property name="cam3d_tower_height" value="0.49" />
-  <property name="cam3d_tower_width" value="0.03" />
-  <property name="cam3d_tower_depth" value="0.03" />
-  <property name="cam3d_tower_collision_offset" value="0.03" />
+       xmlns:xacro="http://www.ros.org/wiki/xacro">
+  <xacro:property name="cam3d_tower_height" value="0.49" />
+  <xacro:property name="cam3d_tower_width" value="0.03" />
+  <xacro:property name="cam3d_tower_depth" value="0.03" />
+  <xacro:property name="cam3d_tower_collision_offset" value="0.03" />
   <xacro:macro name="cam3d_tower" params="name parent *origin">
   	<link name="${name}_link">
@@ -30,5 +30,5 @@
     </link>
     <joint name="${name}_joint" type="fixed">
-      <insert_block name="origin" />
+      <xacro:insert_block name="origin" />
       <parent link="${parent}"/>
       <child link="${name}_link"/>

File: mir_common/mir_description/urdf/misc/distance_screw.urdf.xacro (robot description, xacro)
@@ -3,5 +3,5 @@
        xmlns:controller="http://playerstage.sourceforge.net/gazebo/xmlschema/#controller"
        xmlns:interface="http://playerstage.sourceforge.net/gazebo/xmlschema/#interface"
-       xmlns:xacro="http://ros.org/wiki/xacro">
+       xmlns:xacro="http://www.ros.org/wiki/xacro">
 	<xacro:macro name="distance_screw" params="name parent *origin">
 		<link name="${name}_link">
@@ -26,5 +26,5 @@
 		</link>
 		<joint name="${name}_part1_joint" type="fixed">
-			<insert_block name="origin" />
+			<xacro:insert_block name="origin" />
 			<parent link="${parent}"/>
 			<child link="${name}_link"/>

File: mir_common/mir_description/urdf/misc/laptop_case_frame.urdf.xacro (robot description, xacro)
@@ -3,8 +3,8 @@
        xmlns:controller="http://playerstage.sourceforge.net/gazebo/xmlschema/#controller"
        xmlns:interface="http://playerstage.sourceforge.net/gazebo/xmlschema/#interface"
-       xmlns:xacro="http://ros.org/wiki/xacro">
-	<property name="laptop_case_frame_width"  value="0.25" />
-	<property name="laptop_case_frame_height" value="0.005" />
-	<property name="laptop_case_frame_depth"  value="0.03" />
+       xmlns:xacro="http://www.ros.org/wiki/xacro">
+	<xacro:property name="laptop_case_frame_width"  value="0.25" />
+	<xacro:property name="laptop_case_frame_height" value="0.005" />
+	<xacro:property name="laptop_case_frame_depth"  value="0.03" />
 	<xacro:macro name="laptop_case_frame" params="name parent *origin">
 		<link name="${name}_bottom_link">
@@ -29,5 +29,5 @@
 		</link>
 		<joint name="${name}_bottom_joint" type="fixed">
-			<insert_block name="origin" />
+			<xacro:insert_block name="origin" />
 			<parent link="${parent}"/>
 			<child link="${name}_bottom_link"/>

File: mir_common/mir_description/urdf/misc/plugbar.xacro (robot description, xacro)
@@ -3,8 +3,8 @@
        xmlns:controller="http://playerstage.sourceforge.net/gazebo/xmlschema/#controller"
        xmlns:interface="http://playerstage.sourceforge.net/gazebo/xmlschema/#interface"
-       xmlns:xacro="http://ros.org/wiki/xacro">
+       xmlns:xacro="http://www.ros.org/wiki/xacro">
 	<xacro:macro name="plugbar" params="parent name *origin">
 		<joint name="${name}_joint" type="fixed" >
-			<insert_block name="origin" />
+			<xacro:insert_block name="origin" />
 			<parent link="${parent}" />
 			<child link="${name}_link" />

File: mir_common/mir_description/urdf/misc/rear_platform.urdf.xacro (robot description, xacro)
@@ -3,8 +3,8 @@
        xmlns:controller="http://playerstage.sourceforge.net/gazebo/xmlschema/#controller"
        xmlns:interface="http://playerstage.sourceforge.net/gazebo/xmlschema/#interface"
-       xmlns:xacro="http://ros.org/wiki/xacro">
+       xmlns:xacro="http://www.ros.org/wiki/xacro">
 	<xacro:macro name="rear_platform" params="parent name *origin">
 		<joint name="${name}_joint" type="fixed" >
-			<insert_block name="origin" />
+			<xacro:insert_block name="origin" />
 			<parent link="${parent}" />
 			<child link="${name}_link" />

File: mir_common/mir_description/urdf/misc/rear_platform_v2.urdf.xacro (robot description, xacro)
@@ -3,9 +3,9 @@
        xmlns:controller="http://playerstage.sourceforge.net/gazebo/xmlschema/#controller"
        xmlns:interface="http://playerstage.sourceforge.net/gazebo/xmlschema/#interface"
-       xmlns:xacro="http://ros.org/wiki/xacro">
+       xmlns:xacro="http://www.ros.org/wiki/xacro">
 	<xacro:macro name="rear_platform_v2" params="parent name *origin">
         <!-- base plate -->
 		<joint name="${name}_base_joint" type="fixed" >
-			<insert_block name="origin" />
+			<xacro:insert_block name="origin" />
 			<parent link="${parent}" />
 			<child link="${name}_base_link" />

File: mir_common/mir_description/urdf/misc/sensor_angle.urdf.xacro (robot description, xacro)
@@ -3,8 +3,8 @@
        xmlns:controller="http://playerstage.sourceforge.net/gazebo/xmlschema/#controller"
        xmlns:interface="http://playerstage.sourceforge.net/gazebo/xmlschema/#interface"
-       xmlns:xacro="http://ros.org/wiki/xacro">
-	<property name="sensor_angle_width"  value="0.097" />
-	<property name="sensor_angle_height" value="0.0015" />
-	<property name="sensor_angle_depth"  value="0.0625" />
+       xmlns:xacro="http://www.ros.org/wiki/xacro">
+	<xacro:property name="sensor_angle_width"  value="0.097" />
+	<xacro:property name="sensor_angle_height" value="0.0015" />
+	<xacro:property name="sensor_angle_depth"  value="0.0625" />
 	<xacro:macro name="sensor_angle" params="name parent *origin">
 		<link name="${name}_part1_link">
@@ -29,5 +29,5 @@
 		</link>
 		<joint name="${name}_part1_joint" type="fixed">
-			<insert_block name="origin" />
+			<xacro:insert_block name="origin" />
 			<parent link="${parent}"/>
 			<child link="${name}_part1_link"/>

File: mir_common/mir_description/urdf/misc/sensor_angle_shortend.urdf.xacro (robot description, xacro)
@@ -3,8 +3,8 @@
        xmlns:controller="http://playerstage.sourceforge.net/gazebo/xmlschema/#controller"
        xmlns:interface="http://playerstage.sourceforge.net/gazebo/xmlschema/#interface"
-       xmlns:xacro="http://ros.org/wiki/xacro">
-	<property name="sensor_angle_width"  value="0.097" />
-	<property name="sensor_angle_height" value="0.0015" />
-	<property name="sensor_angle_depth"  value="0.04" />
+       xmlns:xacro="http://www.ros.org/wiki/xacro">
+	<xacro:property name="sensor_angle_width"  value="0.097" />
+	<xacro:property name="sensor_angle_height" value="0.0015" />
+	<xacro:property name="sensor_angle_depth"  value="0.04" />
 	<xacro:macro name="sensor_angle_shortend" params="name parent *origin">
 		<link name="${name}_part1_link">
@@ -29,5 +29,5 @@
 		</link>
 		<joint name="${name}_part1_joint" type="fixed">
-			<insert_block name="origin" />
+			<xacro:insert_block name="origin" />
 			<parent link="${parent}"/>
 			<child link="${name}_part1_link"/>

File: mir_common/mir_description/urdf/sensor_mounts/intel_f200_camera_mount.urdf.xacro (robot description, xacro)
@@ -3,8 +3,8 @@
        xmlns:controller="http://playerstage.sourceforge.net/gazebo/xmlschema/#controller"
        xmlns:interface="http://playerstage.sourceforge.net/gazebo/xmlschema/#interface"
-       xmlns:xacro="http://ros.org/wiki/xacro">
+       xmlns:xacro="http://www.ros.org/wiki/xacro">
 	<xacro:macro name="intel_f200_camera_mount" params="parent name *origin">
 		<joint name="${name}_joint" type="fixed" >
-			<insert_block name="origin" />
+			<xacro:insert_block name="origin" />
 			<parent link="${parent}" />
 			<child link="${name}_link" />

File: mir_robots/mir_hardware_config/youbot-brsu-1/urdf/robot.urdf.xacro (robot description, xacro)
@@ -3,5 +3,5 @@
        xmlns:controller="http://playerstage.sourceforge.net/gazebo/xmlschema/#controller"
        xmlns:interface="http://playerstage.sourceforge.net/gazebo/xmlschema/#interface"
-       xmlns:xacro="http://playerstage.sourceforge.net/gazebo/xmlschema/#interface"
+       xmlns:xacro="http://www.ros.org/wiki/xacro"
        name="youbot" >
   <!-- The following included files set up definitions of parts of the robot body -->

File: mir_robots/mir_hardware_config/youbot-brsu-2/urdf/robot.urdf.xacro (robot description, xacro)
@@ -3,5 +3,5 @@
        xmlns:controller="http://playerstage.sourceforge.net/gazebo/xmlschema/#controller"
        xmlns:interface="http://playerstage.sourceforge.net/gazebo/xmlschema/#interface"
-       xmlns:xacro="http://playerstage.sourceforge.net/gazebo/xmlschema/#interface"
+       xmlns:xacro="http://www.ros.org/wiki/xacro"
        name="youbot" >
   <!-- The following included files set up definitions of parts of the robot body -->
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