Commit message: make youbot-brsu-1 the same config as youbot-brsu-3

File: mir_robots/mir_hardware_config/youbot-brsu-1/urdf/robot.urdf.xacro (robot description, xacro)
@@ -30,6 +30,9 @@
   <!-- foot for arm-->
   <xacro:youbot_base name="base"/>
- <xacro:youbot_arm name="arm" parent="base_link">
-    <origin xyz="0.223 0.003 0.084" rpy="0 0 0" />
+  <xacro:youbot_plate name="plate" parent="base_link">
+    <origin xyz="-0.159 0 0.046" rpy="0 0 0" />
+  </xacro:youbot_plate>
+  <xacro:youbot_arm name="arm" parent="base_link">
+    <origin xyz="0.143 0 0.046" rpy="0 0 0" />
   </xacro:youbot_arm>
   <xacro:youbot_gripper name="gripper" parent="arm_link_5">
@@ -37,77 +40,9 @@
   </xacro:youbot_gripper>
   <!-- BRSU SPECIFIC STUFF -->
-  <xacro:include filename="$(find mir_calibration_data)/youbot-brsu-1/calibration.urdf.xacro" />
-  <xacro:include filename="$(find mir_description)/urdf/misc/sensor_angle_shortend.urdf.xacro" />
-  <xacro:include filename="$(find mir_description)/urdf/misc/cam3d_tower.urdf.xacro" />
-  <xacro:include filename="$(find mir_description)/urdf/sensors/kinect_camera.urdf.xacro" />
-  <!--<xacro:include filename="$(find mir_description)/urdf/sensors/pmd_camboard_nano_camera.urdf.xacro" />-->
-  <xacro:include filename="$(find mir_description)/urdf/misc/laptop_case_frame.urdf.xacro" />
-  <xacro:include filename="$(find mir_description)/urdf/misc/distance_screw.urdf.xacro" />
-  <xacro:include filename="$(find mir_description)/urdf/misc/brsu_front_plate.urdf.xacro" />
-  <xacro:include filename="$(find mir_description)/urdf/misc/brsu_rear_plate.urdf.xacro" />
-  <!-- brsu specific platforms -->
   <xacro:include filename="$(find mcr_description)/urdf/materials.urdf.xacro" />
-  <xacro:brsu_rear_plate name="plate" parent="base_link">
-    <origin xyz="-0.009 -0.175 0.100" rpy="0 0 0" />
-  </xacro:brsu_rear_plate>
-  <xacro:brsu_front_plate name="plate_front" parent="base_link">
-    <origin xyz="0.340 -0.175 0.049" rpy="0 0 0" />
-  </xacro:brsu_front_plate>
-  <!-- base laser rear -->
+  <!-- base laser rear
   <xacro:hokuyo_urg04_laser name="base_laser_rear" parent="base" ros_topic="scan_rear" update_rate="10" min_angle="-1.57" max_angle="1.57" >
-     <origin xyz="-0.3 0.0 -0.03" rpy="0 0 ${M_PI}" />
+     <origin xyz="-0.3 0 -0.03" rpy="0 0 ${M_PI}" />
   </xacro:hokuyo_urg04_laser>
-  <!-- distance screws -->
-  <xacro:distance_screw name="distance_screw_fl" parent="base_link">
-    <origin xyz="-0.11 0.075 0.035" rpy="0 0 0" />
-  </xacro:distance_screw>
-  <xacro:distance_screw name="distance_screw_fr" parent="base_link">
-    <origin xyz="-0.11 -0.075 0.035" rpy="0 0 0" />
-  </xacro:distance_screw>
-  <xacro:distance_screw name="distance_screw_rl" parent="base_link">
-    <origin xyz="-0.20 0.075 0.035" rpy="0 0 0" />
-  </xacro:distance_screw>
-  <xacro:distance_screw name="distance_screw_rr" parent="base_link">
-    <origin xyz="-0.20 -0.075 0.035" rpy="0 0 0" />
-  </xacro:distance_screw>
-<!-- distance screws front -->
-  <xacro:distance_screw name="front_distance_screw_fl" parent="base_link">
-    <origin xyz="0.088 0.055 0.035" rpy="0 0 0" />
-  </xacro:distance_screw>
-  <xacro:distance_screw name="front_distance_screw_fr" parent="base_link">
-    <origin xyz="0.088 -0.055 0.035" rpy="0 0 0" />
-  </xacro:distance_screw>
-  <xacro:distance_screw name="front_distance_screw_rl" parent="base_link">
-    <origin xyz="0.228 0.055 0.035" rpy="0 0 0" />
-  </xacro:distance_screw>
-  <xacro:distance_screw name="front_distance_screw_rr" parent="base_link">
-    <origin xyz="0.228 -0.055 0.035" rpy="0 0 0" />
-  </xacro:distance_screw>
-  <!-- laptop case frame -->
-  <xacro:laptop_case_frame name="laptop_case_frame_left" parent="base_link">
-    <origin xyz="-0.15 0.075 0.05" rpy="0 0 ${-M_PI/2}" />
-  </xacro:laptop_case_frame>
-  <xacro:laptop_case_frame name="laptop_case_frame_right" parent="base_link">
-    <origin xyz="-0.15 -0.075 0.05" rpy="0 0 ${M_PI/2}" />
-  </xacro:laptop_case_frame>
-  <!-- Sensor angle on arm -->
-  <xacro:sensor_angle_shortend name="arm_sensor_angle_shortend" parent="arm_link_5">
-    <origin xyz="0.015 0.0 -0.023" rpy="0.0 0.0 ${M_PI}" />
-  </xacro:sensor_angle_shortend>
-  <!-- pmd on arm -->
-  <!--<xacro:pmd_camboard_nano_camera name="arm_cam3d" parent="arm_sensor_angle_shortend_part2_link">-->
-    <!--<origin xyz="${cal_arm_cam3d_x} ${cal_arm_cam3d_y} ${cal_arm_cam3d_z}" rpy="${cal_arm_cam3d_roll} ${cal_arm_cam3d_pitch} ${cal_arm_cam3d_yaw}" />-->
-  <!--</xacro:pmd_camboard_nano_camera> -->
-  <!-- tower -->
-  <!--<xacro:cam3d_tower name="tower" parent="plate_link">
-    <origin xyz="-0.0659 0.0 0.025" rpy="0 0 0" />
-  </xacro:cam3d_tower>
--->
-  <xacro:cam3d_tower name="tower" parent="plate_link">
-    <origin xyz="-0.245 0.175 0.0" rpy="0 0 0" />
-  </xacro:cam3d_tower>
-  <!-- 3D camera on tower -->
-  <xacro:kinect_camera name="tower_cam3d" parent="tower_link">
-    <origin xyz="${cal_tower_cam3d_x} ${cal_tower_cam3d_y} ${cal_tower_cam3d_z}" rpy="${cal_tower_cam3d_roll} ${cal_tower_cam3d_pitch} ${cal_tower_cam3d_yaw}" />
-  </xacro:kinect_camera>
+  -->
 </robot>

Commit message: add front laser scanner

File: mir_robots/mir_hardware_config/youbot-brsu-1/urdf/robot.urdf.xacro (robot description, xacro)
@@ -20,4 +20,6 @@
   <!-- materials for visualization -->
   <xacro:include filename="$(find youbot_description)/urdf/materials.urdf.xacro" />
+  <!-- sensors -->
+  <xacro:include filename="$(find youbot_description)/urdf/sensors/hokuyo_urg04_laser.urdf.xacro"/>
   <!-- Now we can start using the macros included above to define the actual youbot -->
   <!-- The first use of a macro.  This one was defined in base.urdf.xacro above.
@@ -41,4 +43,8 @@
   <!-- BRSU SPECIFIC STUFF -->
   <xacro:include filename="$(find mcr_description)/urdf/materials.urdf.xacro" />
+  <!-- base laser front -->
+  <xacro:hokuyo_urg04_laser name="base_laser_front" parent="base" ros_topic="scan_front" update_rate="10" min_angle="-1.57" max_angle="1.57">
+    <origin xyz="0.3 0 -0.03" rpy="0 0 0"/>
+  </xacro:hokuyo_urg04_laser>
   <!-- base laser rear
   <xacro:hokuyo_urg04_laser name="base_laser_rear" parent="base" ros_topic="scan_rear" update_rate="10" min_angle="-1.57" max_angle="1.57" >

File: mir_robots/mir_hardware_config/youbot-brsu-2/urdf/robot.urdf.xacro (robot description, xacro)
@@ -10,4 +10,6 @@
   <!-- youbot base -->
   <xacro:include filename="$(find youbot_description)/urdf/youbot_base/base.urdf.xacro" />
+  <!-- youbot plate -->
+  <xacro:include filename="$(find youbot_description)/urdf/youbot_plate/plate.urdf.xacro" />
   <!-- youbot arm -->
   <xacro:include filename="$(find youbot_description)/urdf/youbot_arm/arm.urdf.xacro"/>
@@ -18,4 +20,6 @@
   <!-- materials for visualization -->
   <xacro:include filename="$(find youbot_description)/urdf/materials.urdf.xacro" />
+  <!-- sensors -->
+  <xacro:include filename="$(find youbot_description)/urdf/sensors/hokuyo_urg04_laser.urdf.xacro"/>
   <!-- Now we can start using the macros included above to define the actual youbot -->
   <!-- The first use of a macro.  This one was defined in base.urdf.xacro above.
@@ -28,6 +32,9 @@
   <!-- foot for arm-->
   <xacro:youbot_base name="base"/>
+  <xacro:youbot_plate name="plate" parent="base_link">
+    <origin xyz="-0.159 0 0.046" rpy="0 0 0" />
+  </xacro:youbot_plate>
   <xacro:youbot_arm name="arm" parent="base_link">
-    <origin xyz="0.223 0.003 0.084" rpy="0 0 0" />
+    <origin xyz="0.143 0 0.046" rpy="0 0 0" />
   </xacro:youbot_arm>
   <xacro:youbot_gripper name="gripper" parent="arm_link_5">
@@ -36,5 +43,5 @@
   <!-- BRSU SPECIFIC STUFF -->
   <xacro:include filename="$(find mcr_description)/urdf/materials.urdf.xacro" />
-  <xacro:include filename="$(find mcr_description)/urdf/sensors/kinect_camera.urdf.xacro" />
+  <!--xacro:include filename="$(find mcr_description)/urdf/sensors/kinect_camera.urdf.xacro" />
   <xacro:include filename="$(find mcr_description)/urdf/sensors/pmd_camboard_nano_camera.urdf.xacro" />
   <xacro:include filename="$(find mir_calibration_data)/youbot-brsu-2/calibration.urdf.xacro" />
@@ -44,6 +51,10 @@
   <xacro:include filename="$(find mir_description)/urdf/misc/distance_screw.urdf.xacro" />
   <xacro:include filename="$(find mir_description)/urdf/misc/adapter_plate.urdf.xacro" />
-  <xacro:include filename="$(find mir_description)/urdf/misc/rear_platform.urdf.xacro" />
-  <!-- brsu specific platforms -->
+  <xacro:include filename="$(find mir_description)/urdf/misc/rear_platform.urdf.xacro" /-->
+  <!-- base laser front -->
+  <xacro:hokuyo_urg04_laser name="base_laser_front" parent="base" ros_topic="scan_front" update_rate="10" min_angle="-1.57" max_angle="1.57">
+    <origin xyz="0.3 0 -0.03" rpy="0 0 0"/>
+  </xacro:hokuyo_urg04_laser>
+  <!-- brsu specific platforms
   <xacro:rear_platform name="rear_platform" parent="base_link">
     <origin xyz="-0.029 -0.175 0.100" rpy="0 0 0" />
@@ -51,10 +62,10 @@
   <xacro:adapter_plate name="front_plate" parent="base_link">
     <origin xyz="0.340 -0.175 0.049" rpy="0 0 0" />
-  </xacro:adapter_plate>
+  </xacro:adapter_plate-->
   <!-- base laser rear -->
   <xacro:hokuyo_urg04_laser name="base_laser_rear" parent="base" ros_topic="scan_rear" update_rate="10" min_angle="-1.57" max_angle="1.57" >
      <origin xyz="-0.3 0.0 -0.03" rpy="0 0 ${M_PI}" />
   </xacro:hokuyo_urg04_laser>
-  <!-- distance screws -->
+  <!-- distance screws
   <xacro:distance_screw name="distance_screw_fl" parent="base_link">
     <origin xyz="-0.11 0.075 0.035" rpy="0 0 0" />
@@ -68,6 +79,6 @@
   <xacro:distance_screw name="distance_screw_rr" parent="base_link">
     <origin xyz="-0.20 -0.075 0.035" rpy="0 0 0" />
-  </xacro:distance_screw>
-<!-- distance screws front -->
+  </xacro:distance_screw-->
+  <!-- distance screws front
   <xacro:distance_screw name="front_distance_screw_fl" parent="base_link">
     <origin xyz="0.088 0.055 0.035" rpy="0 0 0" />
@@ -81,6 +92,6 @@
   <xacro:distance_screw name="front_distance_screw_rr" parent="base_link">
     <origin xyz="0.228 -0.055 0.035" rpy="0 0 0" />
-  </xacro:distance_screw>
-  <!-- laptop case frame -->
+  </xacro:distance_screw-->
+  <!-- laptop case frame
   <xacro:laptop_case_frame name="laptop_case_frame_left" parent="base_link">
     <origin xyz="-0.15 0.075 0.05" rpy="0 0 ${-M_PI/2}" />
@@ -88,10 +99,10 @@
   <xacro:laptop_case_frame name="laptop_case_frame_right" parent="base_link">
     <origin xyz="-0.15 -0.075 0.05" rpy="0 0 ${M_PI/2}" />
-  </xacro:laptop_case_frame>
-  <!-- Sensor angle on arm -->
+  </xacro:laptop_case_frame-->
+  <!-- Sensor angle on arm
   <xacro:sensor_angle_shortend name="arm_sensor_angle_shortend" parent="arm_link_5">
     <origin xyz="0.015 0.0 -0.023" rpy="0.0 0.0 ${M_PI}" />
-  </xacro:sensor_angle_shortend>
-  <!-- pmd on arm -->
+  </xacro:sensor_angle_shortend-->
+  <!-- pmd on arm
   <xacro:pmd_camboard_nano_camera name="arm_cam3d" parent="arm_sensor_angle_shortend_part2_link">
     <origin xyz="${cal_arm_cam3d_x} ${cal_arm_cam3d_y} ${cal_arm_cam3d_z}" rpy="${cal_arm_cam3d_roll} ${cal_arm_cam3d_pitch} ${cal_arm_cam3d_yaw}" />
@@ -99,8 +110,8 @@
   <xacro:cam3d_tower name="tower" parent="rear_platform_link">
     <origin xyz="-0.245 0.175 0.0" rpy="0 0 0" />
-  </xacro:cam3d_tower>
-  <!-- 3D camera on tower -->
+  </xacro:cam3d_tower-->
+  <!-- 3D camera on tower
   <xacro:kinect_camera name="tower_cam3d" parent="tower_link">
     <origin xyz="${cal_tower_cam3d_x} ${cal_tower_cam3d_y} ${cal_tower_cam3d_z}" rpy="${cal_tower_cam3d_roll} ${cal_tower_cam3d_pitch} ${cal_tower_cam3d_yaw}" />
-  </xacro:kinect_camera>
+  </xacro:kinect_camera-->
 </robot>

File: mir_robots/mir_hardware_config/youbot-brsu-3/urdf/robot.urdf.xacro (robot description, xacro)
@@ -20,4 +20,6 @@
   <!-- materials for visualization -->
   <xacro:include filename="$(find youbot_description)/urdf/materials.urdf.xacro" />
+  <!-- sensors -->
+  <xacro:include filename="$(find youbot_description)/urdf/sensors/hokuyo_urg04_laser.urdf.xacro"/>
   <!-- Now we can start using the macros included above to define the actual youbot -->
   <!-- The first use of a macro.  This one was defined in base.urdf.xacro above.
@@ -41,4 +43,8 @@
   <!-- BRSU SPECIFIC STUFF -->
   <xacro:include filename="$(find mcr_description)/urdf/materials.urdf.xacro" />
+  <!-- base laser front -->
+  <xacro:hokuyo_urg04_laser name="base_laser_front" parent="base" ros_topic="scan_front" update_rate="10" min_angle="-1.57" max_angle="1.57">
+    <origin xyz="0.3 0 -0.03" rpy="0 0 0"/>
+  </xacro:hokuyo_urg04_laser>
   <!-- base laser rear
   <xacro:hokuyo_urg04_laser name="base_laser_rear" parent="base" ros_topic="scan_rear" update_rate="10" min_angle="-1.57" max_angle="1.57" >

File: mir_robots/mir_hardware_config/youbot-brsu-4/urdf/robot.urdf.xacro (robot description, xacro)
@@ -20,4 +20,6 @@
   <!-- materials for visualization -->
   <xacro:include filename="$(find youbot_description)/urdf/materials.urdf.xacro" />
+  <!-- sensors -->
+  <xacro:include filename="$(find youbot_description)/urdf/sensors/hokuyo_urg04_laser.urdf.xacro"/>
   <!-- Now we can start using the macros included above to define the actual youbot -->
   <!-- The first use of a macro.  This one was defined in base.urdf.xacro above.
@@ -41,4 +43,8 @@
   <!-- BRSU SPECIFIC STUFF -->
   <xacro:include filename="$(find mcr_description)/urdf/materials.urdf.xacro" />
+  <!-- base laser front -->
+  <xacro:hokuyo_urg04_laser name="base_laser_front" parent="base" ros_topic="scan_front" update_rate="10" min_angle="-1.57" max_angle="1.57">
+    <origin xyz="0.3 0 -0.03" rpy="0 0 0"/>
+  </xacro:hokuyo_urg04_laser>
   <!-- base laser rear
   <xacro:hokuyo_urg04_laser name="base_laser_rear" parent="base" ros_topic="scan_rear" update_rate="10" min_angle="-1.57" max_angle="1.57" >

Commit message: add camera tower to URDF of yb1

File: mir_robots/mir_hardware_config/youbot-brsu-1/urdf/robot.urdf.xacro (robot description, xacro)
@@ -43,4 +43,5 @@
   <!-- BRSU SPECIFIC STUFF -->
   <xacro:include filename="$(find mcr_description)/urdf/materials.urdf.xacro" />
+  <xacro:include filename="$(find mir_description)/urdf/misc/cam3d_tower.urdf.xacro"/>
   <!-- base laser front -->
   <xacro:hokuyo_urg04_laser name="base_laser_front" parent="base" ros_topic="scan_front" update_rate="10" min_angle="-1.57" max_angle="1.57">
@@ -51,3 +52,7 @@
      <origin xyz="-0.3 0 -0.03" rpy="0 0 ${M_PI}" />
   </xacro:hokuyo_urg04_laser>
+  <!-- camera tower -->
+  <xacro:cam3d_tower name="camera_tower" parent="plate_link">
+    <origin xyz="-0.10 0.0 -0.01" rpy="0 0 0" />
+  </xacro:cam3d_tower>
 </robot>

Commit message: add ASUS Xtion to URDF of yb1

File: mir_robots/mir_hardware_config/youbot-brsu-1/urdf/robot.urdf.xacro (robot description, xacro)
@@ -44,4 +44,5 @@
   <xacro:include filename="$(find mcr_description)/urdf/materials.urdf.xacro" />
   <xacro:include filename="$(find mir_description)/urdf/misc/cam3d_tower.urdf.xacro"/>
+  <xacro:include filename="$(find mcr_description)/urdf/sensors/asus_xtion_camera.urdf.xacro"/>
   <!-- base laser front -->
   <xacro:hokuyo_urg04_laser name="base_laser_front" parent="base" ros_topic="scan_front" update_rate="10" min_angle="-1.57" max_angle="1.57">
@@ -56,3 +57,7 @@
     <origin xyz="-0.10 0.0 -0.01" rpy="0 0 0" />
   </xacro:cam3d_tower>
+  <!-- 3D camera on tower -->
+  <xacro:asus_xtion_camera name="tower_cam3d" parent="camera_tower_link" tilt="0.5">
+    <origin xyz="0.015 0 0.47" rpy="0 0 0" />
+  </xacro:asus_xtion_camera>
 </robot>

Commit message: add Microsoft RGB camera tower to URDF of yb1

File: mir_robots/mir_hardware_config/youbot-brsu-1/urdf/robot.urdf.xacro (robot description, xacro)
@@ -45,4 +45,5 @@
   <xacro:include filename="$(find mir_description)/urdf/misc/cam3d_tower.urdf.xacro"/>
   <xacro:include filename="$(find mcr_description)/urdf/sensors/asus_xtion_camera.urdf.xacro"/>
+  <xacro:include filename="$(find mcr_description)/urdf/mounts/microsoft_lifecam_1080_mount.urdf.xacro"/>
   <!-- base laser front -->
   <xacro:hokuyo_urg04_laser name="base_laser_front" parent="base" ros_topic="scan_front" update_rate="10" min_angle="-1.57" max_angle="1.57">
@@ -61,3 +62,7 @@
     <origin xyz="0.015 0 0.47" rpy="0 0 0" />
   </xacro:asus_xtion_camera>
+  <!-- Arm POV Mount -->
+  <xacro:microsoft_lifecam_1080_mount name="microsoft_lifecam_1080_mount" parent="arm_link_5">
+    <origin xyz="-0.035 0.0 -0.025" rpy="0 0 3.14159265" />
+  </xacro:microsoft_lifecam_1080_mount>
 </robot>

Commit message: replace the standard gripper with the new Festo gripper

File: mir_robots/mir_hardware_config/youbot-brsu-1/urdf/robot.urdf.xacro (robot description, xacro)
@@ -14,6 +14,4 @@
   <!-- youbot arm -->
   <xacro:include filename="$(find youbot_description)/urdf/youbot_arm/arm.urdf.xacro"/>
-  <!-- youbot gripper -->
-  <xacro:include filename="$(find youbot_description)/urdf/youbot_gripper/gripper.urdf.xacro" />
   <!-- controller manager -->
   <xacro:include filename="$(find youbot_description)/controller/ros_controller.urdf.xacro" />
@@ -38,7 +36,4 @@
     <origin xyz="0.143 0 0.046" rpy="0 0 0" />
   </xacro:youbot_arm>
-  <xacro:youbot_gripper name="gripper" parent="arm_link_5">
-    <origin xyz="0 0 0" rpy="0 0 0" />
-  </xacro:youbot_gripper>
   <!-- BRSU SPECIFIC STUFF -->
   <xacro:include filename="$(find mcr_description)/urdf/materials.urdf.xacro" />
@@ -46,4 +41,5 @@
   <xacro:include filename="$(find mcr_description)/urdf/sensors/asus_xtion_camera.urdf.xacro"/>
   <xacro:include filename="$(find mcr_description)/urdf/mounts/microsoft_lifecam_1080_mount.urdf.xacro"/>
+  <xacro:include filename="$(find mir_description)/urdf/grippers/festo_gripper.urdf.xacro" />
   <!-- base laser front -->
   <xacro:hokuyo_urg04_laser name="base_laser_front" parent="base" ros_topic="scan_front" update_rate="10" min_angle="-1.57" max_angle="1.57">
@@ -66,3 +62,6 @@
     <origin xyz="-0.035 0.0 -0.025" rpy="0 0 3.14159265" />
   </xacro:microsoft_lifecam_1080_mount>
+  <xacro:festo_gripper name="gripper" parent="arm_link_5">
+    <origin xyz="0 0 0" rpy="0 0 0" />
+  </xacro:festo_gripper>
 </robot>

Commit message: Updated arms on yb 1,3,4 to include adapter plate
This closes #64

File: mir_robots/mir_hardware_config/youbot-brsu-1/urdf/robot.urdf.xacro (robot description, xacro)
@@ -34,5 +34,5 @@
   </xacro:youbot_plate>
   <xacro:youbot_arm name="arm" parent="base_link">
-    <origin xyz="0.143 0 0.046" rpy="0 0 0" />
+    <origin xyz="0.223 0.017 0.088" rpy="0 0 ${-M_PI / 4}" />
   </xacro:youbot_arm>
   <!-- BRSU SPECIFIC STUFF -->
@@ -42,4 +42,8 @@
   <xacro:include filename="$(find mcr_description)/urdf/mounts/microsoft_lifecam_1080_mount.urdf.xacro"/>
   <xacro:include filename="$(find mir_description)/urdf/grippers/festo_gripper.urdf.xacro" />
+  <xacro:include filename="$(find mir_description)/urdf/misc/adapter_plate.urdf.xacro" />
+  <xacro:adapter_plate name="adapter_plate" parent="base_link">
+    <origin xyz="${0.159+0.08} 0 0.051" rpy="0 0 0" />
+  </xacro:adapter_plate>
   <!-- base laser front -->
   <xacro:hokuyo_urg04_laser name="base_laser_front" parent="base" ros_topic="scan_front" update_rate="10" min_angle="-1.57" max_angle="1.57">

File: mir_robots/mir_hardware_config/youbot-brsu-3/urdf/robot.urdf.xacro (robot description, xacro)
@@ -36,5 +36,5 @@
   </xacro:youbot_plate>
   <xacro:youbot_arm name="arm" parent="base_link">
-    <origin xyz="0.143 0 0.046" rpy="0 0 0" />
+    <origin xyz="0.223 0.017 0.088" rpy="0 0 ${-M_PI / 4}" />
   </xacro:youbot_arm>
   <xacro:youbot_gripper name="gripper" parent="arm_link_5">
@@ -45,4 +45,8 @@
   <xacro:include filename="$(find youbot_description)/urdf/sensors/asus_xtion_camera.urdf.xacro"/>
   <xacro:include filename="$(find youbot_description)/urdf/misc/camera_tower.urdf.xacro"/>
+  <xacro:include filename="$(find mir_description)/urdf/misc/adapter_plate.urdf.xacro" />
+  <xacro:adapter_plate name="adapter_plate" parent="base_link">
+    <origin xyz="${0.159+0.08} 0 0.051" rpy="0 0 0" />
+  </xacro:adapter_plate>
   <!-- base laser front -->
   <xacro:hokuyo_urg04_laser name="base_laser_front" parent="base" ros_topic="scan_front" update_rate="10" min_angle="-1.57" max_angle="1.57">

File: mir_robots/mir_hardware_config/youbot-brsu-4/urdf/robot.urdf.xacro (robot description, xacro)
@@ -36,5 +36,5 @@
   </xacro:youbot_plate>
   <xacro:youbot_arm name="arm" parent="base_link">
-    <origin xyz="0.143 0 0.046" rpy="0 0 0" />
+    <origin xyz="0.223 0.017 0.088" rpy="0 0 ${-M_PI / 4}" />
   </xacro:youbot_arm>
   <xacro:youbot_gripper name="gripper" parent="arm_link_5">
@@ -43,4 +43,8 @@
   <!-- BRSU SPECIFIC STUFF -->
   <xacro:include filename="$(find mcr_description)/urdf/materials.urdf.xacro" />
+  <xacro:include filename="$(find mir_description)/urdf/misc/adapter_plate.urdf.xacro" />
+  <xacro:adapter_plate name="adapter_plate" parent="base_link">
+    <origin xyz="${0.159+0.08} 0 0.051" rpy="0 0 0" />
+  </xacro:adapter_plate>
   <!-- base laser front -->
   <xacro:hokuyo_urg04_laser name="base_laser_front" parent="base" ros_topic="scan_front" update_rate="10" min_angle="-1.57" max_angle="1.57">
