Commit message: Sync robot descriptions
- Update YB1 and YB2 to use adapter_plate macro with arm_angle
- Rotate yb-4 arm the other direction to match yb1 and yb2

File: mir_robots/mir_hardware_config/youbot-brsu-1/urdf/robot.urdf.xacro (robot description, xacro)
@@ -33,7 +33,4 @@
     <origin xyz="-0.159 0 0.046" rpy="0 0 0" />
   </xacro:youbot_plate>
-  <xacro:youbot_arm name="arm" parent="base_link">
-    <origin xyz="0.223 0.017 0.088" rpy="0 0 ${-M_PI / 4}" />
-  </xacro:youbot_arm>
   <!-- BRSU SPECIFIC STUFF -->
   <xacro:include filename="$(find mcr_description)/urdf/materials.urdf.xacro" />
@@ -43,7 +40,11 @@
   <xacro:include filename="$(find mir_description)/urdf/grippers/festo_gripper.urdf.xacro" />
   <xacro:include filename="$(find mir_description)/urdf/misc/adapter_plate.urdf.xacro" />
-  <xacro:adapter_plate name="adapter_plate" parent="base_link">
+  <!-- Arm Plate moving arm 8cm foward and 45 degree rotation -->
+  <xacro:adapter_plate name="adapter_plate" parent="base_link" arm_angle="${-M_PI / 4}">
     <origin xyz="${0.159+0.08} 0 0.051" rpy="0 0 0" />
   </xacro:adapter_plate>
+  <xacro:youbot_arm name="arm" parent="adapter_plate_arm_root_link">
+    <origin xyz="-0.022 0.0 0.037" rpy="0 0 0" />
+  </xacro:youbot_arm>
   <!-- base laser front -->
   <xacro:hokuyo_urg04_laser name="base_laser_front" parent="base" ros_topic="scan_front" update_rate="10" min_angle="-1.57" max_angle="1.57">

File: mir_robots/mir_hardware_config/youbot-brsu-2/urdf/robot.urdf.xacro (robot description, xacro)
@@ -23,10 +23,4 @@
   <!-- standard youBot configuration -->
   <xacro:youbot_base name="base"/>
-  <xacro:rear_platform name="rear_platform" parent="base_link">
-    <origin xyz="-0.005 -0.175 0.051" rpy="0 0 0" />
-  </xacro:rear_platform>
-  <xacro:youbot_arm name="arm" parent="base_link">
-    <origin xyz="0.223 0.017 0.088" rpy="0 0 ${-M_PI / 4}" />
-  </xacro:youbot_arm>
   <!-- BRSU SPECIFIC STUFF -->
   <xacro:include filename="$(find mcr_description)/urdf/materials.urdf.xacro" />
@@ -37,7 +31,15 @@
   <xacro:include filename="$(find mir_description)/urdf/misc/rear_platform.urdf.xacro" />
   <xacro:include filename="$(find mir_description)/urdf/misc/adapter_plate.urdf.xacro" />
-  <xacro:adapter_plate name="adapter_plate" parent="base_link">
+  <!-- Rear Platform -->
+  <xacro:rear_platform name="rear_platform" parent="base_link">
+    <origin xyz="-0.005 -0.175 0.051" rpy="0 0 0" />
+  </xacro:rear_platform>
+  <!-- Arm Plate moving arm 8cm foward and 45 degree rotation -->
+  <xacro:adapter_plate name="adapter_plate" parent="base_link" arm_angle="${-M_PI / 4}">
     <origin xyz="${0.159+0.08} 0 0.051" rpy="0 0 0" />
   </xacro:adapter_plate>
+  <xacro:youbot_arm name="arm" parent="adapter_plate_arm_root_link">
+    <origin xyz="-0.022 0.0 0.037" rpy="0 0 0" />
+  </xacro:youbot_arm>
   <!-- base laser front -->
   <xacro:hokuyo_urg04_laser name="base_laser_front" parent="base" ros_topic="scan_front" update_rate="10" min_angle="-1.57" max_angle="1.57">

File: mir_robots/mir_hardware_config/youbot-brsu-4/urdf/robot.urdf.xacro (robot description, xacro)
@@ -44,5 +44,5 @@
   </xacro:rear_platform>
   <!-- Arm Plate moving arm 8cm foward and 45 degree rotation -->
-  <xacro:adapter_plate name="adapter_plate" parent="base_link" arm_angle="${M_PI / 4}">
+  <xacro:adapter_plate name="adapter_plate" parent="base_link" arm_angle="${-M_PI / 4}">
     <origin xyz="${0.159+0.08} 0 0.051" rpy="0 0 0" />
   </xacro:adapter_plate>

Commit message: Updating urdf model for yb1, just copied over from yb2

File: mir_robots/mir_hardware_config/youbot-brsu-1/urdf/robot.urdf.xacro (robot description, xacro)
@@ -21,16 +21,6 @@
   <xacro:include filename="$(find youbot_description)/urdf/sensors/hokuyo_urg04_laser.urdf.xacro"/>
   <!-- Now we can start using the macros included above to define the actual youbot -->
-  <!-- The first use of a macro.  This one was defined in base.urdf.xacro above.
-       A macro like this will expand to a set of link and joint definitions, and to additional
-       Gazebo-related extensions (sensor plugins, etc).  The macro takes an argument, name,
-       that equals "base", and uses it to generate names for its component links and joints
-       (e.g., base_link).  The included origin block is also an argument to the macro.  By convention,
-       the origin block defines where the component is w.r.t its parent (in this case the parent
-       is the world frame). For more, see http://www.ros.org/wiki/xacro -->
-  <!-- foot for arm-->
+  <!-- standard youBot configuration -->
   <xacro:youbot_base name="base"/>
-  <xacro:youbot_plate name="plate" parent="base_link">
-    <origin xyz="-0.159 0 0.046" rpy="0 0 0" />
-  </xacro:youbot_plate>
   <!-- BRSU SPECIFIC STUFF -->
   <xacro:include filename="$(find mcr_description)/urdf/materials.urdf.xacro" />
@@ -39,5 +29,10 @@
   <xacro:include filename="$(find mcr_description)/urdf/mounts/microsoft_lifecam_1080_mount.urdf.xacro"/>
   <xacro:include filename="$(find mir_description)/urdf/grippers/festo_gripper.urdf.xacro" />
+  <xacro:include filename="$(find mir_description)/urdf/misc/rear_platform.urdf.xacro" />
   <xacro:include filename="$(find mir_description)/urdf/misc/adapter_plate.urdf.xacro" />
+  <!-- Rear Platform -->
+  <xacro:rear_platform name="rear_platform" parent="base_link">
+    <origin xyz="-0.005 -0.175 0.051" rpy="0 0 0" />
+  </xacro:rear_platform>
   <!-- Arm Plate moving arm 8cm foward and 45 degree rotation -->
   <xacro:adapter_plate name="adapter_plate" parent="base_link" arm_angle="${-M_PI / 4}">
@@ -53,9 +48,9 @@
   <!-- base laser rear -->
   <xacro:hokuyo_urg04_laser name="base_laser_rear" parent="base" ros_topic="scan_rear" update_rate="10" min_angle="-1.57" max_angle="1.57" >
-     <origin xyz="-0.3 0 -0.03" rpy="0 0 ${M_PI}" />
+     <origin xyz="-0.3 0.0 -0.03" rpy="0 0 ${M_PI}" />
   </xacro:hokuyo_urg04_laser>
   <!-- camera tower -->
-  <xacro:cam3d_tower name="camera_tower" parent="plate_link">
-    <origin xyz="-0.10 0.0 -0.01" rpy="0 0 0" />
+  <xacro:cam3d_tower name="camera_tower" parent="rear_platform_link">
+    <origin xyz="-0.227 0.165 0.023" rpy="0 0 0" />
   </xacro:cam3d_tower>
   <!-- 3D camera on tower -->

Commit message: [yb1] replace Microsoft arm cam with ASUS 3d cam

File: mir_robots/mir_hardware_config/youbot-brsu-1/urdf/robot.urdf.xacro (robot description, xacro)
@@ -50,16 +50,18 @@
      <origin xyz="-0.3 0.0 -0.03" rpy="0 0 ${M_PI}" />
   </xacro:hokuyo_urg04_laser>
-  <!-- camera tower -->
+  <!-- camera tower
   <xacro:cam3d_tower name="camera_tower" parent="rear_platform_link">
     <origin xyz="-0.227 0.165 0.023" rpy="0 0 0" />
   </xacro:cam3d_tower>
-  <!-- 3D camera on tower -->
-  <xacro:asus_xtion_camera name="tower_cam3d" parent="camera_tower_link" tilt="0.5">
-    <origin xyz="0.015 0 0.47" rpy="0 0 0" />
+  -->
+  <!-- 3D camera on arm -->
+  <xacro:asus_xtion_camera name="tower_cam3d" parent="arm_link_5" tilt="0.0">
+    <origin xyz="${-0.035 - 0.030 + 0.030} ${0 - 0.025} ${-0.025}" rpy="0 ${-M_PI /  2} 0" />
   </xacro:asus_xtion_camera>
-  <!-- Arm POV Mount -->
+  <!-- Arm POV Mount
   <xacro:microsoft_lifecam_1080_mount name="microsoft_lifecam_1080_mount" parent="arm_link_5">
     <origin xyz="-0.035 0.0 -0.025" rpy="0 0 3.14159265" />
   </xacro:microsoft_lifecam_1080_mount>
+  -->
   <xacro:festo_gripper name="gripper" parent="arm_link_5">
     <origin xyz="0 0 0" rpy="0 0 0" />

Commit message: [yb1] remove space

File: mir_robots/mir_hardware_config/youbot-brsu-1/urdf/robot.urdf.xacro (robot description, xacro)
@@ -57,5 +57,5 @@
   <!-- 3D camera on arm -->
   <xacro:asus_xtion_camera name="tower_cam3d" parent="arm_link_5" tilt="0.0">
-    <origin xyz="${-0.035 - 0.030 + 0.030} ${0 - 0.025} ${-0.025}" rpy="0 ${-M_PI /  2} 0" />
+    <origin xyz="${-0.035 - 0.030 + 0.030} ${0 - 0.025} ${-0.025}" rpy="0 ${-M_PI / 2} 0" />
   </xacro:asus_xtion_camera>
   <!-- Arm POV Mount

Commit message: [yb1] add camera tower and camera dummy on it

File: mir_robots/mir_hardware_config/youbot-brsu-1/urdf/robot.urdf.xacro (robot description, xacro)
@@ -50,12 +50,15 @@
      <origin xyz="-0.3 0.0 -0.03" rpy="0 0 ${M_PI}" />
   </xacro:hokuyo_urg04_laser>
-  <!-- camera tower
+  <!-- camera tower -->
   <xacro:cam3d_tower name="camera_tower" parent="rear_platform_link">
     <origin xyz="-0.227 0.165 0.023" rpy="0 0 0" />
   </xacro:cam3d_tower>
-  -->
   <!-- 3D camera on arm -->
   <xacro:asus_xtion_camera name="tower_cam3d" parent="arm_link_5" tilt="0.0">
     <origin xyz="${-0.035 - 0.030 + 0.030} ${0 - 0.025} ${-0.025}" rpy="0 ${-M_PI / 2} 0" />
+  </xacro:asus_xtion_camera>
+  <!-- 3D camera on tower (not used at the moment) -->
+  <xacro:asus_xtion_camera name="tower_cam3d_dummy" parent="camera_tower_link" tilt="0.5">
+    <origin xyz="0.015 0 0.47" rpy="0 0 0" />
   </xacro:asus_xtion_camera>
   <!-- Arm POV Mount

Commit message: [calibration] calibrate ASUS arm cam on yb1

File: mir_robots/mir_hardware_config/youbot-brsu-1/urdf/robot.urdf.xacro (robot description, xacro)
@@ -56,5 +56,5 @@
   <!-- 3D camera on arm -->
   <xacro:asus_xtion_camera name="tower_cam3d" parent="arm_link_5" tilt="0.0">
-    <origin xyz="${-0.035 - 0.030 + 0.030} ${0 - 0.025} ${-0.025}" rpy="0 ${-M_PI / 2} 0" />
+    <origin xyz="${-0.035 - 0.030 + 0.030} ${0 - 0.015} ${-0.09}" rpy="0 ${-M_PI / 2} 0" />
   </xacro:asus_xtion_camera>
   <!-- 3D camera on tower (not used at the moment) -->
