Commit message: Cleanup, simply and syncronize all of the robot.urdf.xacro
All of the robots are now considered to be configured as they were
for German Open 2015. Which assumes we would have enough laser scanners,
rear platforms and grippers to go around. But the code-base expects frames,
sensors, etc. to exist so they would be modified to the same state before being run, so
this is a reasonable assumption.

File: mir_robots/mir_hardware_config/youbot-brsu-1/urdf/robot.urdf.xacro (robot description, xacro)
@@ -6,12 +6,14 @@
        name="youbot" >
   <!-- The following included files set up definitions of parts of the robot body -->
-  <!-- misc common stuff? -->
+  <!-- misc common stuff -->
   <xacro:include filename="$(find youbot_description)/urdf/common.xacro" />
-  <!-- youbot base -->
+  <xacro:include filename="$(find mcr_description)/urdf/materials.urdf.xacro" />
+  <!-- youbot base and rear platform -->
   <xacro:include filename="$(find youbot_description)/urdf/youbot_base/base.urdf.xacro" />
-  <!-- youbot plate -->
-  <xacro:include filename="$(find youbot_description)/urdf/youbot_plate/plate.urdf.xacro" />
-  <!-- youbot arm -->
+  <xacro:include filename="$(find mir_description)/urdf/misc/rear_platform.urdf.xacro" />
+  <!-- youbot arm and gripper-->
   <xacro:include filename="$(find youbot_description)/urdf/youbot_arm/arm.urdf.xacro"/>
+  <xacro:include filename="$(find mir_description)/urdf/misc/adapter_plate.urdf.xacro" />
+  <xacro:include filename="$(find mir_description)/urdf/grippers/festo_gripper.urdf.xacro" />
   <!-- controller manager -->
   <xacro:include filename="$(find youbot_description)/controller/ros_controller.urdf.xacro" />
@@ -20,15 +22,8 @@
   <!-- sensors -->
   <xacro:include filename="$(find youbot_description)/urdf/sensors/hokuyo_urg04_laser.urdf.xacro"/>
+  <xacro:include filename="$(find mcr_description)/urdf/sensors/asus_xtion_camera.urdf.xacro"/>
   <!-- Now we can start using the macros included above to define the actual youbot -->
   <!-- standard youBot configuration -->
   <xacro:youbot_base name="base"/>
-  <!-- BRSU SPECIFIC STUFF -->
-  <xacro:include filename="$(find mcr_description)/urdf/materials.urdf.xacro" />
-  <xacro:include filename="$(find mir_description)/urdf/misc/cam3d_tower.urdf.xacro"/>
-  <xacro:include filename="$(find mcr_description)/urdf/sensors/asus_xtion_camera.urdf.xacro"/>
-  <xacro:include filename="$(find mcr_description)/urdf/mounts/microsoft_lifecam_1080_mount.urdf.xacro"/>
-  <xacro:include filename="$(find mir_description)/urdf/grippers/festo_gripper.urdf.xacro" />
-  <xacro:include filename="$(find mir_description)/urdf/misc/rear_platform.urdf.xacro" />
-  <xacro:include filename="$(find mir_description)/urdf/misc/adapter_plate.urdf.xacro" />
   <!-- Rear Platform -->
   <xacro:rear_platform name="rear_platform" parent="base_link">
@@ -50,21 +45,8 @@
      <origin xyz="-0.3 0.0 -0.03" rpy="0 0 ${M_PI}" />
   </xacro:hokuyo_urg04_laser>
-  <!-- camera tower -->
-  <xacro:cam3d_tower name="camera_tower" parent="rear_platform_link">
-    <origin xyz="-0.227 0.165 0.023" rpy="0 0 0" />
-  </xacro:cam3d_tower>
-  <!-- 3D camera on arm -->
+  <!-- 3D camera on arm --> <!-- NOTE: still called tower_cam3d due to legacy code -->
   <xacro:asus_xtion_camera name="tower_cam3d" parent="arm_link_5" tilt="0.0">
     <origin xyz="${-0.035 - 0.030 + 0.030} ${0 - 0.015} ${-0.09}" rpy="0 ${-M_PI / 2} 0" />
   </xacro:asus_xtion_camera>
-  <!-- 3D camera on tower (not used at the moment) -->
-  <xacro:asus_xtion_camera name="tower_cam3d_dummy" parent="camera_tower_link" tilt="0.5">
-    <origin xyz="0.015 0 0.47" rpy="0 0 0" />
-  </xacro:asus_xtion_camera>
-  <!-- Arm POV Mount
-  <xacro:microsoft_lifecam_1080_mount name="microsoft_lifecam_1080_mount" parent="arm_link_5">
-    <origin xyz="-0.035 0.0 -0.025" rpy="0 0 3.14159265" />
-  </xacro:microsoft_lifecam_1080_mount>
-  -->
   <xacro:festo_gripper name="gripper" parent="arm_link_5">
     <origin xyz="0 0 0" rpy="0 0 0" />

File: mir_robots/mir_hardware_config/youbot-brsu-2/urdf/robot.urdf.xacro (robot description, xacro)
@@ -6,12 +6,14 @@
        name="youbot" >
   <!-- The following included files set up definitions of parts of the robot body -->
-  <!-- misc common stuff? -->
+  <!-- misc common stuff -->
   <xacro:include filename="$(find youbot_description)/urdf/common.xacro" />
-  <!-- youbot base -->
+  <xacro:include filename="$(find mcr_description)/urdf/materials.urdf.xacro" />
+  <!-- youbot base and rear platform -->
   <xacro:include filename="$(find youbot_description)/urdf/youbot_base/base.urdf.xacro" />
-  <!-- youbot plate -->
-  <xacro:include filename="$(find youbot_description)/urdf/youbot_plate/plate.urdf.xacro" />
-  <!-- youbot arm -->
+  <xacro:include filename="$(find mir_description)/urdf/misc/rear_platform.urdf.xacro" />
+  <!-- youbot arm and gripper-->
   <xacro:include filename="$(find youbot_description)/urdf/youbot_arm/arm.urdf.xacro"/>
+  <xacro:include filename="$(find mir_description)/urdf/misc/adapter_plate.urdf.xacro" />
+  <xacro:include filename="$(find mir_description)/urdf/grippers/festo_gripper.urdf.xacro" />
   <!-- controller manager -->
   <xacro:include filename="$(find youbot_description)/controller/ros_controller.urdf.xacro" />
@@ -20,15 +22,8 @@
   <!-- sensors -->
   <xacro:include filename="$(find youbot_description)/urdf/sensors/hokuyo_urg04_laser.urdf.xacro"/>
+  <xacro:include filename="$(find mcr_description)/urdf/sensors/asus_xtion_camera.urdf.xacro"/>
   <!-- Now we can start using the macros included above to define the actual youbot -->
   <!-- standard youBot configuration -->
   <xacro:youbot_base name="base"/>
-  <!-- BRSU SPECIFIC STUFF -->
-  <xacro:include filename="$(find mcr_description)/urdf/materials.urdf.xacro" />
-  <xacro:include filename="$(find mir_description)/urdf/misc/cam3d_tower.urdf.xacro"/>
-  <xacro:include filename="$(find mcr_description)/urdf/sensors/asus_xtion_camera.urdf.xacro"/>
-  <xacro:include filename="$(find mcr_description)/urdf/mounts/microsoft_lifecam_1080_mount.urdf.xacro"/>
-  <xacro:include filename="$(find mir_description)/urdf/grippers/festo_gripper.urdf.xacro" />
-  <xacro:include filename="$(find mir_description)/urdf/misc/rear_platform.urdf.xacro" />
-  <xacro:include filename="$(find mir_description)/urdf/misc/adapter_plate.urdf.xacro" />
   <!-- Rear Platform -->
   <xacro:rear_platform name="rear_platform" parent="base_link">
@@ -50,16 +45,8 @@
      <origin xyz="-0.3 0.0 -0.03" rpy="0 0 ${M_PI}" />
   </xacro:hokuyo_urg04_laser>
-  <!-- camera tower -->
-  <xacro:cam3d_tower name="camera_tower" parent="rear_platform_link">
-    <origin xyz="-0.227 0.165 0.023" rpy="0 0 0" />
-  </xacro:cam3d_tower>
-  <!-- 3D camera on tower -->
-  <xacro:asus_xtion_camera name="tower_cam3d" parent="camera_tower_link" tilt="0.5">
-    <origin xyz="0.015 0 0.47" rpy="0 0 0" />
+  <!-- 3D camera on arm --> <!-- NOTE: still called tower_cam3d due to legacy code -->
+  <xacro:asus_xtion_camera name="tower_cam3d" parent="arm_link_5" tilt="0.0">
+    <origin xyz="${-0.035 - 0.030 + 0.030} ${0 - 0.015} ${-0.09}" rpy="0 ${-M_PI / 2} 0" />
   </xacro:asus_xtion_camera>
-  <!-- Arm POV Mount -->
-  <xacro:microsoft_lifecam_1080_mount name="microsoft_lifecam_1080_mount" parent="arm_link_5">
-    <origin xyz="-0.035 0.0 -0.025" rpy="0 0 3.14159265" />
-  </xacro:microsoft_lifecam_1080_mount>
   <xacro:festo_gripper name="gripper" parent="arm_link_5">
     <origin xyz="0 0 0" rpy="0 0 0" />

File: mir_robots/mir_hardware_config/youbot-brsu-3/urdf/robot.urdf.xacro (robot description, xacro)
@@ -6,12 +6,14 @@
        name="youbot" >
   <!-- The following included files set up definitions of parts of the robot body -->
-  <!-- misc common stuff? -->
+  <!-- misc common stuff -->
   <xacro:include filename="$(find youbot_description)/urdf/common.xacro" />
-  <!-- youbot base -->
+  <xacro:include filename="$(find mcr_description)/urdf/materials.urdf.xacro" />
+  <!-- youbot base and rear platform -->
   <xacro:include filename="$(find youbot_description)/urdf/youbot_base/base.urdf.xacro" />
-  <!-- youbot plate -->
-  <xacro:include filename="$(find youbot_description)/urdf/youbot_plate/plate.urdf.xacro" />
-  <!-- youbot arm -->
+  <xacro:include filename="$(find mir_description)/urdf/misc/rear_platform.urdf.xacro" />
+  <!-- youbot arm and gripper-->
   <xacro:include filename="$(find youbot_description)/urdf/youbot_arm/arm.urdf.xacro"/>
+  <xacro:include filename="$(find mir_description)/urdf/misc/adapter_plate.urdf.xacro" />
+  <xacro:include filename="$(find mir_description)/urdf/grippers/festo_gripper.urdf.xacro" />
   <!-- controller manager -->
   <xacro:include filename="$(find youbot_description)/controller/ros_controller.urdf.xacro" />
@@ -20,25 +22,12 @@
   <!-- sensors -->
   <xacro:include filename="$(find youbot_description)/urdf/sensors/hokuyo_urg04_laser.urdf.xacro"/>
+  <xacro:include filename="$(find mcr_description)/urdf/sensors/asus_xtion_camera.urdf.xacro"/>
   <!-- Now we can start using the macros included above to define the actual youbot -->
-  <!-- The first use of a macro.  This one was defined in base.urdf.xacro above.
-       A macro like this will expand to a set of link and joint definitions, and to additional
-       Gazebo-related extensions (sensor plugins, etc).  The macro takes an argument, name,
-       that equals "base", and uses it to generate names for its component links and joints
-       (e.g., base_link).  The included origin block is also an argument to the macro.  By convention,
-       the origin block defines where the component is w.r.t its parent (in this case the parent
-       is the world frame). For more, see http://www.ros.org/wiki/xacro -->
-  <!-- foot for arm-->
+  <!-- standard youBot configuration -->
   <xacro:youbot_base name="base"/>
-  <!-- rear platform -->
-  <xacro:youbot_plate name="plate" parent="base_link">
-    <origin xyz="-0.159 0 0.046" rpy="0 0 0" />
-  </xacro:youbot_plate>
-  <!-- BRSU SPECIFIC STUFF -->
-  <xacro:include filename="$(find mcr_description)/urdf/materials.urdf.xacro" />
-  <xacro:include filename="$(find mir_description)/urdf/misc/cam3d_tower.urdf.xacro"/>
-  <xacro:include filename="$(find mcr_description)/urdf/sensors/asus_xtion_camera.urdf.xacro"/>
-  <xacro:include filename="$(find mcr_description)/urdf/mounts/microsoft_lifecam_1080_mount.urdf.xacro"/>
-  <xacro:include filename="$(find mir_description)/urdf/grippers/festo_gripper.urdf.xacro" />
-  <xacro:include filename="$(find mir_description)/urdf/misc/adapter_plate.urdf.xacro" />
+  <!-- Rear Platform -->
+  <xacro:rear_platform name="rear_platform" parent="base_link">
+    <origin xyz="-0.005 -0.175 0.051" rpy="0 0 0" />
+  </xacro:rear_platform>
   <!-- Arm Plate moving arm 8cm foward and 45 degree rotation -->
   <xacro:adapter_plate name="adapter_plate" parent="base_link" arm_angle="${-M_PI / 4}">
@@ -54,20 +43,10 @@
   <!-- base laser rear -->
   <xacro:hokuyo_urg04_laser name="base_laser_rear" parent="base" ros_topic="scan_rear" update_rate="10" min_angle="-1.57" max_angle="1.57" >
-     <origin xyz="-0.3 0 -0.03" rpy="0 0 ${M_PI}" />
+     <origin xyz="-0.3 0.0 -0.03" rpy="0 0 ${M_PI}" />
   </xacro:hokuyo_urg04_laser>
-  <!-- camera tower
-  <xacro:cam3d_tower name="camera_tower" parent="plate_link">
-    <origin xyz="-0.10 0.0 -0.01" rpy="0 0 0" />
-  </xacro:cam3d_tower>
-  -->
-  <!-- 3D camera on arm -->
+  <!-- 3D camera on arm --> <!-- NOTE: still called tower_cam3d due to legacy code -->
   <xacro:asus_xtion_camera name="tower_cam3d" parent="arm_link_5" tilt="0.0">
-    <origin xyz="${-0.035 - 0.030 + 0.030 + 0.01} ${0 - 0.055} ${-0.025 - 0.0}" rpy="0 ${-M_PI / 2} 0" />
+    <origin xyz="${-0.035 - 0.030 + 0.030} ${0 - 0.015} ${-0.09}" rpy="0 ${-M_PI / 2} 0" />
   </xacro:asus_xtion_camera>
-  <!-- Arm POV Mount
-  <xacro:microsoft_lifecam_1080_mount name="microsoft_lifecam_1080_mount" parent="arm_link_5">
-    <origin xyz="-0.035 0.0 -0.025" rpy="0 0 3.14159265" />
-  </xacro:microsoft_lifecam_1080_mount>
-  -->
   <xacro:festo_gripper name="gripper" parent="arm_link_5">
     <origin xyz="0 0 0" rpy="0 0 0" />

File: mir_robots/mir_hardware_config/youbot-brsu-4/urdf/robot.urdf.xacro (robot description, xacro)
@@ -6,14 +6,14 @@
        name="youbot" >
   <!-- The following included files set up definitions of parts of the robot body -->
-  <!-- misc common stuff? -->
+  <!-- misc common stuff -->
   <xacro:include filename="$(find youbot_description)/urdf/common.xacro" />
-  <!-- youbot base -->
+  <xacro:include filename="$(find mcr_description)/urdf/materials.urdf.xacro" />
+  <!-- youbot base and rear platform -->
   <xacro:include filename="$(find youbot_description)/urdf/youbot_base/base.urdf.xacro" />
-  <!-- youbot plate -->
-  <xacro:include filename="$(find youbot_description)/urdf/youbot_plate/plate.urdf.xacro" />
-  <!-- youbot arm -->
+  <xacro:include filename="$(find mir_description)/urdf/misc/rear_platform.urdf.xacro" />
+  <!-- youbot arm and gripper-->
   <xacro:include filename="$(find youbot_description)/urdf/youbot_arm/arm.urdf.xacro"/>
-  <!-- youbot gripper -->
-  <xacro:include filename="$(find youbot_description)/urdf/youbot_gripper/gripper.urdf.xacro" />
+  <xacro:include filename="$(find mir_description)/urdf/misc/adapter_plate.urdf.xacro" />
+  <xacro:include filename="$(find mir_description)/urdf/grippers/festo_gripper.urdf.xacro" />
   <!-- controller manager -->
   <xacro:include filename="$(find youbot_description)/controller/ros_controller.urdf.xacro" />
@@ -22,22 +22,8 @@
   <!-- sensors -->
   <xacro:include filename="$(find youbot_description)/urdf/sensors/hokuyo_urg04_laser.urdf.xacro"/>
+  <xacro:include filename="$(find mcr_description)/urdf/sensors/asus_xtion_camera.urdf.xacro"/>
   <!-- Now we can start using the macros included above to define the actual youbot -->
-  <!-- The first use of a macro.  This one was defined in base.urdf.xacro above.
-       A macro like this will expand to a set of link and joint definitions, and to additional
-       Gazebo-related extensions (sensor plugins, etc).  The macro takes an argument, name,
-       that equals "base", and uses it to generate names for its component links and joints
-       (e.g., base_link).  The included origin block is also an argument to the macro.  By convention,
-       the origin block defines where the component is w.r.t its parent (in this case the parent
-       is the world frame). For more, see http://www.ros.org/wiki/xacro -->
-  <!-- foot for arm-->
+  <!-- standard youBot configuration -->
   <xacro:youbot_base name="base"/>
-  <!-- BRSU SPECIFIC STUFF -->
-  <xacro:include filename="$(find mcr_description)/urdf/materials.urdf.xacro" />
-  <xacro:include filename="$(find mir_description)/urdf/misc/cam3d_tower.urdf.xacro"/>
-  <xacro:include filename="$(find mcr_description)/urdf/sensors/asus_xtion_camera.urdf.xacro"/>
-  <xacro:include filename="$(find mcr_description)/urdf/mounts/microsoft_lifecam_1080_mount.urdf.xacro"/>
-  <xacro:include filename="$(find mir_description)/urdf/misc/rear_platform.urdf.xacro" />
-  <xacro:include filename="$(find mir_description)/urdf/misc/adapter_plate.urdf.xacro" />
-  <xacro:include filename="$(find mir_description)/urdf/grippers/festo_gripper.urdf.xacro" />
   <!-- Rear Platform -->
   <xacro:rear_platform name="rear_platform" parent="base_link">
@@ -51,8 +37,4 @@
     <origin xyz="-0.022 0.0 0.037" rpy="0 0 0" />
   </xacro:youbot_arm>
-  <!-- Festo Gripper -->
-  <xacro:festo_gripper name="gripper" parent="arm_link_5">
-    <origin xyz="0 0 0" rpy="0 0 0" />
-  </xacro:festo_gripper>
   <!-- base laser front -->
   <xacro:hokuyo_urg04_laser name="base_laser_front" parent="base" ros_topic="scan_front" update_rate="10" min_angle="-1.57" max_angle="1.57">
@@ -61,17 +43,12 @@
   <!-- base laser rear -->
   <xacro:hokuyo_urg04_laser name="base_laser_rear" parent="base" ros_topic="scan_rear" update_rate="10" min_angle="-1.57" max_angle="1.57" >
-     <origin xyz="-0.3 0 -0.03" rpy="0 0 ${M_PI}" />
+     <origin xyz="-0.3 0.0 -0.03" rpy="0 0 ${M_PI}" />
   </xacro:hokuyo_urg04_laser>
-  <!-- camera tower -->
-  <xacro:cam3d_tower name="camera_tower" parent="rear_platform_link">
-    <origin xyz="-0.227 0.165 0.023" rpy="0 0 0" />
-  </xacro:cam3d_tower>
-  <!-- 3D camera on tower -->
-  <xacro:asus_xtion_camera name="tower_cam3d" parent="camera_tower_link" tilt="0.5">
-    <origin xyz="0.015 0 0.47" rpy="0 0 0" />
+  <!-- 3D camera on arm --> <!-- NOTE: still called tower_cam3d due to legacy code -->
+  <xacro:asus_xtion_camera name="tower_cam3d" parent="arm_link_5" tilt="0.0">
+    <origin xyz="${-0.035 - 0.030 + 0.030} ${0 - 0.015} ${-0.09}" rpy="0 ${-M_PI / 2} 0" />
   </xacro:asus_xtion_camera>
-  <!-- Arm POV Mount -->
-  <xacro:microsoft_lifecam_1080_mount name="microsoft_lifecam_1080_mount" parent="arm_link_5">
-    <origin xyz="-0.035 0.0 -0.025" rpy="0 0 3.14159265" />
-  </xacro:microsoft_lifecam_1080_mount>
+  <xacro:festo_gripper name="gripper" parent="arm_link_5">
+    <origin xyz="0 0 0" rpy="0 0 0" />
+  </xacro:festo_gripper>
 </robot>

Commit message: YouBots 1 and 3 with realsense camera
Otherwise same as German Open 2015.

File: mir_robots/mir_hardware_config/youbot-brsu-1/urdf/robot.urdf.xacro (robot description, xacro)
@@ -22,5 +22,5 @@
   <!-- sensors -->
   <xacro:include filename="$(find youbot_description)/urdf/sensors/hokuyo_urg04_laser.urdf.xacro"/>
-  <xacro:include filename="$(find mcr_description)/urdf/sensors/asus_xtion_camera.urdf.xacro"/>
+  <xacro:include filename="$(find mcr_description)/urdf/sensors/realsense_camera.urdf.xacro"/>
   <!-- Now we can start using the macros included above to define the actual youbot -->
   <!-- standard youBot configuration -->
@@ -46,7 +46,7 @@
   </xacro:hokuyo_urg04_laser>
   <!-- 3D camera on arm --> <!-- NOTE: still called tower_cam3d due to legacy code -->
-  <xacro:asus_xtion_camera name="tower_cam3d" parent="arm_link_5" tilt="0.0">
-    <origin xyz="${-0.035 - 0.030 + 0.030} ${0 - 0.015} ${-0.09}" rpy="0 ${-M_PI / 2} 0" />
-  </xacro:asus_xtion_camera>
+  <xacro:realsense_camera name="tower_cam3d" parent="arm_link_5">
+    <origin xyz="-0.075 0 0.02" rpy="0 ${-M_PI / 2} 0" />
+  </xacro:realsense_camera>
   <xacro:festo_gripper name="gripper" parent="arm_link_5">
     <origin xyz="0 0 0" rpy="0 0 0" />

Commit message: YB1, YB3 with Dynamixel Gripper, update moveit config.

File: mir_robots/mir_hardware_config/youbot-brsu-1/urdf/robot.urdf.xacro (robot description, xacro)
@@ -15,5 +15,5 @@
   <xacro:include filename="$(find youbot_description)/urdf/youbot_arm/arm.urdf.xacro"/>
   <xacro:include filename="$(find mir_description)/urdf/misc/adapter_plate.urdf.xacro" />
-  <xacro:include filename="$(find mir_description)/urdf/grippers/festo_gripper.urdf.xacro" />
+  <xacro:include filename="$(find mir_description)/urdf/grippers/dynamixel_gripper.urdf.xacro" />
   <!-- controller manager -->
   <xacro:include filename="$(find youbot_description)/controller/ros_controller.urdf.xacro" />
@@ -47,8 +47,8 @@
   <!-- 3D camera on arm --> <!-- NOTE: still called tower_cam3d due to legacy code -->
   <xacro:realsense_camera name="tower_cam3d" parent="arm_link_5">
-    <origin xyz="-0.075 0 0.02" rpy="0 ${-M_PI / 2} 0" />
+    <origin xyz="-0.075 0.024 0.04" rpy="0 ${-M_PI / 2} 0" />
   </xacro:realsense_camera>
-  <xacro:festo_gripper name="gripper" parent="arm_link_5">
-    <origin xyz="0 0 0" rpy="0 0 0" />
-  </xacro:festo_gripper>
+  <xacro:dynamixel_gripper name="gripper" parent="arm_link_5">
+    <origin xyz="0 0 -0.02" rpy="0 0 0" />
+  </xacro:dynamixel_gripper>
 </robot>

Commit message: add old gripper to yb1 urdf and simulation

File: mir_robots/mir_hardware_config/youbot-brsu-1/urdf/robot.urdf.xacro (robot description, xacro)
@@ -15,5 +15,6 @@
   <xacro:include filename="$(find youbot_description)/urdf/youbot_arm/arm.urdf.xacro"/>
   <xacro:include filename="$(find mir_description)/urdf/misc/adapter_plate.urdf.xacro" />
-  <xacro:include filename="$(find mir_description)/urdf/grippers/dynamixel/v1/dynamixel_gripper.urdf.xacro" />
+  <!-- youbot gripper -->
+  <xacro:include filename="$(find youbot_description)/urdf/youbot_gripper/gripper.urdf.xacro" />
   <!-- controller manager -->
   <xacro:include filename="$(find youbot_description)/controller/ros_controller.urdf.xacro" />
@@ -45,10 +46,6 @@
      <origin xyz="-0.3 0.0 -0.03" rpy="0 0 ${M_PI}" />
   </xacro:hokuyo_urg04_laser>
-  <!-- 3D camera on arm --> <!-- NOTE: still called arm_cam3d due to legacy code -->
-  <xacro:intel_realsense_f200_camera name="arm_cam3d" parent="arm_link_5">
-    <origin xyz="-0.075 0.024 0.04" rpy="0 ${-M_PI / 2} 0" />
-  </xacro:intel_realsense_f200_camera>
-  <xacro:dynamixel_gripper name="gripper" parent="arm_link_5">
-    <origin xyz="0 0 -0.02" rpy="0 0 0" />
-  </xacro:dynamixel_gripper>
+  <xacro:youbot_gripper name="gripper" parent="arm_link_5">
+    <origin xyz="0 0 0" rpy="0 0 0" />
+  </xacro:youbot_gripper>
 </robot>

Commit message: [youBot 1 gripper simulation] Model of the gripper changed to old version

File: mir_robots/mir_hardware_config/youbot-brsu-1/urdf/robot.urdf.xacro (robot description, xacro)
@@ -3,5 +3,5 @@
        xmlns:controller="http://playerstage.sourceforge.net/gazebo/xmlschema/#controller"
        xmlns:interface="http://playerstage.sourceforge.net/gazebo/xmlschema/#interface"
-       xmlns:xacro="http://playerstage.sourceforge.net/gazebo/xmlschema/#interface"
+       xmlns:xacro="http://ros.org/wiki/xacro"
        name="youbot" >
   <!-- The following included files set up definitions of parts of the robot body -->
@@ -15,5 +15,6 @@
   <xacro:include filename="$(find youbot_description)/urdf/youbot_arm/arm.urdf.xacro"/>
   <xacro:include filename="$(find mir_description)/urdf/misc/adapter_plate.urdf.xacro" />
-  <xacro:include filename="$(find mir_description)/urdf/grippers/dynamixel/v1/dynamixel_gripper.urdf.xacro" />
+  <!-- youbot gripper -->
+  <xacro:include filename="$(find youbot_description)/urdf/youbot_gripper/gripper.urdf.xacro" />
   <!-- controller manager -->
   <xacro:include filename="$(find youbot_description)/controller/ros_controller.urdf.xacro" />
@@ -45,10 +46,6 @@
      <origin xyz="-0.3 0.0 -0.03" rpy="0 0 ${M_PI}" />
   </xacro:hokuyo_urg04_laser>
-  <!-- 3D camera on arm --> <!-- NOTE: still called arm_cam3d due to legacy code -->
-  <xacro:intel_realsense_f200_camera name="arm_cam3d" parent="arm_link_5">
-    <origin xyz="-0.075 0.024 0.04" rpy="0 ${-M_PI / 2} 0" />
-  </xacro:intel_realsense_f200_camera>
-  <xacro:dynamixel_gripper name="gripper" parent="arm_link_5">
-    <origin xyz="0 0 -0.02" rpy="0 0 0" />
-  </xacro:dynamixel_gripper>
+  <xacro:youbot_gripper name="gripper" parent="arm_link_5">
+    <origin xyz="0 0 0" rpy="0 0 0" />
+  </xacro:youbot_gripper>
 </robot>
