Commit message: Corrected position of camera mount and camera

File: mir_common/mir_description/urdf/grippers/dynamixel/d435_center/dynamixel_gripper.urdf.xacro (robot description, xacro)
@@ -17,4 +17,7 @@
       <child link="${name}_motor_mount_link" />
     </joint>
+    <material name="black">
+        <color rgba="0 0 0 1"/>
+    </material>
     <!-- motor mount -->
     <link name="${name}_motor_mount_link">
@@ -25,11 +28,12 @@
       </inertial>
       <visual>
-        <origin xyz="0 0 -0.0275" rpy="0 ${M_PI/2} 0" />
+        <origin xyz="-0.029 -0.046 0.0185" rpy="0 ${M_PI/2} 0" />
         <geometry>
           <mesh filename="package://mir_description/meshes/grippers/dynamixel/d435_center/dynamixel_motor_mount.stl" scale="0.001 0.001 0.001" />
         </geometry>
+        <material name="black"/>
       </visual>
       <collision>
-        <origin xyz="0 0 -0.0275" rpy="0 ${M_PI/2} 0" />
+        <origin xyz="-0.029 -0.046 0.0185" rpy="0 ${M_PI/2} 0" />
         <geometry>
           <mesh filename="package://mir_description/meshes/grippers/dynamixel/d435_center/dynamixel_motor_mount_convex_hull.dae" scale="0.001 0.001 0.001" />

File: mir_robots/mir_hardware_config/youbot-brsu-4/urdf/robot.urdf.xacro (robot description, xacro)
@@ -73,5 +73,5 @@
    </xacro:sensor_d435>
    <xacro:sensor_d435  name="d435_arm" parent="arm_link_5">
-       <origin xyz="0.0 0.0 -0.005" rpy="0.0 ${-M_PI / 2} ${-M_PI / 2}" />
+       <origin xyz="0.0 -0.011 0.009" rpy="0.0 ${-M_PI / 2} ${-M_PI / 2}" />
    </xacro:sensor_d435>
 </robot>

Commit message: Corrected collision block for gripper mount

File: mir_common/mir_description/urdf/grippers/dynamixel/d435_center/dynamixel_gripper.urdf.xacro (robot description, xacro)
@@ -37,5 +37,5 @@
         <origin xyz="-0.029 -0.046 0.0185" rpy="0 ${M_PI/2} 0" />
         <geometry>
-          <mesh filename="package://mir_description/meshes/grippers/dynamixel/d435_center/dynamixel_motor_mount_convex_hull.dae" scale="0.001 0.001 0.001" />
+          <mesh filename="package://mir_description/meshes/grippers/dynamixel/d435_center/dynamixel_motor_mount.stl" scale="0.001 0.001 0.001" />
         </geometry>
       </collision>

Commit message: [sciroc 2019] Changes from sciroc competition

File: mir_common/mir_description/urdf/grippers/dynamixel/d435_center/dynamixel_gripper.urdf.xacro (robot description, xacro)
@@ -16,4 +16,9 @@
       <parent link="${parent}" />
       <child link="${name}_motor_mount_link" />
+    </joint>
+    <joint name="${name}_static_grasp_link_joint" type="fixed" >
+        <origin xyz="0 0 0.08" rpy="0 0 0"/>
+      <parent link="${parent}" />
+      <child link="${name}_static_grasp_link" />
     </joint>
     <material name="black">
@@ -38,4 +43,22 @@
         <geometry>
           <mesh filename="package://mir_description/meshes/grippers/dynamixel/d435_center/dynamixel_motor_mount.stl" scale="0.001 0.001 0.001" />
+        </geometry>
+      </collision>
+    </link>
+    <link name="${name}_static_grasp_link">
+      <inertial>
+        <origin xyz="0 0 0" rpy="0 0 0"/>
+        <mass value="0.038"/>
+        <inertia ixx="0.01" ixy="0" ixz="0" iyy="0.01" iyz="0" izz="0.01" />
+      </inertial>
+      <visual>
+        <geometry>
+            <cylinder length="0.01" radius="0.001"/>
+        </geometry>
+        <material name="black"/>
+      </visual>
+      <collision>
+        <geometry>
+            <cylinder length="0.01" radius="0.001"/>
         </geometry>
       </collision>

Commit message: [sciroc-2019] Added variable for grasp link

File: mir_common/mir_description/urdf/grippers/dynamixel/d435_center/dynamixel_gripper.urdf.xacro (robot description, xacro)
@@ -11,4 +11,5 @@
   <xacro:include filename="$(find mir_description)/urdf/grippers/dynamixel/d435_center/festo_finger_mount.urdf.xacro" />
   <xacro:include filename="$(find mcr_description)/urdf/fingers/festo_finger_dhas-gf-shm.urdf.xacro" />
+  <xacro:arg name="grasp_link_offset" default="0.08"/>
   <xacro:macro name="dynamixel_gripper_d435_center" params="parent name *origin">
     <joint name="${name}_motor_mount_joint" type="fixed" >
@@ -18,5 +19,5 @@
     </joint>
     <joint name="${name}_static_grasp_link_joint" type="fixed" >
-        <origin xyz="0 0 0.08" rpy="0 0 0"/>
+        <origin xyz="0 0 $(arg grasp_link_offset)" rpy="0 0 0"/>
       <parent link="${parent}" />
       <child link="${name}_static_grasp_link" />

Commit message: [description] remove inertial, visual and collision tags for static grasp link of gripper This removes the tiny cylinder visible in the robot model.

File: mir_common/mir_description/urdf/grippers/dynamixel/d435_center/dynamixel_gripper.urdf.xacro (robot description, xacro)
@@ -48,20 +48,4 @@
     </link>
     <link name="${name}_static_grasp_link">
-      <inertial>
-        <origin xyz="0 0 0" rpy="0 0 0"/>
-        <mass value="0.038"/>
-        <inertia ixx="0.01" ixy="0" ixz="0" iyy="0.01" iyz="0" izz="0.01" />
-      </inertial>
-      <visual>
-        <geometry>
-            <cylinder length="0.01" radius="0.001"/>
-        </geometry>
-        <material name="black"/>
-      </visual>
-      <collision>
-        <geometry>
-            <cylinder length="0.01" radius="0.001"/>
-        </geometry>
-      </collision>
     </link>
     <!-- motors -->
