Commit message: Youbot 4 Manipulation URDF Changes
- Attaches arm to adapter_plate, rotated 45 degrees
- Uses Standard YB Gripper

File: mir_robots/mir_hardware_config/youbot-brsu-4/urdf/robot.urdf.xacro (robot description, xacro)
@@ -35,16 +35,18 @@
     <origin xyz="-0.159 0 0.046" rpy="0 0 0" />
   </xacro:youbot_plate>
-  <xacro:youbot_arm name="arm" parent="base_link">
-    <origin xyz="0.223 0.017 0.088" rpy="0 0 ${-M_PI / 4}" />
+  <!-- BRSU SPECIFIC STUFF -->
+  <xacro:include filename="$(find mcr_description)/urdf/materials.urdf.xacro" />
+  <xacro:include filename="$(find mir_description)/urdf/misc/adapter_plate.urdf.xacro" />
+  <!-- Arm Plate moving arm 8cm foward and 45 degree rotation -->
+  <xacro:adapter_plate name="adapter_plate" parent="base_link" arm_angle="${M_PI / 4}">
+    <origin xyz="${0.159+0.08} 0 0.051" rpy="0 0 0" />
+  </xacro:adapter_plate>
+  <xacro:youbot_arm name="arm" parent="adapter_plate_arm_root_link">
+    <origin xyz="-0.022 0.0 0.037" rpy="0 0 0" />
   </xacro:youbot_arm>
+  <!-- Standard YB Gripper -->
   <xacro:youbot_gripper name="gripper" parent="arm_link_5">
     <origin xyz="0 0 0" rpy="0 0 0" />
   </xacro:youbot_gripper>
-  <!-- BRSU SPECIFIC STUFF -->
-  <xacro:include filename="$(find mcr_description)/urdf/materials.urdf.xacro" />
-  <xacro:include filename="$(find mir_description)/urdf/misc/adapter_plate.urdf.xacro" />
-  <xacro:adapter_plate name="adapter_plate" parent="base_link">
-    <origin xyz="${0.159+0.08} 0 0.051" rpy="0 0 0" />
-  </xacro:adapter_plate>
   <!-- base laser front -->
   <xacro:hokuyo_urg04_laser name="base_laser_front" parent="base" ros_topic="scan_front" update_rate="10" min_angle="-1.57" max_angle="1.57">

Commit message: Youbot 4 with BRSU rear platform

File: mir_robots/mir_hardware_config/youbot-brsu-4/urdf/robot.urdf.xacro (robot description, xacro)
@@ -32,10 +32,12 @@
   <!-- foot for arm-->
   <xacro:youbot_base name="base"/>
-  <xacro:youbot_plate name="plate" parent="base_link">
-    <origin xyz="-0.159 0 0.046" rpy="0 0 0" />
-  </xacro:youbot_plate>
   <!-- BRSU SPECIFIC STUFF -->
   <xacro:include filename="$(find mcr_description)/urdf/materials.urdf.xacro" />
+  <xacro:include filename="$(find mir_description)/urdf/misc/rear_platform.urdf.xacro" />
   <xacro:include filename="$(find mir_description)/urdf/misc/adapter_plate.urdf.xacro" />
+  <!-- Rear Platform -->
+  <xacro:rear_platform name="rear_platform" parent="base_link">
+    <origin xyz="-0.005 -0.175 0.051" rpy="0 0 0" />
+  </xacro:rear_platform>
   <!-- Arm Plate moving arm 8cm foward and 45 degree rotation -->
   <xacro:adapter_plate name="adapter_plate" parent="base_link" arm_angle="${M_PI / 4}">

Commit message: Youbot 4 with 3d sensor and tower

File: mir_robots/mir_hardware_config/youbot-brsu-4/urdf/robot.urdf.xacro (robot description, xacro)
@@ -34,4 +34,6 @@
   <!-- BRSU SPECIFIC STUFF -->
   <xacro:include filename="$(find mcr_description)/urdf/materials.urdf.xacro" />
+  <xacro:include filename="$(find mir_description)/urdf/misc/cam3d_tower.urdf.xacro"/>
+  <xacro:include filename="$(find mcr_description)/urdf/sensors/asus_xtion_camera.urdf.xacro"/>
   <xacro:include filename="$(find mir_description)/urdf/misc/rear_platform.urdf.xacro" />
   <xacro:include filename="$(find mir_description)/urdf/misc/adapter_plate.urdf.xacro" />
@@ -59,3 +61,11 @@
      <origin xyz="-0.3 0 -0.03" rpy="0 0 ${M_PI}" />
   </xacro:hokuyo_urg04_laser>
+  <!-- camera tower -->
+  <xacro:cam3d_tower name="camera_tower" parent="rear_platform_link">
+    <origin xyz="-0.227 0.165 0.023" rpy="0 0 0" />
+  </xacro:cam3d_tower>
+  <!-- 3D camera on tower -->
+  <xacro:asus_xtion_camera name="tower_cam3d" parent="camera_tower_link" tilt="0.5">
+    <origin xyz="0.015 0 0.47" rpy="0 0 0" />
+  </xacro:asus_xtion_camera>
 </robot>

Commit message: Youbot 4 with arm POV camera

File: mir_robots/mir_hardware_config/youbot-brsu-4/urdf/robot.urdf.xacro (robot description, xacro)
@@ -36,4 +36,5 @@
   <xacro:include filename="$(find mir_description)/urdf/misc/cam3d_tower.urdf.xacro"/>
   <xacro:include filename="$(find mcr_description)/urdf/sensors/asus_xtion_camera.urdf.xacro"/>
+  <xacro:include filename="$(find mcr_description)/urdf/mounts/microsoft_lifecam_1080_mount.urdf.xacro"/>
   <xacro:include filename="$(find mir_description)/urdf/misc/rear_platform.urdf.xacro" />
   <xacro:include filename="$(find mir_description)/urdf/misc/adapter_plate.urdf.xacro" />
@@ -69,3 +70,7 @@
     <origin xyz="0.015 0 0.47" rpy="0 0 0" />
   </xacro:asus_xtion_camera>
+  <!-- Arm POV Mount -->
+  <xacro:microsoft_lifecam_1080_mount name="microsoft_lifecam_1080_mount" parent="arm_link_5">
+    <origin xyz="-0.035 0.0 -0.025" rpy="0 0 3.14159265" />
+  </xacro:microsoft_lifecam_1080_mount>
 </robot>

Commit message: [hardware config] use config from yb5 + calibrate intel cam pose

File: mir_robots/mir_hardware_config/youbot-brsu-4/urdf/robot.urdf.xacro (robot description, xacro)
@@ -11,9 +11,9 @@
   <!-- youbot base and rear platform -->
   <xacro:include filename="$(find youbot_description)/urdf/youbot_base/base.urdf.xacro" />
-  <xacro:include filename="$(find mir_description)/urdf/misc/rear_platform.urdf.xacro" />
+  <xacro:include filename="$(find mir_description)/urdf/misc/rear_platform_v2.urdf.xacro" />
   <!-- youbot arm and gripper-->
   <xacro:include filename="$(find youbot_description)/urdf/youbot_arm/arm.urdf.xacro"/>
   <xacro:include filename="$(find mir_description)/urdf/misc/adapter_plate.urdf.xacro" />
-  <xacro:include filename="$(find mir_description)/urdf/grippers/festo_gripper.urdf.xacro" />
+  <xacro:include filename="$(find mir_description)/urdf/grippers/dynamixel/v2/dynamixel_gripper.urdf.xacro" />
   <!-- controller manager -->
   <xacro:include filename="$(find youbot_description)/controller/ros_controller.urdf.xacro" />
@@ -22,15 +22,16 @@
   <!-- sensors -->
   <xacro:include filename="$(find youbot_description)/urdf/sensors/hokuyo_urg04_laser.urdf.xacro"/>
-  <xacro:include filename="$(find mcr_description)/urdf/sensors/asus_xtion_camera.urdf.xacro"/>
+  <xacro:include filename="$(find mir_description)/urdf/sensor_mounts/intel_f200_camera_mount.urdf.xacro"/>
+  <xacro:include filename="$(find mcr_description)/urdf/sensors/intel_realsense_f200_camera.urdf.xacro"/>
   <!-- Now we can start using the macros included above to define the actual youbot -->
   <!-- standard youBot configuration -->
   <xacro:youbot_base name="base"/>
   <!-- Rear Platform -->
-  <xacro:rear_platform name="rear_platform" parent="base_link">
-    <origin xyz="-0.005 -0.175 0.051" rpy="0 0 0" />
-  </xacro:rear_platform>
+  <xacro:rear_platform_v2 name="rear_platform" parent="base_link">
+    <origin xyz="0.12 -0.175 ${0.021 + 0.0062 + 0.025 + 0.012}" rpy="0 0 0" />  <!-- ${alignment with base top + nut height + spacer height + slide height } -->
+  </xacro:rear_platform_v2>
   <!-- Arm Plate moving arm 8cm foward and 45 degree rotation -->
   <xacro:adapter_plate name="adapter_plate" parent="base_link" arm_angle="${-M_PI / 4}">
-    <origin xyz="${0.159+0.08} 0 0.051" rpy="0 0 0" />
+    <origin xyz="${0.159+0.08} 0 ${0.021 + 0.025 + 0.025}" rpy="0 0 0" />    <!-- ${alignment with base top + spacer height + spacer height } -->
   </xacro:adapter_plate>
   <xacro:youbot_arm name="arm" parent="adapter_plate_arm_root_link">
@@ -39,16 +40,20 @@
   <!-- base laser front -->
   <xacro:hokuyo_urg04_laser name="base_laser_front" parent="base" ros_topic="scan_front" update_rate="10" min_angle="-1.57" max_angle="1.57">
-    <origin xyz="0.3 0 -0.03" rpy="0 0 0"/>
+    <origin xyz="0.3 0 -0.035" rpy="${M_PI} 0 0"/>
   </xacro:hokuyo_urg04_laser>
   <!-- base laser rear -->
   <xacro:hokuyo_urg04_laser name="base_laser_rear" parent="base" ros_topic="scan_rear" update_rate="10" min_angle="-1.57" max_angle="1.57" >
-     <origin xyz="-0.3 0.0 -0.03" rpy="0 0 ${M_PI}" />
+     <origin xyz="-0.3 0.0 -0.035" rpy="${M_PI} 0 ${M_PI}" />
   </xacro:hokuyo_urg04_laser>
-  <!-- 3D camera on arm --> <!-- NOTE: still called arm_cam3d due to legacy code -->
-  <xacro:asus_xtion_camera name="arm_cam3d" parent="arm_link_5" tilt="0.0">
-    <origin xyz="${-0.035 - 0.030 + 0.030} ${0 - 0.015} ${-0.09}" rpy="0 ${-M_PI / 2} 0" />
-  </xacro:asus_xtion_camera>
-  <xacro:festo_gripper name="gripper" parent="arm_link_5">
-    <origin xyz="0 0 0" rpy="0 0 0" />
-  </xacro:festo_gripper>
+  <xacro:dynamixel_gripper_v2 name="gripper" parent="arm_link_5">
+    <origin xyz="0.003 0 0.0052" rpy="0 0 0" />
+  </xacro:dynamixel_gripper_v2>
+  <!-- camera mount for Intel RealSense F200 -->
+  <xacro:intel_f200_camera_mount name="camera_mount" parent="gripper_motor_mount_link">
+    <origin xyz="-0.00375 -0.0007 0.012" rpy="-0.05 -0.04 0" />
+  </xacro:intel_f200_camera_mount>
+  <!-- 3D camera on arm -->
+  <xacro:intel_realsense_f200_camera name="arm_cam3d" parent="camera_mount_link">
+    <origin xyz="-0.0405 0.0 0.029" rpy="0 -${M_PI/2} 0" />
+  </xacro:intel_realsense_f200_camera>
 </robot>

Commit message: [hardware config] calibrate intel cam3d pose

File: mir_robots/mir_hardware_config/youbot-brsu-4/urdf/robot.urdf.xacro (robot description, xacro)
@@ -55,5 +55,5 @@
   <!-- 3D camera on arm -->
   <xacro:intel_realsense_f200_camera name="arm_cam3d" parent="camera_mount_link">
-    <origin xyz="-0.0405 0.0 0.029" rpy="0 -${M_PI/2} 0" />
+    <origin xyz="-0.0405 -0.008 0.025" rpy="-0.2 -${M_PI/2} 0" />
   </xacro:intel_realsense_f200_camera>
 </robot>

Commit message: [urdf] camera calibration

File: mir_robots/mir_hardware_config/youbot-brsu-4/urdf/robot.urdf.xacro (robot description, xacro)
@@ -55,5 +55,5 @@
   <!-- 3D camera on arm -->
   <xacro:intel_realsense_f200_camera name="arm_cam3d" parent="camera_mount_link">
-    <origin xyz="-0.05 -0.03 0.03" rpy="0.3 -${M_PI/2 - 0.03} -0.25" />
+    <origin xyz="-0.03 0.0 0.03" rpy="0.3 -${M_PI/2 - 0.03} -0.2" />
   </xacro:intel_realsense_f200_camera>
 </robot>

Commit message: [yb4 urdf] camera calibration

File: mir_robots/mir_hardware_config/youbot-brsu-4/urdf/robot.urdf.xacro (robot description, xacro)
@@ -55,5 +55,5 @@
   <!-- 3D camera on arm -->
   <xacro:intel_realsense_f200_camera name="arm_cam3d" parent="camera_mount_link">
-    <origin xyz="-0.05 0.0 0.03" rpy="0.0 -${M_PI/2 - 0.03} 0.0" />
+    <origin xyz="-0.05 0.01 0.03" rpy="0.0 -${M_PI/2 - 0.03} 0.0" />
   </xacro:intel_realsense_f200_camera>
 </robot>

Commit message: [urdf] use asus camera instead of intel realsense

File: mir_robots/mir_hardware_config/youbot-brsu-4/urdf/robot.urdf.xacro (robot description, xacro)
@@ -23,5 +23,6 @@
   <xacro:include filename="$(find youbot_description)/urdf/sensors/hokuyo_urg04_laser.urdf.xacro"/>
   <xacro:include filename="$(find mir_description)/urdf/sensor_mounts/intel_f200_camera_mount.urdf.xacro"/>
-  <xacro:include filename="$(find mcr_description)/urdf/sensors/intel_realsense_f200_camera.urdf.xacro"/>
+  <!--xacro:include filename="$(find mcr_description)/urdf/sensors/intel_realsense_f200_camera.urdf.xacro"/-->
+  <xacro:include filename="$(find mcr_description)/urdf/sensors/asus_xtion_camera.urdf.xacro"/>
   <!-- Now we can start using the macros included above to define the actual youbot -->
   <!-- standard youBot configuration -->
@@ -50,10 +51,15 @@
   </xacro:dynamixel_gripper_v2>
   <!-- camera mount for Intel RealSense F200 -->
-  <xacro:intel_f200_camera_mount name="camera_mount" parent="gripper_motor_mount_link">
-    <origin xyz="-0.00375 -0.0007 0.012" rpy="0.04 -0.04 0" />
-  </xacro:intel_f200_camera_mount>
+  <!--xacro:intel_f200_camera_mount name="camera_mount" parent="gripper_motor_mount_link">
+    <origin xyz="-0.00375 -0.0007 0.012" rpy="0.0 -0.04 0.00" />
+  </xacro:intel_f200_camera_mount-->
   <!-- 3D camera on arm -->
-  <xacro:intel_realsense_f200_camera name="arm_cam3d" parent="camera_mount_link">
-    <origin xyz="-0.05 0.01 0.03" rpy="0.0 -${M_PI/2 - 0.03} 0.0" />
-  </xacro:intel_realsense_f200_camera>
+  <!--xacro:intel_realsense_f200_camera name="arm_cam3d" parent="camera_mount_link">
+    <origin xyz="-0.05 -0.01 0.03" rpy="0.0 -${M_PI/2 - 0.03} 0.0" />
+  </xacro:intel_realsense_f200_camera-->
+   <xacro:asus_xtion_camera name="arm_cam3d" parent="gripper_motor_mount_link" tilt="-0.0">
+       <!--origin xyz="-0.01 -0.012 0.05" rpy="0 ${M_PI/2 - 0.25} 0.00" /-->
+       <!--<origin xyz="0.016 0 0.01" rpy="0 ${M_PI/2 - 0} -0.09" />  -->
+       <origin xyz="0.05 -0.00 0.015" rpy="0 ${M_PI/2 - 0} -0.07" />
+   </xacro:asus_xtion_camera>
 </robot>

Commit message: [wbc] integration updates

File: mir_robots/mir_hardware_config/youbot-brsu-4/urdf/robot.urdf.xacro (robot description, xacro)
@@ -61,5 +61,5 @@
        <!--origin xyz="-0.01 -0.012 0.05" rpy="0 ${M_PI/2 - 0.25} 0.00" /-->
        <!--<origin xyz="0.016 0 0.01" rpy="0 ${M_PI/2 - 0} -0.09" />  -->
-       <origin xyz="0.05 -0.00 0.015" rpy="0 ${M_PI/2 - 0} -0.07" />
+       <origin xyz="0.05 -0.00 0.015" rpy="0 ${M_PI/2 - 0.001} -0.00" />
    </xacro:asus_xtion_camera>
 </robot>

Commit message: camera calib

File: mir_robots/mir_hardware_config/youbot-brsu-4/urdf/robot.urdf.xacro (robot description, xacro)
@@ -61,5 +61,5 @@
        <!--origin xyz="-0.01 -0.012 0.05" rpy="0 ${M_PI/2 - 0.25} 0.00" /-->
        <!--<origin xyz="0.016 0 0.01" rpy="0 ${M_PI/2 - 0} -0.09" />  -->
-       <origin xyz="0.05 -0.00 0.015" rpy="0 ${M_PI/2 - 0.001} -0.00" />
+       <origin xyz="0.05 -0.00 0.015" rpy="0 ${M_PI/2 - 0.02} -0.00" />
    </xacro:asus_xtion_camera>
 </robot>

Commit message: [yb4 urdf] camera calib

File: mir_robots/mir_hardware_config/youbot-brsu-4/urdf/robot.urdf.xacro (robot description, xacro)
@@ -61,5 +61,5 @@
        <!--origin xyz="-0.01 -0.012 0.05" rpy="0 ${M_PI/2 - 0.25} 0.00" /-->
        <!--<origin xyz="0.016 0 0.01" rpy="0 ${M_PI/2 - 0} -0.09" />  -->
-       <origin xyz="0.05 -0.00 0.015" rpy="0 ${M_PI/2 - 0.02} -0.00" />
+       <origin xyz="0.05 0.01 0.015" rpy="0 ${M_PI/2 - 0.02} -0.00" />
    </xacro:asus_xtion_camera>
 </robot>

Commit message: [integration] kinetic integration test bugfixes

File: mir_robots/mir_hardware_config/youbot-brsu-4/urdf/robot.urdf.xacro (robot description, xacro)
@@ -61,5 +61,5 @@
        <!--origin xyz="-0.01 -0.012 0.05" rpy="0 ${M_PI/2 - 0.25} 0.00" /-->
        <!--<origin xyz="0.016 0 0.01" rpy="0 ${M_PI/2 - 0} -0.09" />  -->
-       <origin xyz="0.05 -0.00 0.015" rpy="0 ${M_PI/2 - 0} -0.07" />
+       <origin xyz="0.05 -0.00 0.040" rpy="-0.05 ${M_PI/2 - 0.178} -0.07" />
    </xacro:asus_xtion_camera>
 </robot>

Commit message: [camera mount] Adding new asus camera mount

File: mir_robots/mir_hardware_config/youbot-brsu-4/urdf/robot.urdf.xacro (robot description, xacro)
@@ -23,6 +23,7 @@
   <xacro:include filename="$(find youbot_description)/urdf/sensors/hokuyo_urg04_laser.urdf.xacro"/>
   <xacro:include filename="$(find mir_description)/urdf/sensor_mounts/intel_f200_camera_mount.urdf.xacro"/>
-  <!--xacro:include filename="$(find mcr_description)/urdf/sensors/intel_realsense_f200_camera.urdf.xacro"/-->
-  <xacro:include filename="$(find mcr_description)/urdf/sensors/asus_xtion_camera.urdf.xacro"/>
+  <xacro:include filename="$(find mcr_description)/urdf/sensors/intel_realsense_f200_camera.urdf.xacro"/>
+  <xacro:include filename="$(find mir_description)/urdf/sensors/asus_xtion_camera.urdf.xacro"/>
+  <xacro:include filename="$(find mir_description)/urdf/sensor_mounts/asus_xtion_camera_mount.urdf.xacro"/>
   <!-- Now we can start using the macros included above to define the actual youbot -->
   <!-- standard youBot configuration -->
@@ -51,15 +52,15 @@
   </xacro:dynamixel_gripper_v2>
   <!-- camera mount for Intel RealSense F200 -->
-  <!--xacro:intel_f200_camera_mount name="camera_mount" parent="gripper_motor_mount_link">
-    <origin xyz="-0.00375 -0.0007 0.012" rpy="0.0 -0.04 0.00" />
-  </xacro:intel_f200_camera_mount-->
+  <xacro:asus_xtion_camera_mount  name="camera_mount" parent="gripper_motor_mount_link">
+    <origin xyz="0.035 -0.00 0.0" rpy="-${M_PI/2} 0 0 " />
+  </xacro:asus_xtion_camera_mount>
   <!-- 3D camera on arm -->
-  <!--xacro:intel_realsense_f200_camera name="arm_cam3d" parent="camera_mount_link">
+  <!-- xacro:intel_realsense_f200_camera name="arm_cam3d" parent="camera_mount_link">
     <origin xyz="-0.05 -0.01 0.03" rpy="0.0 -${M_PI/2 - 0.03} 0.0" />
-  </xacro:intel_realsense_f200_camera-->
-   <xacro:asus_xtion_camera name="arm_cam3d" parent="gripper_motor_mount_link" tilt="-0.0">
+  </xacro:intel_realsense_f200_camera -->
+   <xacro:asus_xtion_camera name="arm_cam3d" parent="camera_mount_link">
        <!--origin xyz="-0.01 -0.012 0.05" rpy="0 ${M_PI/2 - 0.25} 0.00" /-->
-       <!--<origin xyz="0.016 0 0.01" rpy="0 ${M_PI/2 - 0} -0.09" />  -->
-       <origin xyz="0.05 -0.00 0.015" rpy="0 ${M_PI/2 - 0} -0.07" />
+       <!--origin xyz="0.016 0 0.01" rpy="0 ${M_PI/2 - 0} -0.09" />  -->
+       <origin xyz="0.023 -0.015 0.03" rpy="${M_PI/2} 0 ${M_PI/2 - 0.17}" />
    </xacro:asus_xtion_camera>
 </robot>

Commit message: [Camera Mount] Fixed the position

File: mir_robots/mir_hardware_config/youbot-brsu-4/urdf/robot.urdf.xacro (robot description, xacro)
@@ -53,5 +53,5 @@
   <!-- camera mount for Intel RealSense F200 -->
   <xacro:asus_xtion_camera_mount  name="camera_mount" parent="gripper_motor_mount_link">
-    <origin xyz="0.035 -0.00 0.0" rpy="-${M_PI/2} 0 0 " />
+      <origin xyz="0.035 -0.00 0.0" rpy="0 0.025 ${M_PI/2} " />
   </xacro:asus_xtion_camera_mount>
   <!-- 3D camera on arm -->
@@ -62,5 +62,6 @@
        <!--origin xyz="-0.01 -0.012 0.05" rpy="0 ${M_PI/2 - 0.25} 0.00" /-->
        <!--origin xyz="0.016 0 0.01" rpy="0 ${M_PI/2 - 0} -0.09" />  -->
-       <origin xyz="0.023 -0.015 0.03" rpy="${M_PI/2} 0 ${M_PI/2 - 0.17}" />
+   <origin xyz="0.010 -0.022 0.017" rpy="0 ${M_PI/2 - 0.18} -${M_PI/2}" />
+       <!--origin xyz="0.023 -0.015 0.03" rpy="0 0 0" /-->
    </xacro:asus_xtion_camera>
 </robot>

Commit message: [Camera calibration and gripper conf]

File: mir_robots/mir_hardware_config/youbot-brsu-4/urdf/robot.urdf.xacro (robot description, xacro)
@@ -62,5 +62,5 @@
        <!--origin xyz="-0.01 -0.012 0.05" rpy="0 ${M_PI/2 - 0.25} 0.00" /-->
        <!--origin xyz="0.016 0 0.01" rpy="0 ${M_PI/2 - 0} -0.09" />  -->
-   <origin xyz="0.010 -0.022 0.017" rpy="0 ${M_PI/2 - 0.18} -${M_PI/2}" />
+       <origin xyz="0.010 -0.015 0.017" rpy="0 ${M_PI/2 - 0.18} -${M_PI/2}" />
        <!--origin xyz="0.023 -0.015 0.03" rpy="0 0 0" /-->
    </xacro:asus_xtion_camera>

Commit message: [yb4 camera calib] camera calibration montreal 2018

File: mir_robots/mir_hardware_config/youbot-brsu-4/urdf/robot.urdf.xacro (robot description, xacro)
@@ -53,5 +53,5 @@
   <!-- camera mount for Intel RealSense F200 -->
   <xacro:asus_xtion_camera_mount  name="camera_mount" parent="gripper_motor_mount_link">
-      <origin xyz="0.035 -0.00 0.0" rpy="0 0.025 ${M_PI/2} " />
+      <origin xyz="0.020 -0.00 0.0" rpy="0 0.025 ${M_PI/2} " />
   </xacro:asus_xtion_camera_mount>
   <!-- 3D camera on arm -->
@@ -62,5 +62,5 @@
        <!--origin xyz="-0.01 -0.012 0.05" rpy="0 ${M_PI/2 - 0.25} 0.00" /-->
        <!--origin xyz="0.016 0 0.01" rpy="0 ${M_PI/2 - 0} -0.09" />  -->
-       <origin xyz="0.010 -0.015 0.017" rpy="0 ${M_PI/2 - 0.18} -${M_PI/2}" />
+       <origin xyz="0.025 -0.010 0.017" rpy="0.02 ${M_PI/2 - 0.20} -${M_PI/2}" />
        <!--origin xyz="0.023 -0.015 0.03" rpy="0 0 0" /-->
    </xacro:asus_xtion_camera>

Commit message: camera calibration for yb4

File: mir_robots/mir_hardware_config/youbot-brsu-4/urdf/robot.urdf.xacro (robot description, xacro)
@@ -62,5 +62,7 @@
        <!--origin xyz="-0.01 -0.012 0.05" rpy="0 ${M_PI/2 - 0.25} 0.00" /-->
        <!--origin xyz="0.016 0 0.01" rpy="0 ${M_PI/2 - 0} -0.09" />  -->
-       <origin xyz="0.025 -0.010 0.017" rpy="0.02 ${M_PI/2 - 0.20} -${M_PI/2}" />
+       <origin xyz="0.025 -0.013 0.017" rpy="0.02 ${M_PI/2 - 0.20} -${M_PI/2}" />
+       <!-- <origin xyz="0.022 -0.0 0.017" rpy="0.02 ${M_PI/2 - 0.20} -${M_PI/2}" /> -->
+       <!-- <origin xyz="0.025 -0.010 0.017" rpy="0.02 ${M_PI/2 - 0.20} -${M_PI/2}" /> -->
        <!--origin xyz="0.023 -0.015 0.03" rpy="0 0 0" /-->
    </xacro:asus_xtion_camera>

Commit message: integrated intel realsense d435 urdf

File: mir_robots/mir_hardware_config/youbot-brsu-4/urdf/robot.urdf.xacro (robot description, xacro)
@@ -25,4 +25,5 @@
   <xacro:include filename="$(find mcr_description)/urdf/sensors/intel_realsense_f200_camera.urdf.xacro"/>
   <xacro:include filename="$(find mir_description)/urdf/sensors/asus_xtion_camera.urdf.xacro"/>
+  <xacro:include filename="$(find mir_description)/urdf/sensors/_d435.urdf.xacro"/>
   <xacro:include filename="$(find mir_description)/urdf/sensor_mounts/asus_xtion_camera_mount.urdf.xacro"/>
   <!-- Now we can start using the macros included above to define the actual youbot -->
@@ -65,3 +66,9 @@
        <!--origin xyz="0.023 -0.015 0.03" rpy="0 0 0" /-->
    </xacro:asus_xtion_camera>
+   <xacro:sensor_d435  parent="base_link">
+       <!--origin xyz="-0.01 -0.012 0.05" rpy="0 ${M_PI/2 - 0.25} 0.00" /-->
+       <!--origin xyz="0.016 0 0.01" rpy="0 ${M_PI/2 - 0} -0.09" />  -->
+       <origin xyz="-0.263 0.0 0.0875" rpy="0.0 0.61 ${M_PI}" />
+       <!--origin xyz="0.023 -0.015 0.03" rpy="0 0 0" /-->
+   </xacro:sensor_d435>
 </robot>

Commit message: [Sydney-2019] New Camera calibration

File: mir_robots/mir_hardware_config/youbot-brsu-4/urdf/robot.urdf.xacro (robot description, xacro)
@@ -63,5 +63,5 @@
        <!--origin xyz="-0.01 -0.012 0.05" rpy="0 ${M_PI/2 - 0.25} 0.00" /-->
        <!--origin xyz="0.016 0 0.01" rpy="0 ${M_PI/2 - 0} -0.09" />  -->
-       <origin xyz="0.025 -0.013 0.017" rpy="0.02 ${M_PI/2 - 0.20} -${M_PI/2}" />
+       <origin xyz="0.025 -0.012 0.013" rpy="0.02 ${M_PI/2 - 0.20} -${M_PI/2}" />
        <!-- <origin xyz="0.022 -0.0 0.017" rpy="0.02 ${M_PI/2 - 0.20} -${M_PI/2}" /> -->
        <!-- <origin xyz="0.025 -0.010 0.017" rpy="0.02 ${M_PI/2 - 0.20} -${M_PI/2}" /> -->
