Commit message: Rob urdf and SRDF changes
URDF canges for adding the intel camera

SRDF changes for resolving collision avoidance according to new poses
for intel realsense camera

File: mir_robots/mir_hardware_config/youbot-brsu-4/urdf/robot.urdf.xacro (robot description, xacro)
@@ -23,7 +23,7 @@
   <xacro:include filename="$(find youbot_description)/urdf/sensors/hokuyo_urg04_laser.urdf.xacro"/>
   <xacro:include filename="$(find mir_description)/urdf/sensor_mounts/intel_f200_camera_mount.urdf.xacro"/>
-  <xacro:include filename="$(find mcr_description)/urdf/sensors/intel_realsense_f200_camera.urdf.xacro"/>
+  <!--xacro:include filename="$(find mcr_description)/urdf/sensors/intel_realsense_f200_camera.urdf.xacro"/-->
   <xacro:include filename="$(find mir_description)/urdf/sensors/asus_xtion_camera.urdf.xacro"/>
-  <xacro:include filename="$(find mir_description)/urdf/sensors/_d435.urdf.xacro"/>
+  <xacro:include filename="$(find mir_description)/urdf/sensors/d435.urdf.xacro"/>
   <xacro:include filename="$(find mir_description)/urdf/sensor_mounts/asus_xtion_camera_mount.urdf.xacro"/>
   <!-- Now we can start using the macros included above to define the actual youbot -->
@@ -60,16 +60,19 @@
     <origin xyz="-0.05 -0.01 0.03" rpy="0.0 -${M_PI/2 - 0.03} 0.0" />
   </xacro:intel_realsense_f200_camera -->
-   <xacro:asus_xtion_camera name="arm_cam3d" parent="camera_mount_link">
+  <!-- <xacro:asus_xtion_camera name="arm_cam3d" parent="camera_mount_link"-->
        <!--origin xyz="-0.01 -0.012 0.05" rpy="0 ${M_PI/2 - 0.25} 0.00" /-->
        <!--origin xyz="0.016 0 0.01" rpy="0 ${M_PI/2 - 0} -0.09" />  -->
-       <origin xyz="0.025 -0.013 0.017" rpy="0.02 ${M_PI/2 - 0.20} -${M_PI/2}" />
+  <!--     <origin xyz="0.025 -0.012 0.013" rpy="0.02 ${M_PI/2 - 0.20} -${M_PI/2}" /-->
        <!-- <origin xyz="0.022 -0.0 0.017" rpy="0.02 ${M_PI/2 - 0.20} -${M_PI/2}" /> -->
        <!-- <origin xyz="0.025 -0.010 0.017" rpy="0.02 ${M_PI/2 - 0.20} -${M_PI/2}" /> -->
        <!--origin xyz="0.023 -0.015 0.03" rpy="0 0 0" /-->
-   </xacro:asus_xtion_camera>
-   <xacro:sensor_d435  parent="base_link">
+  <!-- </xacro:asus_xtion_camera-->
+   <!--xacro:sensor_d435  name="back_camera" parent="base_link">
+       <origin xyz="-0.263 0.0 0.0875" rpy="0.0 0.61 ${M_PI}" />
+   </xacro:sensor_d435-->
+   <xacro:sensor_d435  name="d435_arm_camera" parent="arm_link_5">
        <!--origin xyz="-0.01 -0.012 0.05" rpy="0 ${M_PI/2 - 0.25} 0.00" /-->
        <!--origin xyz="0.016 0 0.01" rpy="0 ${M_PI/2 - 0} -0.09" />  -->
-       <origin xyz="-0.263 0.0 0.0875" rpy="0.0 0.61 ${M_PI}" />
+       <origin xyz="0.0 0.0 0.0875" rpy="0.0 0.0 ${M_PI}" />
        <!--origin xyz="0.023 -0.015 0.03" rpy="0 0 0" /-->
    </xacro:sensor_d435>

Commit message: [urdf] add fixed camera link; update extrinsic camera calibration
fixed camera link is added because the TF between arm_cam3d_camera_link
and arm_cam3d_camera_depth_optical_frame is not reliable (i.e. the
transform listener will sometimes get a zero TF between those links)

File: mir_robots/mir_hardware_config/youbot-brsu-4/urdf/robot.urdf.xacro (robot description, xacro)
@@ -53,25 +53,28 @@
     <origin xyz="0.003 0 0.0052" rpy="0 0 0" />
   </xacro:dynamixel_gripper_d435_center>
-  <!-- camera mount for Intel RealSense F200 -->
-  <!-- xacro:asus_xtion_camera_mount  name="camera_mount" parent="gripper_motor_mount_link">
-      <origin xyz="0.020 -0.00 0.0" rpy="0 0.025 ${M_PI/2} " />
-  </xacro:asus_xtion_camera_mount -->
-  <!-- 3D camera on arm -->
-  <!-- xacro:intel_realsense_f200_camera name="arm_cam3d" parent="camera_mount_link">
-    <origin xyz="-0.05 -0.01 0.03" rpy="0.0 -${M_PI/2 - 0.03} 0.0" />
-  </xacro:intel_realsense_f200_camera -->
-  <!-- <xacro:asus_xtion_camera name="arm_cam3d" parent="camera_mount_link"-->
-       <!--origin xyz="-0.01 -0.012 0.05" rpy="0 ${M_PI/2 - 0.25} 0.00" /-->
-       <!--origin xyz="0.016 0 0.01" rpy="0 ${M_PI/2 - 0} -0.09" />  -->
-  <!--     <origin xyz="0.025 -0.012 0.013" rpy="0.02 ${M_PI/2 - 0.20} -${M_PI/2}" /-->
-       <!-- <origin xyz="0.022 -0.0 0.017" rpy="0.02 ${M_PI/2 - 0.20} -${M_PI/2}" /> -->
-       <!-- <origin xyz="0.025 -0.010 0.017" rpy="0.02 ${M_PI/2 - 0.20} -${M_PI/2}" /> -->
-       <!--origin xyz="0.023 -0.015 0.03" rpy="0 0 0" /-->
-  <!-- </xacro:asus_xtion_camera-->
    <xacro:realsense_d435  name="d435_back" parent="base_link">
        <origin xyz="-0.263 0.0 0.0875" rpy="0.0 0.61 ${M_PI}" />
    </xacro:realsense_d435>
    <xacro:realsense_d435  name="arm_cam3d" parent="arm_link_5">
-       <origin xyz="0.0 -0.011 0.009" rpy="0.0 ${-M_PI / 2} ${-M_PI / 2}" />
+      <origin xyz="-0.005 -0.008 0.009" rpy="0.0 ${-M_PI / 2} ${-M_PI / 2}" />
    </xacro:realsense_d435>
+   <joint name="fixed_camera_joint" type="fixed">
+       <origin xyz="0.0149 0.0325 0.0125" rpy="${-M_PI/2} 0 ${-M_PI/2}" />
+       <parent link="arm_cam3d_camera_link"/>
+       <child link="fixed_camera_link"/>
+   </joint>
+   <!-- we create a fixed link from arm_cam3d_camera_link to
+        arm_cam3d_camera_color_optical_frame. See issue -->
+   <link name="fixed_camera_link">
+       <visual>
+           <geometry>
+               <box size="0.0000001 0.000001 0.000001"/>
+           </geometry>
+       </visual>
+       <collision>
+           <geometry>
+               <box size="0.0000001 0.000001 0.000001"/>
+           </geometry>
+       </collision>
+   </link>
 </robot>

Commit message: [hardware_config][yb4] Fixed gazebo error with size of dummy link

File: mir_robots/mir_hardware_config/youbot-brsu-4/urdf/robot.urdf.xacro (robot description, xacro)
@@ -66,15 +66,4 @@
    <!-- we create a fixed link from arm_cam3d_camera_link to
         arm_cam3d_camera_color_optical_frame. See issue -->
-   <link name="fixed_camera_link">
-       <visual>
-           <geometry>
-               <box size="0.0000001 0.000001 0.000001"/>
-           </geometry>
-       </visual>
-       <collision>
-           <geometry>
-               <box size="0.0000001 0.000001 0.000001"/>
-           </geometry>
-       </collision>
-   </link>
+   <link name="fixed_camera_link"/>
 </robot>
