Commit message: calibrate camera tower position on yb3

File: mir_robots/mir_hardware_config/youbot-brsu-3/urdf/robot.urdf.xacro (robot description, xacro)
@@ -51,5 +51,5 @@
   <!-- camera tower -->
   <xacro:camera_tower name="camera_tower" parent="plate_link">
-    <origin xyz="-0.11 0.0 0.03" rpy="0 0 0" />
+    <origin xyz="-0.075 0.0 0.023" rpy="0 0 0" />
   </xacro:camera_tower>
   <!-- 3D camera on tower -->

Commit message: calibrate ASUS 3D cam on yb3

File: mir_robots/mir_hardware_config/youbot-brsu-3/urdf/robot.urdf.xacro (robot description, xacro)
@@ -47,13 +47,13 @@
   <!-- base laser front -->
   <xacro:hokuyo_urg04_laser name="base_laser_front" parent="base" ros_topic="scan_front" update_rate="10" min_angle="-1.57" max_angle="1.57">
-    <origin xyz="0.3 0 -0.03" rpy="0 0 0"/>
+    <origin xyz="0.3 0 -0.04" rpy="0 0 0"/>
   </xacro:hokuyo_urg04_laser>
   <!-- camera tower -->
   <xacro:camera_tower name="camera_tower" parent="plate_link">
-    <origin xyz="-0.075 0.0 0.023" rpy="0 0 0" />
+    <origin xyz="-0.05 0.0 0.023" rpy="0 0 0" />
   </xacro:camera_tower>
   <!-- 3D camera on tower -->
   <xacro:asus_xtion_camera name="tower_cam3d" parent="camera_tower_link" tilt="0.5">
-    <origin xyz="0 0 0.49" rpy="0 0 0" />
+    <origin xyz="-0.04 0.01 0.445" rpy="0 0 0" />
   </xacro:asus_xtion_camera>
   <!-- base laser rear

Commit message: Update youbot-3 urdf to same as youbot-4 urdf

File: mir_robots/mir_hardware_config/youbot-brsu-3/urdf/robot.urdf.xacro (robot description, xacro)
@@ -32,37 +32,46 @@
   <!-- foot for arm-->
   <xacro:youbot_base name="base"/>
-  <xacro:youbot_plate name="plate" parent="base_link">
-    <origin xyz="-0.159 0 0.046" rpy="0 0 0" />
-  </xacro:youbot_plate>
-  <xacro:youbot_arm name="arm" parent="base_link">
-    <origin xyz="0.223 0.017 0.088" rpy="0 0 ${-M_PI / 4}" />
-  </xacro:youbot_arm>
-  <xacro:youbot_gripper name="gripper" parent="arm_link_5">
-    <origin xyz="0 0 0" rpy="0 0 0" />
-  </xacro:youbot_gripper>
   <!-- BRSU SPECIFIC STUFF -->
   <xacro:include filename="$(find mcr_description)/urdf/materials.urdf.xacro" />
-  <xacro:include filename="$(find youbot_description)/urdf/sensors/asus_xtion_camera.urdf.xacro"/>
-  <xacro:include filename="$(find youbot_description)/urdf/misc/camera_tower.urdf.xacro"/>
+  <xacro:include filename="$(find mir_description)/urdf/misc/cam3d_tower.urdf.xacro"/>
+  <xacro:include filename="$(find mcr_description)/urdf/sensors/asus_xtion_camera.urdf.xacro"/>
+  <xacro:include filename="$(find mcr_description)/urdf/mounts/microsoft_lifecam_1080_mount.urdf.xacro"/>
+  <xacro:include filename="$(find mir_description)/urdf/misc/rear_platform.urdf.xacro" />
   <xacro:include filename="$(find mir_description)/urdf/misc/adapter_plate.urdf.xacro" />
-  <xacro:adapter_plate name="adapter_plate" parent="base_link">
+  <xacro:include filename="$(find mir_description)/urdf/grippers/festo_gripper.urdf.xacro" />
+  <!-- Rear Platform -->
+  <xacro:rear_platform name="rear_platform" parent="base_link">
+    <origin xyz="-0.005 -0.175 0.051" rpy="0 0 0" />
+  </xacro:rear_platform>
+  <!-- Arm Plate moving arm 8cm foward and 45 degree rotation -->
+  <xacro:adapter_plate name="adapter_plate" parent="base_link" arm_angle="${-M_PI / 4}">
     <origin xyz="${0.159+0.08} 0 0.051" rpy="0 0 0" />
   </xacro:adapter_plate>
+  <xacro:youbot_arm name="arm" parent="adapter_plate_arm_root_link">
+    <origin xyz="-0.022 0.0 0.037" rpy="0 0 0" />
+  </xacro:youbot_arm>
+  <!-- Festo Gripper -->
+  <xacro:festo_gripper name="gripper" parent="arm_link_5">
+    <origin xyz="0 0 0" rpy="0 0 0" />
+  </xacro:festo_gripper>
   <!-- base laser front -->
   <xacro:hokuyo_urg04_laser name="base_laser_front" parent="base" ros_topic="scan_front" update_rate="10" min_angle="-1.57" max_angle="1.57">
-    <origin xyz="0.3 0 -0.04" rpy="0 0 0"/>
+    <origin xyz="0.3 0 -0.03" rpy="0 0 0"/>
   </xacro:hokuyo_urg04_laser>
-  <!-- camera tower -->
-  <xacro:camera_tower name="camera_tower" parent="plate_link">
-    <origin xyz="-0.05 0.0 0.023" rpy="0 0 0" />
-  </xacro:camera_tower>
-  <!-- 3D camera on tower -->
-  <xacro:asus_xtion_camera name="tower_cam3d" parent="camera_tower_link" tilt="0.5">
-    <origin xyz="-0.04 0.01 0.445" rpy="0 0 0" />
-  </xacro:asus_xtion_camera>
-  <!-- base laser rear
+  <!-- base laser rear -->
   <xacro:hokuyo_urg04_laser name="base_laser_rear" parent="base" ros_topic="scan_rear" update_rate="10" min_angle="-1.57" max_angle="1.57" >
      <origin xyz="-0.3 0 -0.03" rpy="0 0 ${M_PI}" />
   </xacro:hokuyo_urg04_laser>
-  -->
+  <!-- camera tower -->
+  <xacro:cam3d_tower name="camera_tower" parent="rear_platform_link">
+    <origin xyz="-0.227 0.165 0.023" rpy="0 0 0" />
+  </xacro:cam3d_tower>
+  <!-- 3D camera on tower -->
+  <xacro:asus_xtion_camera name="tower_cam3d" parent="camera_tower_link" tilt="0.5">
+    <origin xyz="0.015 0 0.47" rpy="0 0 0" />
+  </xacro:asus_xtion_camera>
+  <!-- Arm POV Mount -->
+  <xacro:microsoft_lifecam_1080_mount name="microsoft_lifecam_1080_mount" parent="arm_link_5">
+    <origin xyz="-0.035 0.0 -0.025" rpy="0 0 3.14159265" />
+  </xacro:microsoft_lifecam_1080_mount>
 </robot>

Commit message: preliminary urdf with 3dcam on arm. needs calibration

File: mir_robots/mir_hardware_config/youbot-brsu-3/urdf/robot.urdf.xacro (robot description, xacro)
@@ -14,6 +14,4 @@
   <!-- youbot arm -->
   <xacro:include filename="$(find youbot_description)/urdf/youbot_arm/arm.urdf.xacro"/>
-  <!-- youbot gripper -->
-  <xacro:include filename="$(find youbot_description)/urdf/youbot_gripper/gripper.urdf.xacro" />
   <!-- controller manager -->
   <xacro:include filename="$(find youbot_description)/controller/ros_controller.urdf.xacro" />
@@ -32,4 +30,7 @@
   <!-- foot for arm-->
   <xacro:youbot_base name="base"/>
+  <xacro:youbot_plate name="plate" parent="base_link">
+    <origin xyz="-0.159 0 0.046" rpy="0 0 0" />
+  </xacro:youbot_plate>
   <!-- BRSU SPECIFIC STUFF -->
   <xacro:include filename="$(find mcr_description)/urdf/materials.urdf.xacro" />
@@ -37,11 +38,6 @@
   <xacro:include filename="$(find mcr_description)/urdf/sensors/asus_xtion_camera.urdf.xacro"/>
   <xacro:include filename="$(find mcr_description)/urdf/mounts/microsoft_lifecam_1080_mount.urdf.xacro"/>
-  <xacro:include filename="$(find mir_description)/urdf/misc/rear_platform.urdf.xacro" />
+  <xacro:include filename="$(find mir_description)/urdf/grippers/festo_gripper.urdf.xacro" />
   <xacro:include filename="$(find mir_description)/urdf/misc/adapter_plate.urdf.xacro" />
-  <xacro:include filename="$(find mir_description)/urdf/grippers/festo_gripper.urdf.xacro" />
-  <!-- Rear Platform -->
-  <xacro:rear_platform name="rear_platform" parent="base_link">
-    <origin xyz="-0.005 -0.175 0.051" rpy="0 0 0" />
-  </xacro:rear_platform>
   <!-- Arm Plate moving arm 8cm foward and 45 degree rotation -->
   <xacro:adapter_plate name="adapter_plate" parent="base_link" arm_angle="${-M_PI / 4}">
@@ -51,8 +47,4 @@
     <origin xyz="-0.022 0.0 0.037" rpy="0 0 0" />
   </xacro:youbot_arm>
-  <!-- Festo Gripper -->
-  <xacro:festo_gripper name="gripper" parent="arm_link_5">
-    <origin xyz="0 0 0" rpy="0 0 0" />
-  </xacro:festo_gripper>
   <!-- base laser front -->
   <xacro:hokuyo_urg04_laser name="base_laser_front" parent="base" ros_topic="scan_front" update_rate="10" min_angle="-1.57" max_angle="1.57">
@@ -63,15 +55,20 @@
      <origin xyz="-0.3 0 -0.03" rpy="0 0 ${M_PI}" />
   </xacro:hokuyo_urg04_laser>
-  <!-- camera tower -->
-  <xacro:cam3d_tower name="camera_tower" parent="rear_platform_link">
-    <origin xyz="-0.227 0.165 0.023" rpy="0 0 0" />
+  <!-- camera tower
+  <xacro:cam3d_tower name="camera_tower" parent="plate_link">
+    <origin xyz="-0.10 0.0 -0.01" rpy="0 0 0" />
   </xacro:cam3d_tower>
-  <!-- 3D camera on tower -->
-  <xacro:asus_xtion_camera name="tower_cam3d" parent="camera_tower_link" tilt="0.5">
-    <origin xyz="0.015 0 0.47" rpy="0 0 0" />
+  -->
+  <!-- 3D camera on arm -->
+  <xacro:asus_xtion_camera name="arm_cam3d" parent="arm_link_5" tilt="0.0">
+    <origin xyz="${-0.035 + 0.030} ${0 - 0.025} ${-0.025}" rpy="0 ${-M_PI /  2} 0" />
   </xacro:asus_xtion_camera>
-  <!-- Arm POV Mount -->
+  <!-- Arm POV Mount
   <xacro:microsoft_lifecam_1080_mount name="microsoft_lifecam_1080_mount" parent="arm_link_5">
     <origin xyz="-0.035 0.0 -0.025" rpy="0 0 3.14159265" />
   </xacro:microsoft_lifecam_1080_mount>
+  -->
+  <xacro:festo_gripper name="gripper" parent="arm_link_5">
+    <origin xyz="0 0 0" rpy="0 0 0" />
+  </xacro:festo_gripper>
 </robot>

Commit message: more accurate arm cam positon

File: mir_robots/mir_hardware_config/youbot-brsu-3/urdf/robot.urdf.xacro (robot description, xacro)
@@ -30,7 +30,4 @@
   <!-- foot for arm-->
   <xacro:youbot_base name="base"/>
-  <xacro:youbot_plate name="plate" parent="base_link">
-    <origin xyz="-0.159 0 0.046" rpy="0 0 0" />
-  </xacro:youbot_plate>
   <!-- BRSU SPECIFIC STUFF -->
   <xacro:include filename="$(find mcr_description)/urdf/materials.urdf.xacro" />
@@ -62,5 +59,5 @@
   <!-- 3D camera on arm -->
   <xacro:asus_xtion_camera name="arm_cam3d" parent="arm_link_5" tilt="0.0">
-    <origin xyz="${-0.035 + 0.030} ${0 - 0.025} ${-0.025}" rpy="0 ${-M_PI /  2} 0" />
+    <origin xyz="${-0.035 - 0.030 + 0.030} ${0 - 0.025} ${-0.025}" rpy="0 ${-M_PI /  2} 0" />
   </xacro:asus_xtion_camera>
   <!-- Arm POV Mount

Commit message: [yb3] add rear platform to the urdf model

File: mir_robots/mir_hardware_config/youbot-brsu-3/urdf/robot.urdf.xacro (robot description, xacro)
@@ -30,4 +30,8 @@
   <!-- foot for arm-->
   <xacro:youbot_base name="base"/>
+  <!-- rear platform -->
+  <xacro:youbot_plate name="plate" parent="base_link">
+    <origin xyz="-0.159 0 0.046" rpy="0 0 0" />
+  </xacro:youbot_plate>
   <!-- BRSU SPECIFIC STUFF -->
   <xacro:include filename="$(find mcr_description)/urdf/materials.urdf.xacro" />

Commit message: calibrate ASUS on the arm 5 link

File: mir_robots/mir_hardware_config/youbot-brsu-3/urdf/robot.urdf.xacro (robot description, xacro)
@@ -63,5 +63,5 @@
   <!-- 3D camera on arm -->
   <xacro:asus_xtion_camera name="tower_cam3d" parent="arm_link_5" tilt="0.0">
-    <origin xyz="${-0.035 - 0.030 + 0.030} ${0 - 0.025} ${-0.025}" rpy="0 ${-M_PI /  2} 0" />
+    <origin xyz="${-0.035 - 0.030 + 0.030 + 0.01} ${0 - 0.055} ${-0.025 - 0.0}" rpy="0 ${-M_PI / 2} 0" />
   </xacro:asus_xtion_camera>
   <!-- Arm POV Mount

Commit message: [hardware config] calibrate camera based on pointcloud2laser vs hokuyo scans

File: mir_robots/mir_hardware_config/youbot-brsu-3/urdf/robot.urdf.xacro (robot description, xacro)
@@ -47,5 +47,5 @@
   <!-- 3D camera on arm --> <!-- NOTE: still called tower_cam3d due to legacy code -->
   <xacro:realsense_camera name="tower_cam3d" parent="arm_link_5">
-    <origin xyz="-0.075 0 0.02" rpy="0 ${-M_PI / 2} 0" />
+    <origin xyz="-0.075 0.05 0.05" rpy="-0.05 ${-M_PI / 2 + 0.25} 0" />
   </xacro:realsense_camera>
   <xacro:festo_gripper name="gripper" parent="arm_link_5">

Commit message: [urdf] calibrate arm cam on yb3

File: mir_robots/mir_hardware_config/youbot-brsu-3/urdf/robot.urdf.xacro (robot description, xacro)
@@ -47,5 +47,5 @@
   <!-- 3D camera on arm --> <!-- NOTE: still called tower_cam3d due to legacy code -->
   <xacro:realsense_camera name="tower_cam3d" parent="arm_link_5">
-    <origin xyz="-0.075 0.05 0.05" rpy="-0.05 ${-M_PI / 2 + 0.25} 0" />
+    <origin xyz="-0.055 0.03 0.02" rpy="-0.09 ${-M_PI / 2 + 0.15} -0.05" />
   </xacro:realsense_camera>
   <xacro:dynamixel_gripper name="gripper" parent="arm_link_5">

Commit message: [hardware config] update yb3 URDF

File: mir_robots/mir_hardware_config/youbot-brsu-3/urdf/robot.urdf.xacro (robot description, xacro)
@@ -11,9 +11,9 @@
   <!-- youbot base and rear platform -->
   <xacro:include filename="$(find youbot_description)/urdf/youbot_base/base.urdf.xacro" />
-  <xacro:include filename="$(find mir_description)/urdf/misc/rear_platform.urdf.xacro" />
+  <xacro:include filename="$(find mir_description)/urdf/misc/rear_platform_v2.urdf.xacro" />
   <!-- youbot arm and gripper-->
   <xacro:include filename="$(find youbot_description)/urdf/youbot_arm/arm.urdf.xacro"/>
   <xacro:include filename="$(find mir_description)/urdf/misc/adapter_plate.urdf.xacro" />
-  <xacro:include filename="$(find mir_description)/urdf/grippers/dynamixel/v1/dynamixel_gripper.urdf.xacro" />
+  <xacro:include filename="$(find mir_description)/urdf/grippers/dynamixel/v2/dynamixel_gripper.urdf.xacro" />
   <!-- controller manager -->
   <xacro:include filename="$(find youbot_description)/controller/ros_controller.urdf.xacro" />
@@ -22,4 +22,5 @@
   <!-- sensors -->
   <xacro:include filename="$(find youbot_description)/urdf/sensors/hokuyo_urg04_laser.urdf.xacro"/>
+  <xacro:include filename="$(find mir_description)/urdf/sensor_mounts/intel_f200_camera_mount.urdf.xacro"/>
   <xacro:include filename="$(find mcr_description)/urdf/sensors/intel_realsense_f200_camera.urdf.xacro"/>
   <!-- Now we can start using the macros included above to define the actual youbot -->
@@ -27,10 +28,10 @@
   <xacro:youbot_base name="base"/>
   <!-- Rear Platform -->
-  <xacro:rear_platform name="rear_platform" parent="base_link">
-    <origin xyz="-0.005 -0.175 0.051" rpy="0 0 0" />
-  </xacro:rear_platform>
+  <xacro:rear_platform_v2 name="rear_platform" parent="base_link">
+    <origin xyz="0.12 -0.175 ${0.021 + 0.0062 + 0.025 + 0.012}" rpy="0 0 0" />  <!-- ${alignment with base top + nut height + spacer height + slide height } -->
+  </xacro:rear_platform_v2>
   <!-- Arm Plate moving arm 8cm foward and 45 degree rotation -->
   <xacro:adapter_plate name="adapter_plate" parent="base_link" arm_angle="${-M_PI / 4}">
-    <origin xyz="${0.159+0.08} 0 0.051" rpy="0 0 0" />
+    <origin xyz="${0.159+0.08} 0 ${0.021 + 0.025 + 0.025}" rpy="0 0 0" />    <!-- ${alignment with base top + spacer height + spacer height } -->
   </xacro:adapter_plate>
   <xacro:youbot_arm name="arm" parent="adapter_plate_arm_root_link">
@@ -39,16 +40,20 @@
   <!-- base laser front -->
   <xacro:hokuyo_urg04_laser name="base_laser_front" parent="base" ros_topic="scan_front" update_rate="10" min_angle="-1.57" max_angle="1.57">
-    <origin xyz="0.3 0 -0.03" rpy="0 0 0"/>
+    <origin xyz="0.3 0 -0.035" rpy="${M_PI} 0 0"/>
   </xacro:hokuyo_urg04_laser>
   <!-- base laser rear -->
   <xacro:hokuyo_urg04_laser name="base_laser_rear" parent="base" ros_topic="scan_rear" update_rate="10" min_angle="-1.57" max_angle="1.57" >
-     <origin xyz="-0.3 0.0 -0.03" rpy="0 0 ${M_PI}" />
+     <origin xyz="-0.3 0.0 -0.035" rpy="${M_PI} 0 ${M_PI}" />
   </xacro:hokuyo_urg04_laser>
-  <!-- 3D camera on arm --> <!-- NOTE: still called arm_cam3d due to legacy code -->
-  <xacro:intel_realsense_f200_camera name="arm_cam3d" parent="arm_link_5">
-    <origin xyz="-0.055 0.03 0.02" rpy="-0.09 ${-M_PI / 2 + 0.15} -0.05" />
+  <xacro:dynamixel_gripper_v2 name="gripper" parent="arm_link_5">
+    <origin xyz="0.003 0 0.0052" rpy="0 0 0" />
+  </xacro:dynamixel_gripper_v2>
+  <!-- camera mount for Intel RealSense F200 -->
+  <xacro:intel_f200_camera_mount name="camera_mount" parent="gripper_motor_mount_link">
+    <origin xyz="-0.00375 -0.0007 0.0002" rpy="0 0 0" />
+  </xacro:intel_f200_camera_mount>
+  <!-- 3D camera on arm -->
+  <xacro:intel_realsense_f200_camera name="arm_cam3d" parent="camera_mount_link">
+    <origin xyz="-0.0405 0.0 0.029" rpy="0 -${M_PI/2} 0" />
   </xacro:intel_realsense_f200_camera>
-  <xacro:dynamixel_gripper name="gripper" parent="arm_link_5">
-    <origin xyz="0 0 -0.02" rpy="0 0 0" />
-  </xacro:dynamixel_gripper>
 </robot>

Commit message: [hardware config] configure hokuyos to be in normal orientation

File: mir_robots/mir_hardware_config/youbot-brsu-3/urdf/robot.urdf.xacro (robot description, xacro)
@@ -40,9 +40,9 @@
   <!-- base laser front -->
   <xacro:hokuyo_urg04_laser name="base_laser_front" parent="base" ros_topic="scan_front" update_rate="10" min_angle="-1.57" max_angle="1.57">
-    <origin xyz="0.3 0 -0.035" rpy="${M_PI} 0 0"/>
+    <origin xyz="0.3 0 -0.035" rpy="0 0 0"/>
   </xacro:hokuyo_urg04_laser>
   <!-- base laser rear -->
   <xacro:hokuyo_urg04_laser name="base_laser_rear" parent="base" ros_topic="scan_rear" update_rate="10" min_angle="-1.57" max_angle="1.57" >
-     <origin xyz="-0.3 0.0 -0.035" rpy="${M_PI} 0 ${M_PI}" />
+     <origin xyz="-0.3 0.0 -0.035" rpy="0 0 ${M_PI}" />
   </xacro:hokuyo_urg04_laser>
   <xacro:dynamixel_gripper_v2 name="gripper" parent="arm_link_5">

Commit message: [mir_bringup] modified urdf frile for ybrsu3

File: mir_robots/mir_hardware_config/youbot-brsu-3/urdf/robot.urdf.xacro (robot description, xacro)
@@ -28,13 +28,13 @@
   <xacro:youbot_base name="base"/>
   <!-- Rear Platform -->
-  <xacro:rear_platform_v2 name="rear_platform" parent="base_link">
-    <origin xyz="0.12 -0.175 ${0.021 + 0.0062 + 0.025 + 0.012}" rpy="0 0 0" />  <!-- ${alignment with base top + nut height + spacer height + slide height } -->
-  </xacro:rear_platform_v2>
+  <!-- <xacro:rear_platform_v2 name="rear_platform" parent="base_link">
+    <origin xyz="0.12 -0.175 ${0.021 + 0.0062 + 0.025 + 0.012}" rpy="0 0 0" />  ${alignment with base top + nut height + spacer height + slide height }
+  </xacro:rear_platform_v2> -->
   <!-- Arm Plate moving arm 8cm foward and 45 degree rotation -->
-  <xacro:adapter_plate name="adapter_plate" parent="base_link" arm_angle="${-M_PI / 4}">
-    <origin xyz="${0.159+0.08} 0 ${0.021 + 0.025 + 0.025}" rpy="0 0 0" />    <!-- ${alignment with base top + spacer height + spacer height } -->
-  </xacro:adapter_plate>
-  <xacro:youbot_arm name="arm" parent="adapter_plate_arm_root_link">
-    <origin xyz="-0.022 0.0 0.037" rpy="0 0 0" />
+  <!-- <xacro:adapter_plate name="adapter_plate" parent="base_link" arm_angle="${-M_PI / 4}">
+    <origin xyz="${0.159+0.08} 0 ${0.021 + 0.025 + 0.025}" rpy="0 0 0" />   ${alignment with base top + spacer height + spacer height }
+  </xacro:adapter_plate> -->
+  <xacro:youbot_arm name="arm" parent="base_link">
+    <origin xyz="0.15 0.025 0.05" rpy="0 0 -${pi/2}" />
   </xacro:youbot_arm>
   <!-- base laser front -->
@@ -46,14 +46,14 @@
      <origin xyz="-0.3 0.0 -0.035" rpy="0 0 ${M_PI}" />
   </xacro:hokuyo_urg04_laser>
-  <xacro:dynamixel_gripper_v2 name="gripper" parent="arm_link_5">
+  <!-- <xacro:dynamixel_gripper_v2 name="gripper" parent="arm_link_5">
     <origin xyz="0.003 0 0.0052" rpy="0 0 0" />
-  </xacro:dynamixel_gripper_v2>
+  </xacro:dynamixel_gripper_v2> -->
   <!-- camera mount for Intel RealSense F200 -->
-  <xacro:intel_f200_camera_mount name="camera_mount" parent="gripper_motor_mount_link">
+  <!-- <xacro:intel_f200_camera_mount name="camera_mount" parent="gripper_motor_mount_link">
     <origin xyz="-0.00375 -0.0007 0.0002" rpy="0 0 0" />
-  </xacro:intel_f200_camera_mount>
+  </xacro:intel_f200_camera_mount> -->
   <!-- 3D camera on arm -->
-  <xacro:intel_realsense_f200_camera name="arm_cam3d" parent="camera_mount_link">
+  <!-- <xacro:intel_realsense_f200_camera name="arm_cam3d" parent="camera_mount_link">
     <origin xyz="-0.0405 0.0 0.029" rpy="0 -${M_PI/2} 0" />
-  </xacro:intel_realsense_f200_camera>
+  </xacro:intel_realsense_f200_camera> -->
 </robot>
