Commit message: [mir_description] moved mcr_description into mir_description

File: mir_robots/mir_description/urdf/fingers/festo_finger_dhas-gf-shm.urdf.xacro (robot description, xacro)
@@ -4,5 +4,5 @@
        xmlns:interface="http://playerstage.sourceforge.net/gazebo/xmlschema/#interface"
        xmlns:xacro="http://ros.org/wiki/xacro">
-  <xacro:macro name="dynamixel_bracket_FP04-F2" params="parent name *origin">
+  <xacro:macro name="festo_finger_DHAS-GF-shm" params="parent name *origin">
     <joint name="${name}_joint" type="fixed" >
       <xacro:insert_block name="origin" />
@@ -13,17 +13,17 @@
       <inertial>
         <origin xyz="0 0 0" rpy="0 0 0"/>
-        <mass value="0.011"/>
+        <mass value="0.015"/>
         <inertia ixx="0.01" ixy="0" ixz="0" iyy="0.01" iyz="0" izz="0.01" />
       </inertial>
       <visual>
-        <origin xyz="0 0 0" rpy="0 0 0" />
+        <origin xyz="0 0 0" rpy="${M_PI/2} 0 ${M_PI/2}" />
         <geometry>
-          <mesh filename="package://mcr_description/meshes/motors/dynamixel_bracket_fp04-f2.dae" scale="0.001 0.001 0.001" />
+          <mesh filename="file://$(find mir_description)/meshes/fingers/festo_finger_dhas-gf-shm.dae" scale="0.001 0.001 0.001" />
         </geometry>
       </visual>
       <collision>
-        <origin xyz="0 0 0" rpy="0 0 0" />
+        <origin xyz="0 0 0" rpy="${M_PI/2} 0 ${M_PI/2}" />
         <geometry>
-          <mesh filename="package://mcr_description/meshes/motors/dynamixel_bracket_fp04-f2_convex_hull.dae" scale="0.001 0.001 0.001" />
+          <mesh filename="file://$(find mir_description)/meshes/fingers/festo_finger_dhas-gf-shm_convex_hull.dae" scale="0.001 0.001 0.001" />
         </geometry>
       </collision>

File: mir_robots/mir_description/urdf/grippers/dynamixel/d435_center/dynamixel_gripper.urdf.xacro (robot description, xacro)
@@ -7,10 +7,11 @@
   <!--xacro:include filename="$(find mir_description)/urdf/grippers/dynamixel/v2/dynamixel_gripper.transmission.xacro" /-->
   <!--xacro:include filename="$(find mir_description)/urdf/grippers/dynamixel/v2/dynamixel_gripper_limits.urdf.xacro" /-->
-  <xacro:include filename="$(find mcr_description)/urdf/motors/dynamixel_motor_ax-12a.urdf.xacro" />
-  <xacro:include filename="$(find mcr_description)/urdf/motors/dynamixel_bracket_fp04-f2.urdf.xacro" />
-  <xacro:include filename="$(find mir_description)/urdf/grippers/dynamixel/v2/festo_finger_mount.urdf.xacro" />
-  <xacro:include filename="$(find mcr_description)/urdf/fingers/festo_finger_dhas-gf-shm.urdf.xacro" />
+  <xacro:include filename="$(find mir_description)/urdf/motors/dynamixel_motor_ax-12a.urdf.xacro" />
+  <xacro:include filename="$(find mir_description)/urdf/motors/dynamixel_bracket_fp04-f2.urdf.xacro" />
+  <xacro:include filename="$(find mir_description)/urdf/grippers/dynamixel/d435_center/festo_finger_mount.urdf.xacro" />
+  <xacro:include filename="$(find mir_description)/urdf/grippers/dynamixel/grasp_fix_plugin.urdf.xacro" />
+  <xacro:include filename="$(find mir_description)/urdf/fingers/festo_finger_dhas-gf-shm.urdf.xacro" />
   <xacro:arg name="grasp_link_offset" default="0.11"/>
-  <xacro:macro name="dynamixel_gripper_v2" params="parent name *origin">
+  <xacro:macro name="dynamixel_gripper_d435_center" params="parent name *origin">
     <joint name="${name}_motor_mount_joint" type="fixed" >
       <xacro:insert_block name="origin" />
@@ -19,10 +20,11 @@
     </joint>
     <joint name="${name}_static_grasp_link_joint" type="fixed" >
-      <origin xyz="0 0 $(arg grasp_link_offset)" rpy="0 0 0"/>
+        <origin xyz="0 0 $(arg grasp_link_offset)" rpy="0 0 0"/>
       <parent link="${parent}" />
       <child link="${name}_static_grasp_link" />
     </joint>
-    <link name="${name}_static_grasp_link">
-    </link>
+    <material name="black">
+        <color rgba="0 0 0 1"/>
+    </material>
     <!-- motor mount -->
     <link name="${name}_motor_mount_link">
@@ -33,15 +35,18 @@
       </inertial>
       <visual>
-        <origin xyz="0 0 0.0" rpy="0 ${M_PI/2} 0" />
+        <origin xyz="-0.029 -0.046 0.0185" rpy="0 ${M_PI/2} 0" />
         <geometry>
-          <mesh filename="package://mir_description/meshes/grippers/dynamixel/v3/dynamixel_intel_camera_combined.stl" scale="0.001 0.001 0.001" />
+          <mesh filename="package://mir_description/meshes/grippers/dynamixel/d435_center/dynamixel_motor_mount.stl" scale="0.001 0.001 0.001" />
         </geometry>
+        <material name="black"/>
       </visual>
       <collision>
-        <origin xyz="0 0 -0.0" rpy="0 ${M_PI/2} 0" />
+        <origin xyz="-0.029 -0.046 0.0185" rpy="0 ${M_PI/2} 0" />
         <geometry>
-          <mesh filename="package://mir_description/meshes/grippers/dynamixel/v2/dynamixel_motor_mount_convex_hull.dae" scale="0.001 0.001 0.001" />
+          <mesh filename="package://mir_description/meshes/grippers/dynamixel/d435_center/dynamixel_motor_mount.stl" scale="0.001 0.001 0.001" />
         </geometry>
       </collision>
+    </link>
+    <link name="${name}_static_grasp_link">
     </link>
     <!-- motors -->
@@ -53,8 +58,8 @@
     </xacro:dynamixel_motor_AX-12A>
     <!-- brackets -->
-    <xacro:dynamixel_bracket_FP04-F2 name="${name}_bracket_left" parent="${name}_motor_left_base_link">
+    <xacro:dynamixel_bracket_FP04-F2 name="${name}_bracket_left" parent="${name}_motor_left_link">
       <origin xyz="0 0 0" rpy="0 0 0" />
     </xacro:dynamixel_bracket_FP04-F2>
-    <xacro:dynamixel_bracket_FP04-F2 name="${name}_bracket_right" parent="${name}_motor_right_base_link">
+    <xacro:dynamixel_bracket_FP04-F2 name="${name}_bracket_right" parent="${name}_motor_right_link">
       <origin xyz="0 0 0" rpy="0 0 0" />
     </xacro:dynamixel_bracket_FP04-F2>
@@ -73,4 +78,5 @@
       <origin xyz="0.004 0 0.0045" rpy="0 0 0" />
     </xacro:festo_finger_DHAS-GF-shm>
+    <xacro:gzplugin_grasp_fix />
   </xacro:macro>
 </robot>

File: mir_robots/mir_description/urdf/grippers/dynamixel/v2/dynamixel_gripper.urdf.xacro (robot description, xacro)
@@ -7,46 +7,44 @@
   <!--xacro:include filename="$(find mir_description)/urdf/grippers/dynamixel/v2/dynamixel_gripper.transmission.xacro" /-->
   <!--xacro:include filename="$(find mir_description)/urdf/grippers/dynamixel/v2/dynamixel_gripper_limits.urdf.xacro" /-->
-  <xacro:include filename="$(find mcr_description)/urdf/motors/dynamixel_motor_ax-12a.urdf.xacro" />
-  <xacro:include filename="$(find mcr_description)/urdf/motors/dynamixel_bracket_fp04-f2.urdf.xacro" />
-  <xacro:include filename="$(find mir_description)/urdf/grippers/dynamixel/d435_center/festo_finger_mount.urdf.xacro" />
-  <xacro:include filename="$(find mir_description)/urdf/grippers/dynamixel/grasp_fix_plugin.urdf.xacro" />
-  <xacro:include filename="$(find mcr_description)/urdf/fingers/festo_finger_dhas-gf-shm.urdf.xacro" />
+  <xacro:include filename="$(find mir_description)/urdf/motors/dynamixel_motor_ax-12a.urdf.xacro" />
+  <xacro:include filename="$(find mir_description)/urdf/motors/dynamixel_bracket_fp04-f2.urdf.xacro" />
+  <xacro:include filename="$(find mir_description)/urdf/grippers/dynamixel/v2/festo_finger_mount.urdf.xacro" />
+  <xacro:include filename="$(find mir_description)/urdf/fingers/festo_finger_dhas-gf-shm.urdf.xacro" />
   <xacro:arg name="grasp_link_offset" default="0.11"/>
-  <xacro:macro name="dynamixel_gripper_d435_center" params="parent name *origin">
+  <xacro:macro name="dynamixel_gripper_v2" params="parent name *origin">
     <joint name="${name}_motor_mount_joint" type="fixed" >
-      <xacro:insert_block name="origin" />
+      <origin xyz="0 0 0" rpy="0 0 0"/>
       <parent link="${parent}" />
       <child link="${name}_motor_mount_link" />
     </joint>
     <joint name="${name}_static_grasp_link_joint" type="fixed" >
-        <origin xyz="0 0 $(arg grasp_link_offset)" rpy="0 0 0"/>
+      <origin xyz="0 0 $(arg grasp_link_offset)" rpy="0 0 0"/>
       <parent link="${parent}" />
       <child link="${name}_static_grasp_link" />
     </joint>
-    <material name="black">
-        <color rgba="0 0 0 1"/>
-    </material>
+    <link name="${name}_static_grasp_link">
+    </link>
     <!-- motor mount -->
     <link name="${name}_motor_mount_link">
       <inertial>
-        <origin xyz="0 0 0" rpy="0 0 0"/>
+        <origin xyz="-0.0225 -0.046 0.0245" rpy="0 ${M_PI/2} 0" />
         <mass value="0.038"/>
         <inertia ixx="0.01" ixy="0" ixz="0" iyy="0.01" iyz="0" izz="0.01" />
       </inertial>
       <visual>
-        <origin xyz="-0.029 -0.046 0.0185" rpy="0 ${M_PI/2} 0" />
+        <origin xyz="-0.023 -0.046 0.024" rpy="0 ${M_PI/2} 0" />
         <geometry>
-          <mesh filename="package://mir_description/meshes/grippers/dynamixel/d435_center/dynamixel_motor_mount.stl" scale="0.001 0.001 0.001" />
+          <mesh filename="package://mir_description/meshes/grippers/dynamixel/v3/dynamixel_intel_camera_combined.stl" scale="0.001 0.001 0.001" />
         </geometry>
-        <material name="black"/>
+        <material name="">
+          <color rgba="0.85098 0.85098 0.85098 1"/>
+        </material>
       </visual>
       <collision>
-        <origin xyz="-0.029 -0.046 0.0185" rpy="0 ${M_PI/2} 0" />
+        <origin xyz="-0.0225 -0.046 0.0245" rpy="0 ${M_PI/2} 0" />
         <geometry>
-          <mesh filename="package://mir_description/meshes/grippers/dynamixel/d435_center/dynamixel_motor_mount.stl" scale="0.001 0.001 0.001" />
+          <mesh filename="package://mir_description/meshes/grippers/dynamixel/v2/dynamixel_motor_mount_convex_hull.dae" scale="0.001 0.001 0.001" />
         </geometry>
       </collision>
-    </link>
-    <link name="${name}_static_grasp_link">
     </link>
     <!-- motors -->
@@ -58,8 +56,8 @@
     </xacro:dynamixel_motor_AX-12A>
     <!-- brackets -->
-    <xacro:dynamixel_bracket_FP04-F2 name="${name}_bracket_left" parent="${name}_motor_left_link">
+    <xacro:dynamixel_bracket_FP04-F2 name="${name}_bracket_left" parent="${name}_motor_left_base_link">
       <origin xyz="0 0 0" rpy="0 0 0" />
     </xacro:dynamixel_bracket_FP04-F2>
-    <xacro:dynamixel_bracket_FP04-F2 name="${name}_bracket_right" parent="${name}_motor_right_link">
+    <xacro:dynamixel_bracket_FP04-F2 name="${name}_bracket_right" parent="${name}_motor_right_base_link">
       <origin xyz="0 0 0" rpy="0 0 0" />
     </xacro:dynamixel_bracket_FP04-F2>
@@ -78,5 +76,4 @@
       <origin xyz="0.004 0 0.0045" rpy="0 0 0" />
     </xacro:festo_finger_DHAS-GF-shm>
-    <xacro:gzplugin_grasp_fix />
   </xacro:macro>
 </robot>

File: mir_robots/mir_description/urdf/motors/dynamixel_bracket_fp04-f2.urdf.xacro (robot description, xacro)
@@ -4,5 +4,5 @@
        xmlns:interface="http://playerstage.sourceforge.net/gazebo/xmlschema/#interface"
        xmlns:xacro="http://ros.org/wiki/xacro">
-  <xacro:macro name="festo_finger_DHAS-GF-shm" params="parent name *origin">
+  <xacro:macro name="dynamixel_bracket_FP04-F2" params="parent name *origin">
     <joint name="${name}_joint" type="fixed" >
       <xacro:insert_block name="origin" />
@@ -13,17 +13,17 @@
       <inertial>
         <origin xyz="0 0 0" rpy="0 0 0"/>
-        <mass value="0.015"/>
+        <mass value="0.011"/>
         <inertia ixx="0.01" ixy="0" ixz="0" iyy="0.01" iyz="0" izz="0.01" />
       </inertial>
       <visual>
-        <origin xyz="0 0 0" rpy="${M_PI/2} 0 ${M_PI/2}" />
+        <origin xyz="0 0 0" rpy="0 0 0" />
         <geometry>
-          <mesh filename="package://mcr_description/meshes/fingers/festo_finger_dhas-gf-shm.dae" scale="0.001 0.001 0.001" />
+          <mesh filename="file://$(find mir_description)/meshes/motors/dynamixel_bracket_fp04-f2.dae" scale="0.001 0.001 0.001" />
         </geometry>
       </visual>
       <collision>
-        <origin xyz="0 0 0" rpy="${M_PI/2} 0 ${M_PI/2}" />
+        <origin xyz="0 0 0" rpy="0 0 0" />
         <geometry>
-          <mesh filename="package://mcr_description/meshes/fingers/festo_finger_dhas-gf-shm_convex_hull.dae" scale="0.001 0.001 0.001" />
+          <mesh filename="file://$(find mir_description)/meshes/motors/dynamixel_bracket_fp04-f2_convex_hull.dae" scale="0.001 0.001 0.001" />
         </geometry>
       </collision>

File: mir_robots/mir_description/urdf/motors/dynamixel_motor_ax-12a.urdf.xacro (robot description, xacro)
@@ -4,6 +4,6 @@
        xmlns:interface="http://playerstage.sourceforge.net/gazebo/xmlschema/#interface"
        xmlns:xacro="http://ros.org/wiki/xacro">
-  <xacro:include filename="$(find mcr_description)/urdf/motors/dynamixel_motor_ax-12a.gazebo.xacro" />
-  <xacro:include filename="$(find mcr_description)/urdf/motors/dynamixel_motor_ax-12a.transmission.xacro" />
+  <xacro:include filename="$(find mir_description)/urdf/motors/dynamixel_motor_ax-12a.gazebo.xacro" />
+  <xacro:include filename="$(find mir_description)/urdf/motors/dynamixel_motor_ax-12a.transmission.xacro" />
   <xacro:macro name="dynamixel_motor_AX-12A" params="parent name *origin motor_direction position_offset">
     <joint name="${name}_base_joint" type="fixed" >
@@ -21,5 +21,5 @@
         <origin xyz="0 0 0.03" rpy="0 ${M_PI/2} 0" />
         <geometry>
-          <mesh filename="package://mcr_description/meshes/motors/dynamixel_motor_ax-12a.dae" scale="0.001 0.001 0.001" />
+          <mesh filename="file://$(find mir_description)/meshes/motors/dynamixel_motor_ax-12a.dae" scale="0.001 0.001 0.001" />
         </geometry>
       </visual>
@@ -27,5 +27,5 @@
         <origin xyz="0 0 0.03" rpy="0 ${M_PI/2} 0" />
         <geometry>
-          <mesh filename="package://mcr_description/meshes/motors/dynamixel_motor_ax-12a_convex_hull.dae" scale="0.001 0.001 0.001" />
+          <mesh filename="file://$(find mir_description)/meshes/motors/dynamixel_motor_ax-12a_convex_hull.dae" scale="0.001 0.001 0.001" />
         </geometry>
       </collision>
@@ -36,4 +36,5 @@
       <origin xyz="0 0 0.03" rpy="${position_offset} 0 ${M_PI}"/>
       <axis xyz="${motor_direction} 0 0"/>
+      <dynamics damping="1.0" friction="1.0" />
       <limit effort="1.5" lower="-${M_PI / 180 * 150}" upper="${M_PI / 180 * 150}" velocity="6.178465545"/>
     </joint>

File: mir_robots/mir_description/urdf/mounts/microsoft_lifecam_1080_mount.urdf.xacro (robot description, xacro)
@@ -14,5 +14,5 @@
         <origin xyz="-0.015 0.04 -0.055" rpy="0 0 -1.57079633" />
         <geometry>
-          <mesh filename="package://mcr_description/meshes/mounts/microsoft_lifecam_1080_mount.dae" scale="0.001 0.001 0.001" />
+          <mesh filename="file://$(find mir_description)/meshes/mounts/microsoft_lifecam_1080_mount.dae" scale="0.001 0.001 0.001" />
         </geometry>
         <material name="Black" />
@@ -21,5 +21,5 @@
         <origin xyz="-0.015 0.04 -0.055" rpy="0 0 -1.57079633" />
         <geometry>
-          <mesh filename="package://mcr_description/meshes/mounts/microsoft_lifecam_1080_mount_convexhull.dae" scale="0.001 0.001 0.001"/>
+          <mesh filename="file://$(find mir_description)/meshes/mounts/microsoft_lifecam_1080_mount_convexhull.dae" scale="0.001 0.001 0.001"/>
         </geometry>
       </collision >

File: mir_robots/mir_description/urdf/ptu/ptu46.urdf.xacro (robot description, xacro)
@@ -1,6 +1,6 @@
 <?xml version="1.0"?>
 <robot xmlns:xacro="http://ros.org/wiki/xacro">
-	<xacro:include filename="$(find mcr_description)/urdf/ptu/ptu46.gazebo.xacro" />
-	<xacro:include filename="$(find mcr_description)/urdf/ptu/ptu46.transmission.xacro" />
+	<xacro:include filename="$(find mir_description)/urdf/ptu/ptu46.gazebo.xacro" />
+	<xacro:include filename="$(find mir_description)/urdf/ptu/ptu46.transmission.xacro" />
 	<xacro:macro name="ptu46" params="parent name *origin">
 		<link name="${name}_link">

File: mir_robots/mir_description/urdf/sensors/asus_xtion_camera.urdf.xacro (robot description, xacro)
@@ -28,5 +28,5 @@
         <origin xyz="0.01 0 0" rpy="${M_PI/2} 0 ${M_PI/2}" />
         <geometry>
-           <mesh filename="package://mcr_description/meshes/sensors/asus_xtion_pro_live_base.dae" scale="0.0004 0.0007 0.001"/>
+           <mesh filename="file://$(find mir_description)/meshes/sensors/asus_xtion_pro_live_base.dae" scale="0.0004 0.0007 0.001"/>
         </geometry>
         <material name="Black" />
@@ -35,5 +35,5 @@
         <origin xyz="0.01 0 0" rpy="${M_PI/2} 0 ${M_PI/2}" />
         <geometry>
-           <mesh filename="package://mcr_description/meshes/sensors/asus_xtion_pro_live_base.dae" scale="0.0004 0.0007 0.001"/>
+           <mesh filename="file://$(find mir_description)/meshes/sensors/asus_xtion_pro_live_base.dae" scale="0.0004 0.0007 0.001"/>
         </geometry>
       </collision >
@@ -81,5 +81,5 @@
         <origin xyz="0.02 -0.03 0" rpy="${M_PI/2} 0 ${M_PI/2}" />
         <geometry>
-          <mesh filename="package://mcr_description/meshes/sensors/asus_xtion_pro_live_camera.dae" scale="0.001 0.001 0.001"/>
+          <mesh filename="file://$(find mir_description)/meshes/sensors/asus_xtion_pro_live_camera.dae" scale="0.001 0.001 0.001"/>
         </geometry>
         <material name="Black" />
@@ -88,5 +88,5 @@
         <origin xyz="0.02 -0.03 0" rpy="${M_PI/2} 0 ${M_PI/2}" />
         <geometry>
-           <mesh filename="package://mcr_description/meshes/sensors/asus_xtion_pro_live_camera_convexhull.dae" scale="0.001 0.001 0.001"/>
+           <mesh filename="file://$(find mir_description)/meshes/sensors/asus_xtion_pro_live_camera_convexhull.dae" scale="0.001 0.001 0.001"/>
         </geometry>
       </collision >

File: mir_robots/mir_description/urdf/sensors/hokuyo_lx30.urdf.xacro (robot description, xacro)
@@ -4,5 +4,5 @@
        xmlns:interface="http://playerstage.sourceforge.net/gazebo/xmlschema/#interface"
        xmlns:xacro="http://ros.org/wiki/xacro">
-  <xacro:include filename="$(find mcr_description)/urdf/sensors/hokuyo_lx30.gazebo.xacro" />
+  <xacro:include filename="$(find mir_description)/urdf/sensors/hokuyo_lx30.gazebo.xacro" />
   <xacro:macro name="hokuyo_lx30" params="name parent *origin ros_topic update_rate min_angle max_angle">
     <joint name="${name}_joint" type="fixed">

File: mir_robots/mir_description/urdf/sensors/intel_realsense_f200_camera.urdf.xacro (robot description, xacro)
@@ -4,5 +4,5 @@
        xmlns:interface="http://playerstage.sourceforge.net/gazebo/xmlschema/#interface"
        xmlns:xacro="http://ros.org/wiki/xacro">
-  <xacro:include filename="$(find mcr_description)/urdf/sensors/intel_realsense_f200_camera.gazebo.xacro" />
+  <xacro:include filename="$(find mir_description)/urdf/sensors/intel_realsense_f200_camera.gazebo.xacro" />
   <xacro:property name="eye_x_offset" value="-0.015" />
   <xacro:property name="eye_y_offset" value="0.024" />
@@ -32,5 +32,5 @@
         <origin xyz="0 -0.074 0" rpy="0 0 0" />
         <geometry>
-          <mesh filename="package://mcr_description/meshes/sensors/intel_realsense_f200_camera.dae" scale="0.001 0.001 0.001" />
+          <mesh filename="file://$(find mir_description)/meshes/sensors/intel_realsense_f200_camera.dae" scale="0.001 0.001 0.001" />
         </geometry>
       </visual>
@@ -38,5 +38,5 @@
         <origin xyz="0 -0.074 0" rpy="0 0 0" />
         <geometry>
-          <mesh filename="package://mcr_description/meshes/sensors/intel_realsense_f200_camera_convex_hull.dae" scale="0.001 0.001 0.001" />
+          <mesh filename="file://$(find mir_description)/meshes/sensors/intel_realsense_f200_camera_convex_hull.dae" scale="0.001 0.001 0.001" />
         </geometry>
      </collision>

File: mir_robots/mir_description/urdf/sensors/kinect_camera.urdf.xacro (robot description, xacro)
@@ -4,5 +4,5 @@
       xmlns:interface="http://playerstage.sourceforge.net/gazebo/xmlschema/#interface"
       xmlns:xacro="http://ros.org/wiki/xacro">
-  <xacro:include filename="$(find mcr_description)/urdf/sensors/kinect_camera.gazebo.xacro" />
+  <xacro:include filename="$(find mir_description)/urdf/sensors/kinect_camera.gazebo.xacro" />
   <xacro:macro name="kinect_camera" params="name parent *origin">
     <joint name="${name}_frame_joint" type="fixed">

File: mir_robots/mir_description/urdf/sensors/microsoft_lifecam.urdf.xacro (robot description, xacro)
@@ -4,5 +4,5 @@
       xmlns:interface="http://playerstage.sourceforge.net/gazebo/xmlschema/#interface"
       xmlns:xacro="http://ros.org/wiki/xacro">
-  <xacro:include filename="$(find mcr_description)/urdf/sensors/microsoft_lifecam.gazebo.xacro"/>
+  <xacro:include filename="$(find mir_description)/urdf/sensors/microsoft_lifecam.gazebo.xacro"/>
   <xacro:macro name="microsoft_lifecam" params="name parent *origin">
    <joint name="${name}_camera_joint" type="fixed">
@@ -22,5 +22,5 @@
       <origin xyz="-0.04 -0.0035 -0.031" rpy="${M_PI/2} 0 ${M_PI/2}" />
       <geometry>
-       <mesh filename="package://mcr_description/meshes/sensors/microsoft_lifecam.dae" scale="0.001 0.001 0.001"/>
+       <mesh filename="file://$(find mir_description)/meshes/sensors/microsoft_lifecam.dae" scale="0.001 0.001 0.001"/>
       </geometry>
     </visual>
@@ -28,5 +28,5 @@
       <origin xyz="-0.04 -0.0035 -0.031" rpy="${M_PI/2} 0 ${M_PI/2}" />
       <geometry>
-        <mesh filename="package://mcr_description/meshes/sensors/microsoft_lifecam.dae" scale="0.001 0.001 0.001"/>
+        <mesh filename="file://$(find mir_description)/meshes/sensors/microsoft_lifecam.dae" scale="0.001 0.001 0.001"/>
       </geometry>
     </collision>

File: mir_robots/mir_description/urdf/sensors/pmd_camboard_nano_camera.urdf.xacro (robot description, xacro)
@@ -4,5 +4,5 @@
       xmlns:interface="http://playerstage.sourceforge.net/gazebo/xmlschema/#interface"
       xmlns:xacro="http://ros.org/wiki/xacro">
-  <xacro:include filename="$(find mcr_description)/urdf/sensors/pmd_camboard_nano_camera.gazebo.xacro" />
+  <xacro:include filename="$(find mir_description)/urdf/sensors/pmd_camboard_nano_camera.gazebo.xacro" />
   <xacro:macro name="pmd_camboard_nano_camera" params="name parent *origin">
     <joint name="${name}_frame_joint" type="fixed">

File: mir_robots/mir_description/urdf/sensors/realsense_d435.urdf.xacro (robot description, xacro)
@@ -7,5 +7,5 @@
 -->
 <robot xmlns:xacro="http://ros.org/wiki/xacro">
-  <xacro:include filename="$(find mcr_description)/urdf/sensors/realsense_d435.gazebo.xacro" />
+  <xacro:include filename="$(find mir_description)/urdf/sensors/realsense_d435.gazebo.xacro" />
   <xacro:macro name="realsense_d435" params="name parent *origin">
     <xacro:property name="M_PI" value="3.1415926535897931" />
@@ -40,5 +40,5 @@
       <origin xyz="${d435_cam_mount_from_center_offset} 0.0 ${d435_cam_height/2}" rpy="${M_PI/2} 0 ${M_PI/2}"/>
         <geometry>
-          <mesh filename="package://mcr_description/meshes/sensors/realsense_d435.dae" />
+          <mesh filename="file://$(find mir_description)/meshes/sensors/realsense_d435.dae" />
         </geometry>
         <material name="${name}_aluminum"/>
