Commit message: [mir_description] moved mcr_description into mir_description

File: mir_robots/mir_description/urdf/sensors/sick_lms_200.urdf.xacro (robot description, xacro)
@@ -1,5 +1,5 @@
 <?xml version="1.0"?>
 <robot xmlns:xacro="http://ros.org/wiki/xacro">
-	<xacro:include filename="$(find mcr_description)/urdf/sensors/sick_lms_200.gazebo.xacro" />
+	<xacro:include filename="$(find mir_description)/urdf/sensors/sick_lms_200.gazebo.xacro" />
 	<xacro:macro name="sick_lms_200" params="name parent *origin ros_topic update_rate min_angle max_angle">
 		<joint name="${name}_joint" type="fixed">

File: mir_robots/mir_hardware_config/youbot-brsu-3/urdf/robot.urdf.xacro (robot description, xacro)
@@ -8,5 +8,5 @@
   <!-- misc common stuff -->
   <xacro:include filename="$(find youbot_description)/urdf/common.xacro" />
-  <xacro:include filename="$(find mcr_description)/urdf/materials.urdf.xacro" />
+  <xacro:include filename="$(find mir_description)/urdf/materials.urdf.xacro" />
   <!-- youbot base and rear platform -->
   <xacro:include filename="$(find youbot_description)/urdf/youbot_base/base.urdf.xacro" />
@@ -23,5 +23,5 @@
   <xacro:include filename="$(find youbot_description)/urdf/sensors/hokuyo_urg04_laser.urdf.xacro"/>
   <xacro:include filename="$(find mir_description)/urdf/sensor_mounts/intel_f200_camera_mount.urdf.xacro"/>
-  <xacro:include filename="$(find mcr_description)/urdf/sensors/intel_realsense_f200_camera.urdf.xacro"/>
+  <xacro:include filename="$(find mir_description)/urdf/sensors/intel_realsense_f200_camera.urdf.xacro"/>
   <!-- Now we can start using the macros included above to define the actual youbot -->
   <!-- standard youBot configuration -->
