Commit message: add camera tower and ASUS RGB-D cam to youbot 2 and 3

File: mir_robots/mir_hardware_config/youbot-brsu-2/urdf/robot.urdf.xacro (robot description, xacro)
@@ -43,9 +43,9 @@
   <!-- BRSU SPECIFIC STUFF -->
   <xacro:include filename="$(find mcr_description)/urdf/materials.urdf.xacro" />
-  <!--xacro:include filename="$(find mcr_description)/urdf/sensors/kinect_camera.urdf.xacro" />
-  <xacro:include filename="$(find mcr_description)/urdf/sensors/pmd_camboard_nano_camera.urdf.xacro" />
+  <xacro:include filename="$(find youbot_description)/urdf/sensors/asus_xtion_camera.urdf.xacro"/>
+  <xacro:include filename="$(find youbot_description)/urdf/misc/camera_tower.urdf.xacro"/>
+  <!--xacro:include filename="$(find mcr_description)/urdf/sensors/pmd_camboard_nano_camera.urdf.xacro" />
   <xacro:include filename="$(find mir_calibration_data)/youbot-brsu-2/calibration.urdf.xacro" />
   <xacro:include filename="$(find mir_description)/urdf/misc/sensor_angle_shortend.urdf.xacro" />
-  <xacro:include filename="$(find mir_description)/urdf/misc/cam3d_tower.urdf.xacro" />
   <xacro:include filename="$(find mir_description)/urdf/misc/laptop_case_frame.urdf.xacro" />
   <xacro:include filename="$(find mir_description)/urdf/misc/distance_screw.urdf.xacro" />
@@ -56,4 +56,12 @@
     <origin xyz="0.3 0 -0.03" rpy="0 0 0"/>
   </xacro:hokuyo_urg04_laser>
+  <!-- camera tower -->
+  <xacro:camera_tower name="camera_tower" parent="plate_link">
+    <origin xyz="-0.11 0.0 0.03" rpy="0 0 0" />
+  </xacro:camera_tower>
+  <!-- 3D camera on tower -->
+  <xacro:asus_xtion_camera name="tower_cam3d" parent="camera_tower_link" tilt="0.5">
+    <origin xyz="0 0 0.49" rpy="0 0 0" />
+  </xacro:asus_xtion_camera>
   <!-- brsu specific platforms
   <xacro:rear_platform name="rear_platform" parent="base_link">
@@ -108,10 +116,3 @@
     <origin xyz="${cal_arm_cam3d_x} ${cal_arm_cam3d_y} ${cal_arm_cam3d_z}" rpy="${cal_arm_cam3d_roll} ${cal_arm_cam3d_pitch} ${cal_arm_cam3d_yaw}" />
   </xacro:pmd_camboard_nano_camera>
-  <xacro:cam3d_tower name="tower" parent="rear_platform_link">
-    <origin xyz="-0.245 0.175 0.0" rpy="0 0 0" />
-  </xacro:cam3d_tower-->
-  <!-- 3D camera on tower
-  <xacro:kinect_camera name="tower_cam3d" parent="tower_link">
-    <origin xyz="${cal_tower_cam3d_x} ${cal_tower_cam3d_y} ${cal_tower_cam3d_z}" rpy="${cal_tower_cam3d_roll} ${cal_tower_cam3d_pitch} ${cal_tower_cam3d_yaw}" />
-  </xacro:kinect_camera-->
 </robot>

File: mir_robots/mir_hardware_config/youbot-brsu-3/urdf/robot.urdf.xacro (robot description, xacro)
@@ -43,8 +43,18 @@
   <!-- BRSU SPECIFIC STUFF -->
   <xacro:include filename="$(find mcr_description)/urdf/materials.urdf.xacro" />
+  <xacro:include filename="$(find youbot_description)/urdf/sensors/asus_xtion_camera.urdf.xacro"/>
+  <xacro:include filename="$(find youbot_description)/urdf/misc/camera_tower.urdf.xacro"/>
   <!-- base laser front -->
   <xacro:hokuyo_urg04_laser name="base_laser_front" parent="base" ros_topic="scan_front" update_rate="10" min_angle="-1.57" max_angle="1.57">
     <origin xyz="0.3 0 -0.03" rpy="0 0 0"/>
   </xacro:hokuyo_urg04_laser>
+  <!-- camera tower -->
+  <xacro:camera_tower name="camera_tower" parent="plate_link">
+    <origin xyz="-0.11 0.0 0.03" rpy="0 0 0" />
+  </xacro:camera_tower>
+  <!-- 3D camera on tower -->
+  <xacro:asus_xtion_camera name="tower_cam3d" parent="camera_tower_link" tilt="0.5">
+    <origin xyz="0 0 0.49" rpy="0 0 0" />
+  </xacro:asus_xtion_camera>
   <!-- base laser rear
   <xacro:hokuyo_urg04_laser name="base_laser_rear" parent="base" ros_topic="scan_rear" update_rate="10" min_angle="-1.57" max_angle="1.57" >

Commit message: cleanup youbot-2 urdf

File: mir_robots/mir_hardware_config/youbot-brsu-2/urdf/robot.urdf.xacro (robot description, xacro)
@@ -23,12 +23,5 @@
   <xacro:include filename="$(find youbot_description)/urdf/sensors/hokuyo_urg04_laser.urdf.xacro"/>
   <!-- Now we can start using the macros included above to define the actual youbot -->
-  <!-- The first use of a macro.  This one was defined in base.urdf.xacro above.
-       A macro like this will expand to a set of link and joint definitions, and to additional
-       Gazebo-related extensions (sensor plugins, etc).  The macro takes an argument, name,
-       that equals "base", and uses it to generate names for its component links and joints
-       (e.g., base_link).  The included origin block is also an argument to the macro.  By convention,
-       the origin block defines where the component is w.r.t its parent (in this case the parent
-       is the world frame). For more, see http://www.ros.org/wiki/xacro -->
-  <!-- foot for arm-->
+  <!-- standard youBot configuration -->
   <xacro:youbot_base name="base"/>
   <xacro:youbot_plate name="plate" parent="base_link">
@@ -42,17 +35,14 @@
   </xacro:youbot_gripper>
   <!-- BRSU SPECIFIC STUFF -->
-  <xacro:include filename="$(find mcr_description)/urdf/materials.urdf.xacro" />
   <xacro:include filename="$(find youbot_description)/urdf/sensors/asus_xtion_camera.urdf.xacro"/>
   <xacro:include filename="$(find youbot_description)/urdf/misc/camera_tower.urdf.xacro"/>
-  <!--xacro:include filename="$(find mcr_description)/urdf/sensors/pmd_camboard_nano_camera.urdf.xacro" />
-  <xacro:include filename="$(find mir_calibration_data)/youbot-brsu-2/calibration.urdf.xacro" />
-  <xacro:include filename="$(find mir_description)/urdf/misc/sensor_angle_shortend.urdf.xacro" />
-  <xacro:include filename="$(find mir_description)/urdf/misc/laptop_case_frame.urdf.xacro" />
-  <xacro:include filename="$(find mir_description)/urdf/misc/distance_screw.urdf.xacro" />
-  <xacro:include filename="$(find mir_description)/urdf/misc/adapter_plate.urdf.xacro" />
-  <xacro:include filename="$(find mir_description)/urdf/misc/rear_platform.urdf.xacro" /-->
+  <xacro:include filename="$(find mcr_description)/urdf/materials.urdf.xacro" />
   <!-- base laser front -->
   <xacro:hokuyo_urg04_laser name="base_laser_front" parent="base" ros_topic="scan_front" update_rate="10" min_angle="-1.57" max_angle="1.57">
     <origin xyz="0.3 0 -0.03" rpy="0 0 0"/>
+  </xacro:hokuyo_urg04_laser>
+  <!-- base laser rear -->
+  <xacro:hokuyo_urg04_laser name="base_laser_rear" parent="base" ros_topic="scan_rear" update_rate="10" min_angle="-1.57" max_angle="1.57" >
+     <origin xyz="-0.3 0.0 -0.03" rpy="0 0 ${M_PI}" />
   </xacro:hokuyo_urg04_laser>
   <!-- camera tower -->
@@ -64,55 +54,3 @@
     <origin xyz="0 0 0.49" rpy="0 0 0" />
   </xacro:asus_xtion_camera>
-  <!-- brsu specific platforms
-  <xacro:rear_platform name="rear_platform" parent="base_link">
-    <origin xyz="-0.029 -0.175 0.100" rpy="0 0 0" />
-  </xacro:rear_platform>
-  <xacro:adapter_plate name="front_plate" parent="base_link">
-    <origin xyz="0.340 -0.175 0.049" rpy="0 0 0" />
-  </xacro:adapter_plate-->
-  <!-- base laser rear -->
-  <xacro:hokuyo_urg04_laser name="base_laser_rear" parent="base" ros_topic="scan_rear" update_rate="10" min_angle="-1.57" max_angle="1.57" >
-     <origin xyz="-0.3 0.0 -0.03" rpy="0 0 ${M_PI}" />
-  </xacro:hokuyo_urg04_laser>
-  <!-- distance screws
-  <xacro:distance_screw name="distance_screw_fl" parent="base_link">
-    <origin xyz="-0.11 0.075 0.035" rpy="0 0 0" />
-  </xacro:distance_screw>
-  <xacro:distance_screw name="distance_screw_fr" parent="base_link">
-    <origin xyz="-0.11 -0.075 0.035" rpy="0 0 0" />
-  </xacro:distance_screw>
-  <xacro:distance_screw name="distance_screw_rl" parent="base_link">
-    <origin xyz="-0.20 0.075 0.035" rpy="0 0 0" />
-  </xacro:distance_screw>
-  <xacro:distance_screw name="distance_screw_rr" parent="base_link">
-    <origin xyz="-0.20 -0.075 0.035" rpy="0 0 0" />
-  </xacro:distance_screw-->
-  <!-- distance screws front
-  <xacro:distance_screw name="front_distance_screw_fl" parent="base_link">
-    <origin xyz="0.088 0.055 0.035" rpy="0 0 0" />
-  </xacro:distance_screw>
-  <xacro:distance_screw name="front_distance_screw_fr" parent="base_link">
-    <origin xyz="0.088 -0.055 0.035" rpy="0 0 0" />
-  </xacro:distance_screw>
-  <xacro:distance_screw name="front_distance_screw_rl" parent="base_link">
-    <origin xyz="0.228 0.055 0.035" rpy="0 0 0" />
-  </xacro:distance_screw>
-  <xacro:distance_screw name="front_distance_screw_rr" parent="base_link">
-    <origin xyz="0.228 -0.055 0.035" rpy="0 0 0" />
-  </xacro:distance_screw-->
-  <!-- laptop case frame
-  <xacro:laptop_case_frame name="laptop_case_frame_left" parent="base_link">
-    <origin xyz="-0.15 0.075 0.05" rpy="0 0 ${-M_PI/2}" />
-  </xacro:laptop_case_frame>
-  <xacro:laptop_case_frame name="laptop_case_frame_right" parent="base_link">
-    <origin xyz="-0.15 -0.075 0.05" rpy="0 0 ${M_PI/2}" />
-  </xacro:laptop_case_frame-->
-  <!-- Sensor angle on arm
-  <xacro:sensor_angle_shortend name="arm_sensor_angle_shortend" parent="arm_link_5">
-    <origin xyz="0.015 0.0 -0.023" rpy="0.0 0.0 ${M_PI}" />
-  </xacro:sensor_angle_shortend-->
-  <!-- pmd on arm
-  <xacro:pmd_camboard_nano_camera name="arm_cam3d" parent="arm_sensor_angle_shortend_part2_link">
-    <origin xyz="${cal_arm_cam3d_x} ${cal_arm_cam3d_y} ${cal_arm_cam3d_z}" rpy="${cal_arm_cam3d_roll} ${cal_arm_cam3d_pitch} ${cal_arm_cam3d_yaw}" />
-  </xacro:pmd_camboard_nano_camera-->
 </robot>

Commit message: calibrate tower position on youbot 2

File: mir_robots/mir_hardware_config/youbot-brsu-2/urdf/robot.urdf.xacro (robot description, xacro)
@@ -48,5 +48,5 @@
   <!-- camera tower -->
   <xacro:camera_tower name="camera_tower" parent="plate_link">
-    <origin xyz="-0.11 0.0 0.03" rpy="0 0 0" />
+    <origin xyz="-0.075 0.0 0.023" rpy="0 0 0" />
   </xacro:camera_tower>
   <!-- 3D camera on tower -->

Commit message: calibrate ASUS 3D cam on yb2

File: mir_robots/mir_hardware_config/youbot-brsu-2/urdf/robot.urdf.xacro (robot description, xacro)
@@ -52,5 +52,5 @@
   <!-- 3D camera on tower -->
   <xacro:asus_xtion_camera name="tower_cam3d" parent="camera_tower_link" tilt="0.5">
-    <origin xyz="0 0 0.49" rpy="0 0 0" />
+    <origin xyz="0.015 0 0.47" rpy="0 0 0" />
   </xacro:asus_xtion_camera>
 </robot>

Commit message: Added pov camera mount to arm and festo mount

File: mir_robots/mir_hardware_config/youbot-brsu-2/urdf/robot.urdf.xacro (robot description, xacro)
@@ -37,4 +37,6 @@
   <xacro:include filename="$(find youbot_description)/urdf/sensors/asus_xtion_camera.urdf.xacro"/>
   <xacro:include filename="$(find youbot_description)/urdf/misc/camera_tower.urdf.xacro"/>
+  <xacro:include filename="$(find youbot_description)/urdf/misc/arm_pov_mount.urdf.xacro"/>
+  <xacro:include filename="$(find youbot_description)/urdf/misc/festo_mount.urdf.xacro"/>
   <xacro:include filename="$(find mcr_description)/urdf/materials.urdf.xacro" />
   <!-- base laser front -->
@@ -54,3 +56,11 @@
     <origin xyz="0.015 0 0.47" rpy="0 0 0" />
   </xacro:asus_xtion_camera>
+  <!-- Arm POV Mount -->
+  <xacro:arm_pov_mount name="arm_pov_mount" parent="arm_link_5">
+    <origin xyz="0.075 0.0 -0.02" rpy="0 0 0" />
+  </xacro:arm_pov_mount>
+  <!-- Festo Finger Mount -->
+  <xacro:festo_mount name="festo_mount" parent="gripper_palm_link">
+    <origin xyz="0.0 0.0 0.05" rpy="0 0 0" />
+  </xacro:festo_mount>
 </robot>

Commit message: Added Arm POV camera mount to Youbot 2 URDF
Along the commit here: moriarty/youbot_description@fe9bd0054c1d45b30651b3985e6c780d55a7ddc4 this should
close issue mas-group/mas_industrial_robotics#39

No Festo Finger Mounts were added to the URDF. A better model of the finger mounts is required.

File: mir_robots/mir_hardware_config/youbot-brsu-2/urdf/robot.urdf.xacro (robot description, xacro)
@@ -58,9 +58,5 @@
   <!-- Arm POV Mount -->
   <xacro:arm_pov_mount name="arm_pov_mount" parent="arm_link_5">
-    <origin xyz="0.075 0.0 -0.02" rpy="0 0 0" />
+    <origin xyz="0.035 0.0 -0.03" rpy="0 0 0" />
   </xacro:arm_pov_mount>
-  <!-- Festo Finger Mount -->
-  <xacro:festo_mount name="festo_mount" parent="gripper_palm_link">
-    <origin xyz="0.0 0.0 0.05" rpy="0 0 0" />
-  </xacro:festo_mount>
 </robot>

Commit message: renamed/moved to microsoft_lifecam_1080_mount
- Moved files to mcr_description as requested in mas-group/youbot_description#2
- Adjusted position, and put camera mount on the other side of arm.
- When pre_grasp camera is now ontop of arm.
- Finishes mas-group/mas_industrial_robotics#39

File: mir_robots/mir_hardware_config/youbot-brsu-2/urdf/robot.urdf.xacro (robot description, xacro)
@@ -37,5 +37,5 @@
   <xacro:include filename="$(find youbot_description)/urdf/sensors/asus_xtion_camera.urdf.xacro"/>
   <xacro:include filename="$(find youbot_description)/urdf/misc/camera_tower.urdf.xacro"/>
-  <xacro:include filename="$(find youbot_description)/urdf/misc/arm_pov_mount.urdf.xacro"/>
+  <xacro:include filename="$(find mcr_description)/urdf/sensors/microsoft_lifecam_1080_mount.urdf.xacro"/>
   <xacro:include filename="$(find mcr_description)/urdf/materials.urdf.xacro" />
   <!-- base laser front -->
@@ -56,6 +56,6 @@
   </xacro:asus_xtion_camera>
   <!-- Arm POV Mount -->
-  <xacro:arm_pov_mount name="arm_pov_mount" parent="arm_link_5">
-    <origin xyz="0.035 0.0 -0.03" rpy="0 0 0" />
-  </xacro:arm_pov_mount>
+  <xacro:microsoft_lifecam_1080_mount name="microsoft_lifecam_1080_mount" parent="arm_link_5">
+    <origin xyz="-0.035 0.0 -0.025" rpy="0 0 3.14159265" />
+  </xacro:microsoft_lifecam_1080_mount>
 </robot>

Commit message: Added Festo Gripper in fixed open position
- Adds to mir_description
    - festo_gripper urdf xacro
    - festo_gripper open mesh as one static part
- Modifies robot.urdf.xacro
    - No longer calls youbot_gripper macro
    - Calls festo_gripper macro
- In Festo_gripper xacro
    - All links from youbot_gripper still exist
    - Meshes of original fingers have been removed, not their links
    - 3 new joints: linkage, tip_joint, grasp_joint
- tip_joint is tip of closed festo gripper
- grasp joint is in middle of closed festo fingers
- linkage joint is where festo mechanics being, static for now.

- Includes simple mesh for collision checking

- Removed unused imports

- Moved files into grippers subdirectory

- new include locations

File: mir_robots/mir_hardware_config/youbot-brsu-2/urdf/robot.urdf.xacro (robot description, xacro)
@@ -14,6 +14,4 @@
   <!-- youbot arm -->
   <xacro:include filename="$(find youbot_description)/urdf/youbot_arm/arm.urdf.xacro"/>
-  <!-- youbot gripper -->
-  <xacro:include filename="$(find youbot_description)/urdf/youbot_gripper/gripper.urdf.xacro" />
   <!-- controller manager -->
   <xacro:include filename="$(find youbot_description)/controller/ros_controller.urdf.xacro" />
@@ -31,12 +29,10 @@
     <origin xyz="0.143 0 0.046" rpy="0 0 0" />
   </xacro:youbot_arm>
-  <xacro:youbot_gripper name="gripper" parent="arm_link_5">
-    <origin xyz="0 0 0" rpy="0 0 0" />
-  </xacro:youbot_gripper>
   <!-- BRSU SPECIFIC STUFF -->
   <xacro:include filename="$(find youbot_description)/urdf/sensors/asus_xtion_camera.urdf.xacro"/>
   <xacro:include filename="$(find youbot_description)/urdf/misc/camera_tower.urdf.xacro"/>
-  <xacro:include filename="$(find mcr_description)/urdf/sensors/microsoft_lifecam_1080_mount.urdf.xacro"/>
+  <xacro:include filename="$(find mcr_description)/urdf/mounts/microsoft_lifecam_1080_mount.urdf.xacro"/>
   <xacro:include filename="$(find mcr_description)/urdf/materials.urdf.xacro" />
+  <xacro:include filename="$(find mir_description)/urdf/grippers/festo_gripper.urdf.xacro" />
   <!-- base laser front -->
   <xacro:hokuyo_urg04_laser name="base_laser_front" parent="base" ros_topic="scan_front" update_rate="10" min_angle="-1.57" max_angle="1.57">
@@ -59,3 +55,6 @@
     <origin xyz="-0.035 0.0 -0.025" rpy="0 0 3.14159265" />
   </xacro:microsoft_lifecam_1080_mount>
+  <xacro:festo_gripper name="gripper" parent="arm_link_5">
+    <origin xyz="0 0 0" rpy="0 0 0" />
+  </xacro:festo_gripper>
 </robot>

Commit message: adapt arm position which is now 3cm higher and 6cm more to the front. replace default youbot rear platform with the BRSU customized one

File: mir_robots/mir_hardware_config/youbot-brsu-2/urdf/robot.urdf.xacro (robot description, xacro)
@@ -23,9 +23,12 @@
   <!-- standard youBot configuration -->
   <xacro:youbot_base name="base"/>
-  <xacro:youbot_plate name="plate" parent="base_link">
+  <!--xacro:youbot_plate name="plate" parent="base_link">
     <origin xyz="-0.159 0 0.046" rpy="0 0 0" />
-  </xacro:youbot_plate>
+  </xacro:youbot_plate-->
+  <xacro:rear_platform name="rear_platform" parent="base_link">
+    <origin xyz="-0.005 -0.175 0.051" rpy="0 0 0" />
+  </xacro:rear_platform>
   <xacro:youbot_arm name="arm" parent="base_link">
-    <origin xyz="0.143 0 0.046" rpy="0 0 0" />
+    <origin xyz="0.223 0 0.076" rpy="0 0 0" />
   </xacro:youbot_arm>
   <!-- BRSU SPECIFIC STUFF -->
@@ -35,4 +38,5 @@
   <xacro:include filename="$(find mcr_description)/urdf/materials.urdf.xacro" />
   <xacro:include filename="$(find mir_description)/urdf/grippers/festo_gripper.urdf.xacro" />
+  <xacro:include filename="$(find mir_description)/urdf/misc/rear_platform.urdf.xacro" />
   <!-- base laser front -->
   <xacro:hokuyo_urg04_laser name="base_laser_front" parent="base" ros_topic="scan_front" update_rate="10" min_angle="-1.57" max_angle="1.57">

Commit message: calibrate camera tower position

File: mir_robots/mir_hardware_config/youbot-brsu-2/urdf/robot.urdf.xacro (robot description, xacro)
@@ -48,6 +48,6 @@
   </xacro:hokuyo_urg04_laser>
   <!-- camera tower -->
-  <xacro:camera_tower name="camera_tower" parent="plate_link">
-    <origin xyz="-0.075 0.0 0.023" rpy="0 0 0" />
+  <xacro:camera_tower name="camera_tower" parent="rear_platform_link">
+    <origin xyz="-0.227 0.165 0.023" rpy="0 0 0" />
   </xacro:camera_tower>
   <!-- 3D camera on tower -->

Commit message: included new adapter plate to youbot-2
origin of new adapter plate, the centre of the mounting location, is 0.159 + 0.08
0.159 from the orignal centre of youbot rear place, which i removed, plus 8cm forward offset.

increased arm offset in z and y. the origin of arm_0 does not line up with the origin of the arm mount.
This offset to my best estimate +/- 2mm. I will add images to issue mas-group/mas_industrial_robotics#64

this should close #64

File: mir_robots/mir_hardware_config/youbot-brsu-2/urdf/robot.urdf.xacro (robot description, xacro)
@@ -23,12 +23,9 @@
   <!-- standard youBot configuration -->
   <xacro:youbot_base name="base"/>
-  <!--xacro:youbot_plate name="plate" parent="base_link">
-    <origin xyz="-0.159 0 0.046" rpy="0 0 0" />
-  </xacro:youbot_plate-->
   <xacro:rear_platform name="rear_platform" parent="base_link">
     <origin xyz="-0.005 -0.175 0.051" rpy="0 0 0" />
   </xacro:rear_platform>
   <xacro:youbot_arm name="arm" parent="base_link">
-    <origin xyz="0.223 0 0.076" rpy="0 0 0" />
+    <origin xyz="0.223 0.017 0.088" rpy="0 0 ${-M_PI / 4}" />
   </xacro:youbot_arm>
   <!-- BRSU SPECIFIC STUFF -->
@@ -39,4 +36,8 @@
   <xacro:include filename="$(find mir_description)/urdf/grippers/festo_gripper.urdf.xacro" />
   <xacro:include filename="$(find mir_description)/urdf/misc/rear_platform.urdf.xacro" />
+  <xacro:include filename="$(find mir_description)/urdf/misc/adapter_plate.urdf.xacro" />
+  <xacro:adapter_plate name="adapter_plate" parent="base_link">
+    <origin xyz="${0.159+0.08} 0 0.051" rpy="0 0 0" />
+  </xacro:adapter_plate>
   <!-- base laser front -->
   <xacro:hokuyo_urg04_laser name="base_laser_front" parent="base" ros_topic="scan_front" update_rate="10" min_angle="-1.57" max_angle="1.57">
