Commit message: [robot] update URDF and launch file of yb2

File: mir_robots/mir_hardware_config/youbot-brsu-2/urdf/robot.urdf.xacro (robot description, xacro)
@@ -5,15 +5,15 @@
        xmlns:xacro="http://playerstage.sourceforge.net/gazebo/xmlschema/#interface"
        name="youbot" >
-  <!-- The following included files set up definitions of parts of the robot body -->
-  <!-- misc common stuff -->
+  <!-- The following xacro:included files set up definitions of parts of the robot body -->
+  <!-- misc common stuff? -->
   <xacro:include filename="$(find youbot_description)/urdf/common.xacro" />
-  <xacro:include filename="$(find mcr_description)/urdf/materials.urdf.xacro" />
-  <!-- youbot base and rear platform -->
+  <!-- youbot base -->
   <xacro:include filename="$(find youbot_description)/urdf/youbot_base/base.urdf.xacro" />
-  <xacro:include filename="$(find mir_description)/urdf/misc/rear_platform.urdf.xacro" />
-  <!-- youbot arm and gripper-->
+  <!-- youbot plate -->
+  <xacro:include filename="$(find youbot_description)/urdf/youbot_plate/plate.urdf.xacro" />
+  <!-- youbot arm -->
   <xacro:include filename="$(find youbot_description)/urdf/youbot_arm/arm.urdf.xacro"/>
-  <xacro:include filename="$(find mir_description)/urdf/misc/adapter_plate.urdf.xacro" />
-  <xacro:include filename="$(find mir_description)/urdf/grippers/festo_gripper.urdf.xacro" />
+  <!-- youbot gripper -->
+  <xacro:include filename="$(find youbot_description)/urdf/youbot_gripper/gripper.urdf.xacro" />
   <!-- controller manager -->
   <xacro:include filename="$(find youbot_description)/controller/ros_controller.urdf.xacro" />
@@ -22,33 +22,14 @@
   <!-- sensors -->
   <xacro:include filename="$(find youbot_description)/urdf/sensors/hokuyo_urg04_laser.urdf.xacro"/>
-  <xacro:include filename="$(find mcr_description)/urdf/sensors/asus_xtion_camera.urdf.xacro"/>
-  <!-- Now we can start using the macros included above to define the actual youbot -->
-  <!-- standard youBot configuration -->
+  <!-- foot for arm-->
   <xacro:youbot_base name="base"/>
-  <!-- Rear Platform -->
-  <xacro:rear_platform name="rear_platform" parent="base_link">
-    <origin xyz="-0.005 -0.175 0.051" rpy="0 0 0" />
-  </xacro:rear_platform>
-  <!-- Arm Plate moving arm 8cm foward and 45 degree rotation -->
-  <xacro:adapter_plate name="adapter_plate" parent="base_link" arm_angle="${-M_PI / 4}">
-    <origin xyz="${0.159+0.08} 0 0.051" rpy="0 0 0" />
-  </xacro:adapter_plate>
-  <xacro:youbot_arm name="arm" parent="adapter_plate_arm_root_link">
-    <origin xyz="-0.022 0.0 0.037" rpy="0 0 0" />
+  <xacro:youbot_plate name="plate" parent="base_link">
+    <origin xyz="-0.159 0 0.046" rpy="0 0 0" />
+  </xacro:youbot_plate>
+  <xacro:youbot_arm name="arm" parent="base_link">
+    <origin xyz="0.143 0 0.046" rpy="0 0 0" />
   </xacro:youbot_arm>
-  <!-- base laser front -->
-  <xacro:hokuyo_urg04_laser name="base_laser_front" parent="base" ros_topic="scan_front" update_rate="10" min_angle="-1.57" max_angle="1.57">
-    <origin xyz="0.3 0 -0.03" rpy="0 0 0"/>
-  </xacro:hokuyo_urg04_laser>
-  <!-- base laser rear -->
-  <xacro:hokuyo_urg04_laser name="base_laser_rear" parent="base" ros_topic="scan_rear" update_rate="10" min_angle="-1.57" max_angle="1.57" >
-     <origin xyz="-0.3 0.0 -0.03" rpy="0 0 ${M_PI}" />
-  </xacro:hokuyo_urg04_laser>
-  <!-- 3D camera on arm --> <!-- NOTE: still called tower_cam3d due to legacy code -->
-  <xacro:asus_xtion_camera name="tower_cam3d" parent="arm_link_5" tilt="0.0">
-    <origin xyz="${-0.035 - 0.030 + 0.030} ${0 - 0.015} ${-0.09}" rpy="0 ${-M_PI / 2} 0" />
-  </xacro:asus_xtion_camera>
-  <xacro:festo_gripper name="gripper" parent="arm_link_5">
+  <xacro:youbot_gripper name="gripper" parent="arm_link_5">
     <origin xyz="0 0 0" rpy="0 0 0" />
-  </xacro:festo_gripper>
+  </xacro:youbot_gripper>
 </robot>

Commit message: [hardware config] use urdf from yb4 for yb2

File: mir_robots/mir_hardware_config/youbot-brsu-2/urdf/robot.urdf.xacro (robot description, xacro)
@@ -5,15 +5,15 @@
        xmlns:xacro="http://playerstage.sourceforge.net/gazebo/xmlschema/#interface"
        name="youbot" >
-  <!-- The following xacro:included files set up definitions of parts of the robot body -->
-  <!-- misc common stuff? -->
+  <!-- The following included files set up definitions of parts of the robot body -->
+  <!-- misc common stuff -->
   <xacro:include filename="$(find youbot_description)/urdf/common.xacro" />
-  <!-- youbot base -->
+  <xacro:include filename="$(find mcr_description)/urdf/materials.urdf.xacro" />
+  <!-- youbot base and rear platform -->
   <xacro:include filename="$(find youbot_description)/urdf/youbot_base/base.urdf.xacro" />
-  <!-- youbot plate -->
-  <xacro:include filename="$(find youbot_description)/urdf/youbot_plate/plate.urdf.xacro" />
-  <!-- youbot arm -->
+  <xacro:include filename="$(find mir_description)/urdf/misc/rear_platform_v2.urdf.xacro" />
+  <!-- youbot arm and gripper-->
   <xacro:include filename="$(find youbot_description)/urdf/youbot_arm/arm.urdf.xacro"/>
-  <!-- youbot gripper -->
-  <xacro:include filename="$(find youbot_description)/urdf/youbot_gripper/gripper.urdf.xacro" />
+  <xacro:include filename="$(find mir_description)/urdf/misc/adapter_plate.urdf.xacro" />
+  <xacro:include filename="$(find mir_description)/urdf/grippers/dynamixel/v2/dynamixel_gripper.urdf.xacro" />
   <!-- controller manager -->
   <xacro:include filename="$(find youbot_description)/controller/ros_controller.urdf.xacro" />
@@ -22,14 +22,38 @@
   <!-- sensors -->
   <xacro:include filename="$(find youbot_description)/urdf/sensors/hokuyo_urg04_laser.urdf.xacro"/>
-  <!-- foot for arm-->
+  <xacro:include filename="$(find mir_description)/urdf/sensor_mounts/intel_f200_camera_mount.urdf.xacro"/>
+  <xacro:include filename="$(find mcr_description)/urdf/sensors/intel_realsense_f200_camera.urdf.xacro"/>
+  <!-- Now we can start using the macros included above to define the actual youbot -->
+  <!-- standard youBot configuration -->
   <xacro:youbot_base name="base"/>
-  <xacro:youbot_plate name="plate" parent="base_link">
-    <origin xyz="-0.159 0 0.046" rpy="0 0 0" />
-  </xacro:youbot_plate>
-  <xacro:youbot_arm name="arm" parent="base_link">
-    <origin xyz="0.143 0 0.046" rpy="0 0 0" />
+  <!-- Rear Platform -->
+  <xacro:rear_platform_v2 name="rear_platform" parent="base_link">
+    <origin xyz="0.12 -0.175 ${0.021 + 0.0062 + 0.025 + 0.012}" rpy="0 0 0" />  <!-- ${alignment with base top + nut height + spacer height + slide height } -->
+  </xacro:rear_platform_v2>
+  <!-- Arm Plate moving arm 8cm foward and 45 degree rotation -->
+  <xacro:adapter_plate name="adapter_plate" parent="base_link" arm_angle="${-M_PI / 4}">
+    <origin xyz="${0.159+0.08} 0 ${0.021 + 0.025 + 0.025}" rpy="0 0 0" />    <!-- ${alignment with base top + spacer height + spacer height } -->
+  </xacro:adapter_plate>
+  <xacro:youbot_arm name="arm" parent="adapter_plate_arm_root_link">
+    <origin xyz="-0.022 0.0 0.037" rpy="0 0 0" />
   </xacro:youbot_arm>
-  <xacro:youbot_gripper name="gripper" parent="arm_link_5">
-    <origin xyz="0 0 0" rpy="0 0 0" />
-  </xacro:youbot_gripper>
+  <!-- base laser front -->
+  <xacro:hokuyo_urg04_laser name="base_laser_front" parent="base" ros_topic="scan_front" update_rate="10" min_angle="-1.57" max_angle="1.57">
+    <origin xyz="0.3 0 -0.035" rpy="${M_PI} 0 0"/>
+  </xacro:hokuyo_urg04_laser>
+  <!-- base laser rear -->
+  <xacro:hokuyo_urg04_laser name="base_laser_rear" parent="base" ros_topic="scan_rear" update_rate="10" min_angle="-1.57" max_angle="1.57" >
+     <origin xyz="-0.3 0.0 -0.035" rpy="${M_PI} 0 ${M_PI}" />
+  </xacro:hokuyo_urg04_laser>
+  <xacro:dynamixel_gripper_v2 name="gripper" parent="arm_link_5">
+    <origin xyz="0.003 0 0.0052" rpy="0 0 0" />
+  </xacro:dynamixel_gripper_v2>
+  <!-- camera mount for Intel RealSense F200 -->
+  <xacro:intel_f200_camera_mount name="camera_mount" parent="gripper_motor_mount_link">
+    <origin xyz="-0.00375 -0.0007 0.012" rpy="-0.05 -0.04 0" />
+  </xacro:intel_f200_camera_mount>
+  <!-- 3D camera on arm -->
+  <xacro:intel_realsense_f200_camera name="arm_cam3d" parent="camera_mount_link">
+    <origin xyz="-0.0405 0.0 0.029" rpy="0 -${M_PI/2} 0" />
+  </xacro:intel_realsense_f200_camera>
 </robot>

Commit message: [hardware config] calibrate Intel cam pose

File: mir_robots/mir_hardware_config/youbot-brsu-2/urdf/robot.urdf.xacro (robot description, xacro)
@@ -51,5 +51,5 @@
   <!-- camera mount for Intel RealSense F200 -->
   <xacro:intel_f200_camera_mount name="camera_mount" parent="gripper_motor_mount_link">
-    <origin xyz="-0.00375 -0.0007 0.012" rpy="-0.05 -0.04 0" />
+    <origin xyz="-0.00375 -0.0007 0.012" rpy="-0.03 -0.04 0" />
   </xacro:intel_f200_camera_mount>
   <!-- 3D camera on arm -->

Commit message: [hardware config] calibrate intel cam pose

File: mir_robots/mir_hardware_config/youbot-brsu-2/urdf/robot.urdf.xacro (robot description, xacro)
@@ -55,5 +55,5 @@
   <!-- 3D camera on arm -->
   <xacro:intel_realsense_f200_camera name="arm_cam3d" parent="camera_mount_link">
-    <origin xyz="-0.0405 0.0 0.029" rpy="0 -${M_PI/2} 0" />
+    <origin xyz="-0.0405 0.0 0.03" rpy="-0.1 -${M_PI/2} 0" />
   </xacro:intel_realsense_f200_camera>
 </robot>

Commit message: [urdf] camera calibration

File: mir_robots/mir_hardware_config/youbot-brsu-2/urdf/robot.urdf.xacro (robot description, xacro)
@@ -51,9 +51,9 @@
   <!-- camera mount for Intel RealSense F200 -->
   <xacro:intel_f200_camera_mount name="camera_mount" parent="gripper_motor_mount_link">
-    <origin xyz="-0.00375 -0.0007 0.012" rpy="-0.03 -0.04 0" />
+    <origin xyz="-0.00375 -0.0007 0.012" rpy="-0.05 -0.04 0" />
   </xacro:intel_f200_camera_mount>
   <!-- 3D camera on arm -->
   <xacro:intel_realsense_f200_camera name="arm_cam3d" parent="camera_mount_link">
-    <origin xyz="-0.0405 0.0 0.03" rpy="-0.1 -${M_PI/2} 0" />
+    <origin xyz="-0.035 0.0 0.015" rpy="-0.02 -${M_PI/2} -0.02" />
   </xacro:intel_realsense_f200_camera>
 </robot>

File: mir_robots/mir_hardware_config/youbot-brsu-4/urdf/robot.urdf.xacro (robot description, xacro)
@@ -55,5 +55,5 @@
   <!-- 3D camera on arm -->
   <xacro:intel_realsense_f200_camera name="arm_cam3d" parent="camera_mount_link">
-    <origin xyz="-0.0405 -0.008 0.025" rpy="-0.2 -${M_PI/2} 0" />
+    <origin xyz="-0.05 -0.03 0.03" rpy="0.3 -${M_PI/2 - 0.03} -0.25" />
   </xacro:intel_realsense_f200_camera>
 </robot>

Commit message: [yb2-calib] camera calibration

File: mir_robots/mir_hardware_config/youbot-brsu-2/urdf/robot.urdf.xacro (robot description, xacro)
@@ -55,5 +55,5 @@
   <!-- 3D camera on arm -->
   <xacro:intel_realsense_f200_camera name="arm_cam3d" parent="camera_mount_link">
-    <origin xyz="-0.035 0.0 0.015" rpy="-0.02 -${M_PI/2} -0.02" />
+    <origin xyz="-0.03 -0.00 0.00" rpy="0.0 -${M_PI/2} 0.0" />
   </xacro:intel_realsense_f200_camera>
 </robot>

Commit message: [urdf] camera calibration

File: mir_robots/mir_hardware_config/youbot-brsu-2/urdf/robot.urdf.xacro (robot description, xacro)
@@ -51,9 +51,9 @@
   <!-- camera mount for Intel RealSense F200 -->
   <xacro:intel_f200_camera_mount name="camera_mount" parent="gripper_motor_mount_link">
-    <origin xyz="-0.00375 -0.0007 0.012" rpy="-0.05 -0.04 0" />
+    <origin xyz="-0.00375 -0.0007 0.012" rpy="0.06 -0.04 0" />
   </xacro:intel_f200_camera_mount>
   <!-- 3D camera on arm -->
   <xacro:intel_realsense_f200_camera name="arm_cam3d" parent="camera_mount_link">
-    <origin xyz="-0.03 -0.00 0.00" rpy="0.0 -${M_PI/2} 0.0" />
+    <origin xyz="-0.045 -0.00 0.00" rpy="0.0 -${M_PI/2} 0.0" />
   </xacro:intel_realsense_f200_camera>
 </robot>

File: mir_robots/mir_hardware_config/youbot-brsu-4/urdf/robot.urdf.xacro (robot description, xacro)
@@ -51,9 +51,9 @@
   <!-- camera mount for Intel RealSense F200 -->
   <xacro:intel_f200_camera_mount name="camera_mount" parent="gripper_motor_mount_link">
-    <origin xyz="-0.00375 -0.0007 0.012" rpy="-0.05 -0.04 0" />
+    <origin xyz="-0.00375 -0.0007 0.012" rpy="0.04 -0.04 0" />
   </xacro:intel_f200_camera_mount>
   <!-- 3D camera on arm -->
   <xacro:intel_realsense_f200_camera name="arm_cam3d" parent="camera_mount_link">
-    <origin xyz="-0.03 0.0 0.03" rpy="0.3 -${M_PI/2 - 0.03} -0.2" />
+    <origin xyz="-0.05 0.0 0.03" rpy="0.0 -${M_PI/2 - 0.03} 0.0" />
   </xacro:intel_realsense_f200_camera>
 </robot>

Commit message: [URDF] updating urdf with full back platform
The platform is visual represented as a box and not as dae.
Tested only on rviz.

File: mir_robots/mir_hardware_config/youbot-brsu-2/urdf/robot.urdf.xacro (robot description, xacro)
@@ -14,5 +14,5 @@
   <!-- youbot arm and gripper-->
   <xacro:include filename="$(find youbot_description)/urdf/youbot_arm/arm.urdf.xacro"/>
-  <xacro:include filename="$(find mir_description)/urdf/misc/adapter_plate.urdf.xacro" />
+  <xacro:include filename="$(find mir_description)/urdf/misc/full_platform.urdf.xacro" />
   <xacro:include filename="$(find mir_description)/urdf/grippers/dynamixel/v2/dynamixel_gripper.urdf.xacro" />
   <!-- controller manager -->
@@ -24,16 +24,14 @@
   <xacro:include filename="$(find mir_description)/urdf/sensor_mounts/intel_f200_camera_mount.urdf.xacro"/>
   <xacro:include filename="$(find mcr_description)/urdf/sensors/intel_realsense_f200_camera.urdf.xacro"/>
+  <xacro:include filename="$(find mir_description)/urdf/sensors/asus_xtion_camera.urdf.xacro"/>
+  <xacro:include filename="$(find mir_description)/urdf/sensor_mounts/asus_xtion_camera_mount.urdf.xacro"/>
   <!-- Now we can start using the macros included above to define the actual youbot -->
   <!-- standard youBot configuration -->
   <xacro:youbot_base name="base"/>
-  <!-- Rear Platform -->
-  <xacro:rear_platform_v2 name="rear_platform" parent="base_link">
-    <origin xyz="0.12 -0.175 ${0.021 + 0.0062 + 0.025 + 0.012}" rpy="0 0 0" />  <!-- ${alignment with base top + nut height + spacer height + slide height } -->
-  </xacro:rear_platform_v2>
   <!-- Arm Plate moving arm 8cm foward and 45 degree rotation -->
-  <xacro:adapter_plate name="adapter_plate" parent="base_link" arm_angle="${-M_PI / 4}">
-    <origin xyz="${0.159+0.08} 0 ${0.021 + 0.025 + 0.025}" rpy="0 0 0" />    <!-- ${alignment with base top + spacer height + spacer height } -->
-  </xacro:adapter_plate>
-  <xacro:youbot_arm name="arm" parent="adapter_plate_arm_root_link">
+  <xacro:full_platform name="full_platform" parent="base_link" arm_angle="${-M_PI / 4}">
+    <origin xyz="0.0 0.0 ${0.021 + 0.025 + 0.025}" rpy="0 0 0" />    <!-- ${alignment with base top + spacer height + spacer height } -->
+  </xacro:full_platform>
+  <xacro:youbot_arm name="arm" parent="full_platform_arm_root_link">
     <origin xyz="-0.022 0.0 0.037" rpy="0 0 0" />
   </xacro:youbot_arm>
@@ -50,10 +48,16 @@
   </xacro:dynamixel_gripper_v2>
   <!-- camera mount for Intel RealSense F200 -->
-  <xacro:intel_f200_camera_mount name="camera_mount" parent="gripper_motor_mount_link">
-    <origin xyz="-0.00375 -0.0007 0.012" rpy="0.06 -0.04 0" />
-  </xacro:intel_f200_camera_mount>
+  <xacro:asus_xtion_camera_mount  name="camera_mount" parent="gripper_motor_mount_link">
+      <origin xyz="0.035 -0.00 0.0" rpy="0 0.025 ${M_PI/2} " />
+  </xacro:asus_xtion_camera_mount>
   <!-- 3D camera on arm -->
-  <xacro:intel_realsense_f200_camera name="arm_cam3d" parent="camera_mount_link">
-    <origin xyz="-0.045 -0.00 0.00" rpy="0.0 -${M_PI/2} 0.0" />
-  </xacro:intel_realsense_f200_camera>
+  <!-- xacro:intel_realsense_f200_camera name="arm_cam3d" parent="camera_mount_link">
+    <origin xyz="-0.05 -0.01 0.03" rpy="0.0 -${M_PI/2 - 0.03} 0.0" />
+  </xacro:intel_realsense_f200_camera -->
+   <xacro:asus_xtion_camera name="arm_cam3d" parent="camera_mount_link">
+       <!--origin xyz="-0.01 -0.012 0.05" rpy="0 ${M_PI/2 - 0.25} 0.00" /-->
+       <!--origin xyz="0.016 0 0.01" rpy="0 ${M_PI/2 - 0} -0.09" />  -->
+   <origin xyz="0.010 -0.022 0.017" rpy="0 ${M_PI/2 - 0.18} -${M_PI/2}" />
+       <!--origin xyz="0.023 -0.015 0.03" rpy="0 0 0" /-->
+   </xacro:asus_xtion_camera>
 </robot>

Commit message: [urdf] Fixed inverted laser

File: mir_robots/mir_hardware_config/youbot-brsu-2/urdf/robot.urdf.xacro (robot description, xacro)
@@ -39,9 +39,9 @@
   <!-- base laser front -->
   <xacro:hokuyo_urg04_laser name="base_laser_front" parent="base" ros_topic="scan_front" update_rate="10" min_angle="-1.57" max_angle="1.57">
-    <origin xyz="0.3 0 -0.035" rpy="${M_PI} 0 0"/>
+    <origin xyz="0.3 0 -0.035" rpy="0 0 0"/>
   </xacro:hokuyo_urg04_laser>
   <!-- base laser rear -->
   <xacro:hokuyo_urg04_laser name="base_laser_rear" parent="base" ros_topic="scan_rear" update_rate="10" min_angle="-1.57" max_angle="1.57" >
-     <origin xyz="-0.3 0.0 -0.035" rpy="${M_PI} 0 ${M_PI}" />
+     <origin xyz="-0.3 0.0 -0.035" rpy="0 0 ${M_PI}" />
   </xacro:hokuyo_urg04_laser>
   <xacro:dynamixel_gripper_v2 name="gripper" parent="arm_link_5">

Commit message: [perception][description] Fixed tower cam and arm cam name issue

File: mir_robots/mir_hardware_config/youbot-brsu-2/urdf/robot.urdf.xacro (robot description, xacro)
@@ -57,7 +57,9 @@
     <origin xyz="-0.05 -0.01 0.03" rpy="0.0 -${M_PI/2 - 0.03} 0.0" />
   </xacro:intel_realsense_f200_camera -->
-   <xacro:realsense_d435 name="arm_cam3d" parent="base_link">
-       <!--origin xyz="0.25 0.0 0.83" rpy="-0.05 0.917 -0.1" /-->
+   <xacro:realsense_d435 name="tower_cam3d" parent="base_link">
        <origin xyz="0.30 -0.05 0.80" rpy="0.00 1.137 0.0" />
+   </xacro:realsense_d435>
+   <xacro:realsense_d435  name="arm_cam3d" parent="arm_link_5">
+      <origin xyz="-0.005 -0.008 0.009" rpy="0.0 ${-M_PI / 2} ${-M_PI / 2}" />
    </xacro:realsense_d435>
    <joint name="fixed_camera_joint" type="fixed">

Commit message: [hardware_config] Tuned torso camera tf

File: mir_robots/mir_hardware_config/youbot-brsu-2/urdf/robot.urdf.xacro (robot description, xacro)
@@ -58,5 +58,5 @@
   </xacro:intel_realsense_f200_camera -->
    <xacro:realsense_d435 name="tower_cam3d" parent="base_link">
-       <origin xyz="0.30 -0.05 0.80" rpy="0.00 1.137 0.0" />
+       <origin xyz="0.298 -0.039 0.795" rpy="-0.055 1.16 0.0" />
    </xacro:realsense_d435>
    <xacro:realsense_d435  name="arm_cam3d" parent="arm_link_5">

Commit message: [ybrsu2 urdf] added camera stand and adjusted gripper mount

File: mir_robots/mir_hardware_config/youbot-brsu-2/urdf/robot.urdf.xacro (robot description, xacro)
@@ -8,5 +8,5 @@
   <!-- misc common stuff -->
   <xacro:include filename="$(find youbot_description)/urdf/common.xacro" />
-  <xacro:include filename="$(find mcr_description)/urdf/materials.urdf.xacro" />
+  <xacro:include filename="$(find mir_description)/urdf/materials.urdf.xacro" />
   <!-- youbot base and rear platform -->
   <xacro:include filename="$(find youbot_description)/urdf/youbot_base/base.urdf.xacro" />
@@ -24,7 +24,7 @@
   <xacro:include filename="$(find youbot_description)/urdf/sensors/hokuyo_urg04_laser.urdf.xacro"/>
   <xacro:include filename="$(find mir_description)/urdf/sensor_mounts/intel_f200_camera_mount.urdf.xacro"/>
-  <xacro:include filename="$(find mcr_description)/urdf/sensors/intel_realsense_f200_camera.urdf.xacro"/>
+  <xacro:include filename="$(find mir_description)/urdf/sensors/intel_realsense_f200_camera.urdf.xacro"/>
   <xacro:include filename="$(find mir_description)/urdf/sensors/asus_xtion_camera.urdf.xacro"/>
-  <xacro:include filename="$(find mcr_description)/urdf/sensors/realsense_d435.urdf.xacro"/>
+  <xacro:include filename="$(find mir_description)/urdf/sensors/realsense_d435.urdf.xacro"/>
   <xacro:include filename="$(find mir_description)/urdf/sensor_mounts/asus_xtion_camera_mount.urdf.xacro"/>
   <!-- Now we can start using the macros included above to define the actual youbot -->
@@ -82,3 +82,45 @@
        </collision>
    </link>
+  <!-- tower camera stand link -->
+  <link name="tower_camera_stand_link">
+    <visual>
+      <geometry>
+        <box size="0.025 0.025 0.80"/>
+      </geometry>
+      <material name="">
+          <color rgba="0.85098 0.85098 0.85098 1"/>
+      </material>
+    </visual>
+    <collision>
+      <geometry>
+        <box size="0.025 0.025 0.80"/>
+      </geometry>
+    </collision>
+  </link>
+  <joint name="tower_camera_stand_joint" type="fixed">
+    <origin xyz="-0.10 0.0 0.40" rpy="0 0 0" />
+    <parent link="full_platform_link"/>
+    <child link="tower_camera_stand_link"/>
+  </joint>
+  <!-- tower camera mount link -->
+  <link name="tower_camera_stand_link_2">
+    <visual>
+      <geometry>
+        <box size="0.025 0.025 0.44"/>
+      </geometry>
+      <material name="">
+          <color rgba="0.85098 0.85098 0.85098 1"/>
+      </material>
+    </visual>
+    <collision>
+      <geometry>
+        <box size="0.025 0.025 0.44"/>
+      </geometry>
+    </collision>
+  </link>
+  <joint name="tower_camera_stand_joint_2" type="fixed">
+    <origin xyz="0.16 0.0 0.31" rpy="0 ${M_PI/2} 0" />
+    <parent link="tower_camera_stand_link"/>
+    <child link="tower_camera_stand_link_2"/>
+  </joint>
 </robot>
