Commit message: [mir_hardware_config] added 3 tower cameras and emergency button mounts

File: mir_robots/mir_hardware_config/youbot-brsu-2/urdf/robot.urdf.xacro (robot description, xacro)
@@ -57,4 +57,5 @@
     <origin xyz="-0.05 -0.01 0.03" rpy="0.0 -${M_PI/2 - 0.03} 0.0" />
   </xacro:intel_realsense_f200_camera -->
+  <!-- tower front camera -->
    <xacro:realsense_d435 name="tower_cam3d" parent="base_link">
        <origin xyz="0.328 -0.039 0.795" rpy="-0.055 1.212 -0.052" />
@@ -84,3 +85,129 @@
        </collision>
    </link>
+   <!-- tower vertical mount link -->
+  <link name="tower_camera_stand_link">
+    <visual>
+      <geometry>
+        <box size="0.030 0.030 0.80"/>
+      </geometry>
+      <material name="">
+          <color rgba="0.85098 0.85098 0.85098 1"/>
+      </material>
+    </visual>
+    <collision>
+      <geometry>
+        <box size="0.030 0.030 0.80"/>
+      </geometry>
+    </collision>
+  </link>
+  <joint name="tower_camera_stand_joint" type="fixed">
+    <origin xyz="-0.10 0.0 0.40" rpy="0 0 0" />
+    <parent link="full_platform_link"/>
+    <child link="tower_camera_stand_link"/>
+  </joint>
+  <!-- link for emergency stop mount with stl mesh file -->
+  <link name="emergency_stop_mount_link">
+    <visual>
+      <geometry>
+        <mesh filename="package://mir_description/meshes/e_stop_mount.STL" scale="0.001 0.001 0.001"/>
+      </geometry>
+      <material name="">
+          <color rgba="0.85098 0.85098 0.85098 1"/>
+      </material>
+    </visual>
+    <collision>
+      <geometry>
+        <mesh filename="package://mir_description/meshes/e_stop_mount.STL" scale="0.001 0.001 0.001"/>
+      </geometry>
+    </collision>
+  </link>
+  <joint name="emergency_stop_mount_joint" type="fixed">
+    <origin xyz="0.0 0.0 0.40" rpy="${pi/2} 0 0" />
+    <parent link="tower_camera_stand_link"/>
+    <child link="emergency_stop_mount_link"/>
+  </joint>
+  <!-- tower horizontal mount link -->
+  <link name="tower_camera_stand_link_horizontal">
+    <visual>
+      <geometry>
+        <box size="0.030 0.030 0.608"/>
+      </geometry>
+      <material name="">
+          <color rgba="0.85098 0.85098 0.85098 1"/>
+      </material>
+    </visual>
+    <collision>
+      <geometry>
+        <box size="0.030 0.030 0.608"/>
+      </geometry>
+    </collision>
+  </link>
+  <joint name="tower_camera_stand_joint_horizontal" type="fixed">
+    <origin xyz="0.09 -0.035 0.362" rpy="0 ${M_PI/2} 0" />
+    <parent link="tower_camera_stand_link"/>
+    <child link="tower_camera_stand_link_horizontal"/>
+  </joint>
+  <!-- tower front camera mount link -->
+  <link name="tower_camera_front_mount_link">
+    <visual>
+      <geometry>
+        <mesh filename="package://mir_description/meshes/intel_camera_mount.STL" scale="0.001 0.001 0.001"/>
+      </geometry>
+      <material name="">
+          <color rgba="0.85098 0.85098 0.85098 1"/>
+      </material>
+    </visual>
+    <collision>
+      <geometry>
+        <mesh filename="package://mir_description/meshes/intel_camera_mount.STL" scale="0.001 0.001 0.001"/>
+      </geometry>
+    </collision>
+  </link>
+  <joint name="tower_camera_front_mount_joint" type="fixed">
+    <origin xyz="0.0 0.0 0.304" rpy="-${M_PI/2} ${M_PI/2} 0" />
+    <parent link="tower_camera_stand_link_horizontal"/>
+    <child link="tower_camera_front_mount_link"/>
+  </joint>
+  <!-- tower back camera mount link -->
+  <link name="tower_camera_back_mount_link">
+    <visual>
+      <geometry>
+        <mesh filename="package://mir_description/meshes/intel_camera_mount.STL" scale="0.001 0.001 0.001"/>
+      </geometry>
+      <material name="">
+          <color rgba="0.85098 0.85098 0.85098 1"/>
+      </material>
+    </visual>
+    <collision>
+      <geometry>
+        <mesh filename="package://mir_description/meshes/intel_camera_mount.STL" scale="0.001 0.001 0.001"/>
+      </geometry>
+    </collision>
+  </link>
+  <joint name="tower_camera_back_mount_joint" type="fixed">
+    <origin xyz="0.0 0.0 -0.304" rpy="${M_PI} -${M_PI/2} -${M_PI/2}" />
+    <parent link="tower_camera_stand_link_horizontal"/>
+    <child link="tower_camera_back_mount_link"/>
+  </joint>
+  <!-- tower side camera mount link -->
+  <link name="tower_camera_side_mount_link">
+    <visual>
+      <geometry>
+        <mesh filename="package://mir_description/meshes/side_camera_mount.STL" scale="0.001 0.001 0.001"/>
+      </geometry>
+      <material name="">
+          <color rgba="0.85098 0.85098 0.85098 1"/>
+      </material>
+    </visual>
+    <collision>
+      <geometry>
+        <mesh filename="package://mir_description/meshes/side_camera_mount.STL" scale="0.001 0.001 0.001"/>
+      </geometry>
+    </collision>
+  </link>
+  <joint name="tower_camera_side_mount_joint" type="fixed">
+    <origin xyz="0.0 0.0 0.149" rpy="${M_PI/2} -${M_PI/2} 0" />
+    <parent link="tower_camera_stand_link_horizontal"/>
+    <child link="tower_camera_side_mount_link"/>
+  </joint>
 </robot>

Commit message: [mir_hardware_config] added side camera | orbbec astra

File: mir_robots/mir_hardware_config/youbot-brsu-2/urdf/robot.urdf.xacro (robot description, xacro)
@@ -27,4 +27,5 @@
   <xacro:include filename="$(find mir_description)/urdf/sensors/asus_xtion_camera.urdf.xacro"/>
   <xacro:include filename="$(find mcr_description)/urdf/sensors/realsense_d435.urdf.xacro"/>
+  <xacro:include filename="$(find youbot_description)/urdf/sensors/orbbec_astra.urdf.xacro"/>
   <xacro:include filename="$(find mir_description)/urdf/sensor_mounts/asus_xtion_camera_mount.urdf.xacro"/>
   <!-- Now we can start using the macros included above to define the actual youbot -->
@@ -58,20 +59,25 @@
   </xacro:intel_realsense_f200_camera -->
   <!-- tower front camera -->
-   <xacro:realsense_d435 name="tower_cam3d" parent="base_link">
-       <origin xyz="0.328 -0.039 0.795" rpy="-0.055 1.212 -0.052" />
-   </xacro:realsense_d435>
-   <xacro:realsense_d435  name="arm_cam3d" parent="arm_link_5">
-      <origin xyz="-0.005 -0.008 0.009" rpy="0.0 ${-M_PI / 2} ${-M_PI / 2}" />
-   </xacro:realsense_d435>
-   <joint name="fixed_camera_joint" type="fixed">
+  <xacro:realsense_d435 name="tower_cam3d_front" parent="base_link">
+      <origin xyz="0.328 -0.039 0.795" rpy="-0.055 1.212 -0.052" />
+  </xacro:realsense_d435>
+  <!-- tower middle camera -->
+  <xacro:sensor_orbbec_astra  name="tower_cam3d_middle" parent="base_link" color="">
+    <origin xyz="0.15 -0.06225 0.775" rpy="0 ${M_PI/2} ${-M_PI/2}" />
+  </xacro:sensor_orbbec_astra>
+  <!-- tower back camera -->
+  <xacro:realsense_d435  name="tower_cam3d_back" parent="base_link">
+    <origin xyz="-0.328 -0.039 0.795" rpy="0.0 ${-M_PI / 2} ${-M_PI / 2}" />
+  </xacro:realsense_d435>
+   <!-- <joint name="fixed_camera_joint" type="fixed">
        <origin xyz="0.0149 0.0325 0.0125" rpy="${-M_PI/2} 0 ${-M_PI/2}" />
        <parent link="arm_cam3d_camera_link"/>
        <child link="fixed_camera_link"/>
-   </joint>
+   </joint> -->
    <!-- we create a fixed link from arm_cam3d_camera_link to
         arm_cam3d_camera_color_optical_frame. See commit: https://github.com/b-it-bots/mas_industrial_robotics/commit/f6e3bfa997b430278adbf4b552a285ce43e47936 -->
         <!-- this also means you have to edit the source frame of the input
              pointcloud before transforming it. see commit: https://github.com/b-it-bots/mas_industrial_robotics/commit/f4dd2f3124779fbedd28beb636e9ca7019baa9cf -->
-   <link name="fixed_camera_link">
+   <!-- <link name="fixed_camera_link">
        <visual>
            <geometry>
@@ -84,5 +90,5 @@
            </geometry>
        </collision>
-   </link>
+   </link> -->
    <!-- tower vertical mount link -->
   <link name="tower_camera_stand_link">

Commit message: [mir_hardware_config] Added joints for realsense camera and its 3D printed mount

File: mir_robots/mir_hardware_config/youbot-brsu-2/urdf/robot.urdf.xacro (robot description, xacro)
@@ -59,6 +59,6 @@
   </xacro:intel_realsense_f200_camera -->
   <!-- tower front camera -->
-  <xacro:realsense_d435 name="tower_cam3d_front" parent="base_link">
-      <origin xyz="0.328 -0.039 0.795" rpy="-0.055 1.212 -0.052" />
+  <xacro:realsense_d435 name="tower_cam3d_front" parent="tower_camera_front_bolt_link">
+      <origin xyz="0.0 0.0 0.0" rpy="0.0 0.0 0.0" />
   </xacro:realsense_d435>
   <!-- tower middle camera -->
@@ -67,6 +67,6 @@
   </xacro:sensor_orbbec_astra>
   <!-- tower back camera -->
-  <xacro:realsense_d435  name="tower_cam3d_back" parent="base_link">
-    <origin xyz="-0.328 -0.039 0.795" rpy="0.0 ${-M_PI / 2} ${-M_PI / 2}" />
+  <xacro:realsense_d435  name="tower_cam3d_back" parent="tower_camera_back_bolt_link">
+    <origin xyz="0.0 0.0 0.0" rpy="0 0 0" />
   </xacro:realsense_d435>
    <!-- <joint name="fixed_camera_joint" type="fixed">
@@ -154,4 +154,16 @@
     <child link="tower_camera_stand_link_horizontal"/>
   </joint>
+  <link name="tower_camera_stand_link_horizontal_front" />
+  <joint name="tower_camera_stand_joint_horizontal_front" type="fixed">
+    <origin xyz="0.0 0.0 0.304" rpy="0 0 0" />
+    <parent link="tower_camera_stand_link_horizontal"/>
+    <child link="tower_camera_stand_link_horizontal_front"/>
+  </joint>
+  <link name="tower_camera_stand_link_horizontal_back" />
+  <joint name="tower_camera_stand_joint_horizontal_back" type="fixed">
+    <origin xyz="0.0 0.0 -0.304" rpy="${M_PI} 0 0" />
+    <parent link="tower_camera_stand_link_horizontal"/>
+    <child link="tower_camera_stand_link_horizontal_back"/>
+  </joint>
   <!-- tower front camera mount link -->
   <link name="tower_camera_front_mount_link">
@@ -171,7 +183,14 @@
   </link>
   <joint name="tower_camera_front_mount_joint" type="fixed">
-    <origin xyz="0.0 0.0 0.304" rpy="-${M_PI/2} ${M_PI/2} 0" />
-    <parent link="tower_camera_stand_link_horizontal"/>
+    <origin xyz="0.0 0.0 0.0" rpy="-${M_PI/2} ${M_PI/2} 0" />
+    <parent link="tower_camera_stand_link_horizontal_front"/>
     <child link="tower_camera_front_mount_link"/>
+  </joint>
+  <link name="tower_camera_front_bolt_link" />
+  <!-- final joint values = xyz="0.016645 0.0 0.028855 " (middle of 2 holes) +  xyz="0.0125 0.0 -0.009 " (distance from holes to bolt)-->
+  <joint name="tower_camera_front_bolt_joint" type="fixed">
+    <origin xyz="0.029145 0.0 0.019855" rpy="0 -0.37 0" />
+    <parent link="tower_camera_stand_link_horizontal_front"/>
+    <child link="tower_camera_front_bolt_link"/>
   </joint>
   <!-- tower back camera mount link -->
@@ -192,7 +211,13 @@
   </link>
   <joint name="tower_camera_back_mount_joint" type="fixed">
-    <origin xyz="0.0 0.0 -0.304" rpy="${M_PI} -${M_PI/2} -${M_PI/2}" />
-    <parent link="tower_camera_stand_link_horizontal"/>
+    <origin xyz="0.0 0.0 0.0" rpy="-${M_PI} ${M_PI/2} -${M_PI/2}" />
+    <parent link="tower_camera_stand_link_horizontal_back"/>
     <child link="tower_camera_back_mount_link"/>
+  </joint>
+  <link name="tower_camera_back_bolt_link" />
+  <joint name="tower_camera_back_bolt_joint" type="fixed">
+    <origin xyz="0.029145 0.0 0.019855" rpy="0 -0.37 0" />
+    <parent link="tower_camera_stand_link_horizontal_back"/>
+    <child link="tower_camera_back_bolt_link"/>
   </joint>
   <!-- tower side camera mount link -->

Commit message: [mir_hardware_config] Added 3D printed camera mounts STL files

File: mir_robots/mir_hardware_config/youbot-brsu-2/urdf/robot.urdf.xacro (robot description, xacro)
@@ -116,13 +116,13 @@
     <visual>
       <geometry>
-        <mesh filename="package://mir_description/meshes/e_stop_mount.STL" scale="0.001 0.001 0.001"/>
-      </geometry>
-      <material name="">
-          <color rgba="0.85098 0.85098 0.85098 1"/>
-      </material>
-    </visual>
-    <collision>
-      <geometry>
-        <mesh filename="package://mir_description/meshes/e_stop_mount.STL" scale="0.001 0.001 0.001"/>
+        <mesh filename="package://mir_description/meshes/misc/e_stop_mount.STL" scale="0.001 0.001 0.001"/>
+      </geometry>
+      <material name="">
+          <color rgba="0.85098 0.85098 0.85098 1"/>
+      </material>
+    </visual>
+    <collision>
+      <geometry>
+        <mesh filename="package://mir_description/meshes/misc/e_stop_mount.STL" scale="0.001 0.001 0.001"/>
       </geometry>
     </collision>
@@ -170,13 +170,13 @@
     <visual>
       <geometry>
-        <mesh filename="package://mir_description/meshes/intel_camera_mount.STL" scale="0.001 0.001 0.001"/>
-      </geometry>
-      <material name="">
-          <color rgba="0.85098 0.85098 0.85098 1"/>
-      </material>
-    </visual>
-    <collision>
-      <geometry>
-        <mesh filename="package://mir_description/meshes/intel_camera_mount.STL" scale="0.001 0.001 0.001"/>
+        <mesh filename="package://mir_description/meshes/sensor_mounts/intel_camera_mount.STL" scale="0.001 0.001 0.001"/>
+      </geometry>
+      <material name="">
+          <color rgba="0.85098 0.85098 0.85098 1"/>
+      </material>
+    </visual>
+    <collision>
+      <geometry>
+        <mesh filename="package://mir_description/meshes/sensor_mounts/intel_camera_mount.STL" scale="0.001 0.001 0.001"/>
       </geometry>
     </collision>
@@ -198,13 +198,13 @@
     <visual>
       <geometry>
-        <mesh filename="package://mir_description/meshes/intel_camera_mount.STL" scale="0.001 0.001 0.001"/>
-      </geometry>
-      <material name="">
-          <color rgba="0.85098 0.85098 0.85098 1"/>
-      </material>
-    </visual>
-    <collision>
-      <geometry>
-        <mesh filename="package://mir_description/meshes/intel_camera_mount.STL" scale="0.001 0.001 0.001"/>
+        <mesh filename="package://mir_description/meshes/sensor_mounts/intel_camera_mount.STL" scale="0.001 0.001 0.001"/>
+      </geometry>
+      <material name="">
+          <color rgba="0.85098 0.85098 0.85098 1"/>
+      </material>
+    </visual>
+    <collision>
+      <geometry>
+        <mesh filename="package://mir_description/meshes/sensor_mounts/intel_camera_mount.STL" scale="0.001 0.001 0.001"/>
       </geometry>
     </collision>
@@ -225,13 +225,13 @@
     <visual>
       <geometry>
-        <mesh filename="package://mir_description/meshes/side_camera_mount.STL" scale="0.001 0.001 0.001"/>
-      </geometry>
-      <material name="">
-          <color rgba="0.85098 0.85098 0.85098 1"/>
-      </material>
-    </visual>
-    <collision>
-      <geometry>
-        <mesh filename="package://mir_description/meshes/side_camera_mount.STL" scale="0.001 0.001 0.001"/>
+        <mesh filename="package://mir_description/meshes/sensor_mounts/side_camera_mount.STL" scale="0.001 0.001 0.001"/>
+      </geometry>
+      <material name="">
+          <color rgba="0.85098 0.85098 0.85098 1"/>
+      </material>
+    </visual>
+    <collision>
+      <geometry>
+        <mesh filename="package://mir_description/meshes/sensor_mounts/side_camera_mount.STL" scale="0.001 0.001 0.001"/>
       </geometry>
     </collision>

Commit message: [mir_bringup] updated launch files to include 3 cameras

File: mir_robots/mir_hardware_config/youbot-brsu-2/urdf/robot.urdf.xacro (robot description, xacro)
@@ -26,5 +26,6 @@
   <xacro:include filename="$(find mcr_description)/urdf/sensors/intel_realsense_f200_camera.urdf.xacro"/>
   <xacro:include filename="$(find mir_description)/urdf/sensors/asus_xtion_camera.urdf.xacro"/>
-  <xacro:include filename="$(find mcr_description)/urdf/sensors/realsense_d435.urdf.xacro"/>
+  <!-- xacro:include filename="$(find mcr_description)/urdf/sensors/realsense_d435.urdf.xacro"/ -->
+  <xacro:include filename="$(find realsense2_description)/urdf/_d435.urdf.xacro"/>
   <xacro:include filename="$(find youbot_description)/urdf/sensors/orbbec_astra.urdf.xacro"/>
   <xacro:include filename="$(find mir_description)/urdf/sensor_mounts/asus_xtion_camera_mount.urdf.xacro"/>
@@ -50,16 +51,9 @@
     <origin xyz="0.003 0 0.0052" rpy="0 0 0" />
   </xacro:dynamixel_gripper_v2>
-  <!-- camera mount for Intel RealSense F200 -->
-  <!--xacro:asus_xtion_camera_mount  name="camera_mount" parent="gripper_motor_mount_link">
-      <origin xyz="0.035 -0.00 0.0" rpy="0 0.025 ${M_PI/2} " />
-  </xacro:asus_xtion_camera_mount-->
-  <!-- 3D camera on arm -->
-  <!-- xacro:intel_realsense_f200_camera name="arm_cam3d" parent="camera_mount_link">
-    <origin xyz="-0.05 -0.01 0.03" rpy="0.0 -${M_PI/2 - 0.03} 0.0" />
-  </xacro:intel_realsense_f200_camera -->
   <!-- tower front camera -->
-  <xacro:realsense_d435 name="tower_cam3d_front" parent="tower_camera_front_bolt_link">
-      <origin xyz="0.0 0.0 0.0" rpy="0.0 0.0 0.0" />
-  </xacro:realsense_d435>
+  <xacro:sensor_d435 name="tower_cam3d_front_camera" parent="tower_camera_front_bolt_link" use_nominal_extrinsics="true">
+      <!-- <origin xyz="0.035 0.020 0.0" rpy="0.0 1.22 0.0" /> -->
+      <origin xyz="0.01 0.025 0.0" rpy="0.0 1.22 0.0" />
+  </xacro:sensor_d435>
   <!-- tower middle camera -->
   <xacro:sensor_orbbec_astra  name="tower_cam3d_middle" parent="base_link" color="">
@@ -67,28 +61,7 @@
   </xacro:sensor_orbbec_astra>
   <!-- tower back camera -->
-  <xacro:realsense_d435  name="tower_cam3d_back" parent="tower_camera_back_bolt_link">
+  <xacro:sensor_d435  name="tower_cam3d_back" parent="tower_camera_back_bolt_link" use_nominal_extrinsics="true">
     <origin xyz="0.0 0.0 0.0" rpy="0 0 0" />
-  </xacro:realsense_d435>
-   <!-- <joint name="fixed_camera_joint" type="fixed">
-       <origin xyz="0.0149 0.0325 0.0125" rpy="${-M_PI/2} 0 ${-M_PI/2}" />
-       <parent link="arm_cam3d_camera_link"/>
-       <child link="fixed_camera_link"/>
-   </joint> -->
-   <!-- we create a fixed link from arm_cam3d_camera_link to
-        arm_cam3d_camera_color_optical_frame. See commit: https://github.com/b-it-bots/mas_industrial_robotics/commit/f6e3bfa997b430278adbf4b552a285ce43e47936 -->
-        <!-- this also means you have to edit the source frame of the input
-             pointcloud before transforming it. see commit: https://github.com/b-it-bots/mas_industrial_robotics/commit/f4dd2f3124779fbedd28beb636e9ca7019baa9cf -->
-   <!-- <link name="fixed_camera_link">
-       <visual>
-           <geometry>
-               <box size="0.0000001 0.000001 0.000001"/>
-           </geometry>
-       </visual>
-       <collision>
-           <geometry>
-               <box size="0.0000001 0.000001 0.000001"/>
-           </geometry>
-       </collision>
-   </link> -->
+  </xacro:sensor_d435>
    <!-- tower vertical mount link -->
   <link name="tower_camera_stand_link">
@@ -122,9 +95,9 @@
       </material>
     </visual>
-    <collision>
+    <!-- <collision>
       <geometry>
         <mesh filename="package://mir_description/meshes/misc/e_stop_mount.STL" scale="0.001 0.001 0.001"/>
       </geometry>
-    </collision>
+    </collision> -->
   </link>
   <joint name="emergency_stop_mount_joint" type="fixed">
@@ -156,5 +129,5 @@
   <link name="tower_camera_stand_link_horizontal_front" />
   <joint name="tower_camera_stand_joint_horizontal_front" type="fixed">
-    <origin xyz="0.0 0.0 0.304" rpy="0 0 0" />
+    <origin xyz="0.0 0.0 0.304" rpy="0 -${M_PI/2} 0" />
     <parent link="tower_camera_stand_link_horizontal"/>
     <child link="tower_camera_stand_link_horizontal_front"/>
@@ -176,12 +149,12 @@
       </material>
     </visual>
-    <collision>
-      <geometry>
-        <mesh filename="package://mir_description/meshes/sensor_mounts/intel_camera_mount.STL" scale="0.001 0.001 0.001"/>
-      </geometry>
-    </collision>
+    <!-- <collision>
+      <geometry>
+        <mesh filename="package://mir_description/meshes/sensor_mounts/intel_camera_mount.STL" scale="0.001 0.001 0.001"/>
+      </geometry>
+    </collision> -->
   </link>
   <joint name="tower_camera_front_mount_joint" type="fixed">
-    <origin xyz="0.0 0.0 0.0" rpy="-${M_PI/2} ${M_PI/2} 0" />
+    <origin xyz="0.0 0.0 0.0" rpy="-${M_PI/2} ${M_PI} 0" />
     <parent link="tower_camera_stand_link_horizontal_front"/>
     <child link="tower_camera_front_mount_link"/>
@@ -190,5 +163,6 @@
   <!-- final joint values = xyz="0.016645 0.0 0.028855 " (middle of 2 holes) +  xyz="0.0125 0.0 -0.009 " (distance from holes to bolt)-->
   <joint name="tower_camera_front_bolt_joint" type="fixed">
-    <origin xyz="0.029145 0.0 0.019855" rpy="0 -0.37 0" />
+    <!-- Middle of camera back plate <origin xyz="0.028855 0.0 -0.016645" rpy="0 0 0" /> -->
+    <origin xyz="0.019855 0.0 -0.029145" rpy="0 0 0" />
     <parent link="tower_camera_stand_link_horizontal_front"/>
     <child link="tower_camera_front_bolt_link"/>
@@ -204,9 +178,9 @@
       </material>
     </visual>
-    <collision>
-      <geometry>
-        <mesh filename="package://mir_description/meshes/sensor_mounts/intel_camera_mount.STL" scale="0.001 0.001 0.001"/>
-      </geometry>
-    </collision>
+    <!-- <collision>
+      <geometry>
+        <mesh filename="package://mir_description/meshes/sensor_mounts/intel_camera_mount.STL" scale="0.001 0.001 0.001"/>
+      </geometry>
+    </collision> -->
   </link>
   <joint name="tower_camera_back_mount_joint" type="fixed">
@@ -231,9 +205,9 @@
       </material>
     </visual>
-    <collision>
+    <!-- <collision>
       <geometry>
         <mesh filename="package://mir_description/meshes/sensor_mounts/side_camera_mount.STL" scale="0.001 0.001 0.001"/>
       </geometry>
-    </collision>
+    </collision> -->
   </link>
   <joint name="tower_camera_side_mount_joint" type="fixed">

Commit message: [mir_hardware_config][urdf] updated back camera mount STL file and angle

File: mir_robots/mir_hardware_config/youbot-brsu-2/urdf/robot.urdf.xacro (robot description, xacro)
@@ -52,5 +52,5 @@
   </xacro:dynamixel_gripper_v2>
   <!-- tower front camera -->
-  <xacro:sensor_d435 name="tower_cam3d_front_camera" parent="tower_camera_front_bolt_link" use_nominal_extrinsics="true">
+  <xacro:sensor_d435 name="tower_cam3d_front" parent="tower_camera_front_bolt_link" use_nominal_extrinsics="true">
       <!-- <origin xyz="0.035 0.020 0.0" rpy="0.0 1.22 0.0" /> -->
       <origin xyz="0.01 0.025 0.0" rpy="0.0 1.22 0.0" />
@@ -61,6 +61,6 @@
   </xacro:sensor_orbbec_astra>
   <!-- tower back camera -->
-  <xacro:sensor_d435  name="tower_cam3d_back_camera" parent="tower_camera_back_bolt_link" use_nominal_extrinsics="true">
-    <origin xyz="0.0 0.0 0.0" rpy="0 0 0" />
+  <xacro:sensor_d435  name="tower_cam3d_back" parent="tower_camera_back_bolt_link" use_nominal_extrinsics="true">
+    <origin xyz="0.0 0.0 0.0" rpy="0.0 0.78 0.0" />
   </xacro:sensor_d435>
    <!-- tower vertical mount link -->
@@ -172,5 +172,6 @@
     <visual>
       <geometry>
-        <mesh filename="package://mir_description/meshes/sensor_mounts/intel_camera_mount.STL" scale="0.001 0.001 0.001"/>
+        <!-- <mesh filename="package://mir_description/meshes/sensor_mounts/intel_camera_mount.STL" scale="0.001 0.001 0.001"/> -->
+        <mesh filename="package://mir_description/meshes/sensor_mounts/intel_camera_mount_back.STL" scale="0.001 0.001 0.001"/>
       </geometry>
       <material name="">
