Commit message: [mir_hardware_config][yb2] camera name changes

File: mir_robots/mir_hardware_config/youbot-brsu-2/urdf/robot.urdf.xacro (robot description, xacro)
@@ -52,5 +52,5 @@
   </xacro:dynamixel_gripper_v2>
   <!-- tower front camera -->
-  <xacro:sensor_d435 name="tower_cam3d_front" parent="tower_camera_front_bolt_link" use_nominal_extrinsics="true">
+  <xacro:sensor_d435 name="tower_cam3d_front_camera" parent="tower_camera_front_bolt_link" use_nominal_extrinsics="true">
       <!-- <origin xyz="0.035 0.020 0.0" rpy="0.0 1.22 0.0" /> -->
       <origin xyz="0.01 0.025 0.0" rpy="0.0 1.22 0.0" />
@@ -61,5 +61,5 @@
   </xacro:sensor_orbbec_astra>
   <!-- tower back camera -->
-  <xacro:sensor_d435  name="tower_cam3d_back" parent="tower_camera_back_bolt_link" use_nominal_extrinsics="true">
+  <xacro:sensor_d435  name="tower_cam3d_back_camera" parent="tower_camera_back_bolt_link" use_nominal_extrinsics="true">
     <origin xyz="0.0 0.0 0.0" rpy="0.0 0.78 0.0" />
   </xacro:sensor_d435>
@@ -191,6 +191,8 @@
   </joint>
   <link name="tower_camera_back_bolt_link" />
+  <!-- final joint values = xyz="0.02121 0.00 0.02250 " (middle of 2 holes) +  xyz="0.0125 0.0 -0.009 " (distance from holes to bolt)-->
   <joint name="tower_camera_back_bolt_joint" type="fixed">
-    <origin xyz="0.029145 0.0 0.019855" rpy="0 -0.37 0" />
+    <origin xyz="0.00871 0.0 0.03150" rpy="0 -0.78 0" />
+    <!-- <origin xyz="0.029145 0.0 0.019855" rpy="0 -0.37 0" /> -->
     <parent link="tower_camera_stand_link_horizontal_back"/>
     <child link="tower_camera_back_bolt_link"/>

Commit message: [mir_hardware_config][urdf] disabled middle camera

File: mir_robots/mir_hardware_config/youbot-brsu-2/urdf/robot.urdf.xacro (robot description, xacro)
@@ -28,5 +28,5 @@
   <!-- xacro:include filename="$(find mcr_description)/urdf/sensors/realsense_d435.urdf.xacro"/ -->
   <xacro:include filename="$(find realsense2_description)/urdf/_d435.urdf.xacro"/>
-  <xacro:include filename="$(find youbot_description)/urdf/sensors/orbbec_astra.urdf.xacro"/>
+  <!-- <xacro:include filename="$(find youbot_description)/urdf/sensors/orbbec_astra.urdf.xacro"/> -->
   <xacro:include filename="$(find mir_description)/urdf/sensor_mounts/asus_xtion_camera_mount.urdf.xacro"/>
   <!-- Now we can start using the macros included above to define the actual youbot -->
@@ -57,7 +57,7 @@
   </xacro:sensor_d435>
   <!-- tower middle camera -->
-  <xacro:sensor_orbbec_astra  name="tower_cam3d_middle" parent="base_link" color="">
+  <!-- <xacro:sensor_orbbec_astra  name="tower_cam3d_middle" parent="base_link" color="">
     <origin xyz="0.15 -0.06225 0.775" rpy="0 ${M_PI/2} ${-M_PI/2}" />
-  </xacro:sensor_orbbec_astra>
+  </xacro:sensor_orbbec_astra> -->
   <!-- tower back camera -->
   <xacro:sensor_d435  name="tower_cam3d_back_camera" parent="tower_camera_back_bolt_link" use_nominal_extrinsics="true">
@@ -193,5 +193,5 @@
   <!-- final joint values = xyz="0.02121 0.00 0.02250 " (middle of 2 holes) +  xyz="0.0125 0.0 -0.009 " (distance from holes to bolt)-->
   <joint name="tower_camera_back_bolt_joint" type="fixed">
-    <origin xyz="0.00871 0.0 0.03150" rpy="0 -0.78 0" />
+    <origin xyz="0.00871 0.0 0.03150" rpy="0 -1.57 0" />
     <!-- <origin xyz="0.029145 0.0 0.019855" rpy="0 -0.37 0" /> -->
     <parent link="tower_camera_stand_link_horizontal_back"/>
@@ -199,5 +199,5 @@
   </joint>
   <!-- tower side camera mount link -->
-  <link name="tower_camera_side_mount_link">
+  <!-- <link name="tower_camera_side_mount_link">
     <visual>
       <geometry>
@@ -208,9 +208,4 @@
       </material>
     </visual>
-    <!-- <collision>
-      <geometry>
-        <mesh filename="package://mir_description/meshes/sensor_mounts/side_camera_mount.STL" scale="0.001 0.001 0.001"/>
-      </geometry>
-    </collision> -->
   </link>
   <joint name="tower_camera_side_mount_joint" type="fixed">
@@ -218,4 +213,4 @@
     <parent link="tower_camera_stand_link_horizontal"/>
     <child link="tower_camera_side_mount_link"/>
-  </joint>
+  </joint> -->
 </robot>

Commit message: [camera calibration] updated camera calibration parameters

File: mir_robots/mir_hardware_config/youbot-brsu-2/urdf/robot.urdf.xacro (robot description, xacro)
@@ -53,6 +53,7 @@
   <!-- tower front camera -->
   <xacro:sensor_d435 name="tower_cam3d_front_camera" parent="tower_camera_front_bolt_link" use_nominal_extrinsics="true">
+     <!-- camera calibration -->
       <!-- <origin xyz="0.035 0.020 0.0" rpy="0.0 1.22 0.0" /> -->
-      <origin xyz="0.01 0.025 0.0" rpy="0.0 1.22 0.0" />
+      <origin xyz="0.015 -0.005 0.0" rpy="0.0 1.22 0.0" />
   </xacro:sensor_d435>
   <!-- tower middle camera -->

Commit message: [urdf] camera calib; object was being grasped too far in front

File: mir_robots/mir_hardware_config/youbot-brsu-2/urdf/robot.urdf.xacro (robot description, xacro)
@@ -55,5 +55,5 @@
      <!-- camera calibration -->
       <!-- <origin xyz="0.035 0.020 0.0" rpy="0.0 1.22 0.0" /> -->
-      <origin xyz="0.015 -0.005 0.0" rpy="0.0 1.22 0.0" />
+      <origin xyz="0.010 -0.005 0.0" rpy="0.0 1.22 0.0" />
   </xacro:sensor_d435>
   <!-- tower middle camera -->
